File: Hardware/3/stm32hw03.brd (EAGLE design)
At the start: 100 x 80 mm, 90 parts, among them CN1 AC 9V, Q1 NPN, Q2 NPN, T1 PNP, U1 STM32F303_334RXT

Commit message: rpi upload example
Parts:
- added C22: 1uF, resistor:C0603
- C4: value 1uF -> 4.7uF
Connections:
- net +3V3: now also C22.2
- net GND: now also C22.1
Changed lines of the file:
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@@
 <attribute name="VALUE" x="53.9085" y="16.0355" size="0.8128" layer="27" font="vector" ratio="20"/>
 </element>
-<element name="C4" library="resistor" package="C0603" value="1uF" x="59.75" y="17.75" smashed="yes">
+<element name="C4" library="resistor" package="C0603" value="4.7uF" x="59.75" y="17.75" smashed="yes">
 <attribute name="NAME" x="61.274" y="16.988" size="0.8128" layer="25" font="vector" ratio="20" rot="R180"/>
 <attribute name="VALUE" x="61.274" y="19.4645" size="0.8128" layer="27" font="vector" ratio="20" rot="R180"/>
@@
 <attribute name="OC_FARNELL" value="unknown" x="42.5" y="2.5" size="0.8128" layer="27" font="vector" ratio="20" rot="R180" display="off"/>
 </element>
+<element name="C22" library="resistor" package="C0603" value="1uF" x="31.5" y="37" rot="R270"/>
 </elements>
 <signals>
@@
 <contactref element="RASPBERRYPI" pad="5"/>
 <contactref element="RASPBERRYPI" pad="10"/>
+<contactref element="C22" pad="1"/>
 <wire x1="83.45" y1="21.75" x2="85" y2="25.25" width="0" layer="19" extent="1-1"/>
 <wire x1="68.55" y1="17" x2="80.25" y2="26.65" width="0" layer="19" extent="1-1"/>
@@
 <wire x1="60.85" y1="2" x2="60.25" y2="10.75" width="0" layer="19" extent="1-1"/>
 <wire x1="39.624" y1="38.143" x2="48.624" y2="35.643" width="0" layer="19" extent="1-1"/>
+<wire x1="31.5" y1="37.85" x2="36.25" y2="38.6" width="0" layer="19" extent="1-1"/>
 <wire x1="37.857" y1="44.643" x2="36.25" y2="38.6" width="0" layer="19" extent="1-1"/>
 <wire x1="43.624" y1="47.143" x2="39.624" y2="44.643" width="0" layer="19" extent="1-1"/>
@@
 <wire x1="27.5" y1="52" x2="26.6" y2="56.75" width="0" layer="19" extent="1-1"/>
 <wire x1="27.5" y1="49.46" x2="27.35" y2="51.85" width="0" layer="19" extent="1-1"/>
+<wire x1="23.5" y1="37.85" x2="31.5" y2="37.85" width="0" layer="19" extent="1-1"/>
+<wire x1="19.75" y1="38" x2="23.5" y2="37.85" width="0" layer="19" extent="1-1"/>
+<wire x1="21" y1="29.35" x2="19.75" y2="38" width="0" layer="19" extent="1-1"/>
 <wire x1="27.5" y1="14.5" x2="36.75" y2="17.75" width="0" layer="19" extent="1-1"/>
 <wire x1="27.5" y1="11.96" x2="27.5" y2="14.5" width="0" layer="19" extent="1-1"/>
-<wire x1="23.5" y1="37.85" x2="30.25" y2="45.35" width="0" layer="19" extent="1-1"/>
-<wire x1="19.75" y1="38" x2="23.5" y2="37.85" width="0" layer="19" extent="1-1"/>
-<wire x1="21" y1="29.35" x2="19.75" y2="38" width="0" layer="19" extent="1-1"/>
 <wire x1="3.75" y1="34" x2="14.05" y2="28.55" width="0" layer="19" extent="1-1"/>
-<wire x1="43" y1="1.23" x2="27.5" y2="11.96" width="0" layer="19" extent="1-1"/>
-<wire x1="37.92" y1="3.77" x2="43" y2="1.23" width="0" layer="19" extent="1-1"/>
+<wire x1="37.92" y1="3.77" x2="27.5" y2="11.96" width="0" layer="19" extent="1-1"/>
+<wire x1="43" y1="1.23" x2="37.92" y2="3.77" width="0" layer="19" extent="1-1"/>
 </signal>
 <signal name="OSC_IN">
@@
 <contactref element="CH_PD" pad="1"/>
 <contactref element="C21" pad="2"/>
+<contactref element="C22" pad="2"/>
 <wire x1="60.63" y1="47.34" x2="64.185" y2="50.73" width="0" layer="19" extent="1-1"/>
 <wire x1="54.93" y1="47.545" x2="60.63" y2="47.34" width="0" layer="19" extent="1-1"/>
@@
 <wire x1="39.624" y1="44.143" x2="43.124" y2="47.143" width="0" layer="19" extent="1-1"/>
 <wire x1="33.25" y1="40.15" x2="36.25" y2="43.65" width="0" layer="19" extent="1-1"/>
+<wire x1="31.5" y1="36.15" x2="33.25" y2="37.75" width="0" layer="19" extent="1-1"/>
+<wire x1="23.5" y1="36.15" x2="31.5" y2="36.15" width="0" layer="19" extent="1-1"/>
+<wire x1="19.75" y1="36" x2="23.5" y2="36.15" width="0" layer="19" extent="1-1"/>
 <wire x1="42.75" y1="30.6" x2="39.624" y2="37.643" width="0" layer="19" extent="1-1"/>
 <wire x1="49.124" y1="35.643" x2="42.75" y2="30.6" width="0" layer="19" extent="1-1"/>
-<wire x1="23.5" y1="36.15" x2="33.25" y2="37.75" width="0" layer="19" extent="1-1"/>
-<wire x1="19.75" y1="36" x2="23.5" y2="36.15" width="0" layer="19" extent="1-1"/>
 <wire x1="24" y1="44.4" x2="23.5" y2="36.15" width="0" layer="19" extent="1-1"/>
 <wire x1="24" y1="50.15" x2="24" y2="44.4" width="0" layer="19" extent="1-1"/>
