File: Hardware/3/stm32hw03.sch (EAGLE design)
At the start: 90 parts, among them CN1 AC 9V, Q1 NPN, Q2 NPN, T1 PNP, U1 STM32F303_334RXT

Commit message: rpi upload example
Parts:
- added C22: 1uF, resistor:C-EUC0603
- C4: value 1uF -> 4.7uF
Connections:
- net +3V3: now also C22.2
- net GND: now also C22.1
Changed lines of the file:
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@@
 <part name="P+3" library="supply1" deviceset="+5V" device=""/>
 <part name="+3V1" library="supply1" deviceset="+3V3" device=""/>
-<part name="C4" library="resistor" deviceset="C-EU" device="C0603" value="1uF"/>
+<part name="C4" library="resistor" deviceset="C-EU" device="C0603" value="4.7uF"/>
 <part name="C5" library="resistor" deviceset="C-EU" device="C0603" value="100nF"/>
 <part name="C6" library="resistor" deviceset="C-EU" device="C0603" value="100nF"/>
@@
 <part name="GND5" library="supply1" deviceset="GND" device=""/>
 <part name="GND7" library="supply1" deviceset="GND" device=""/>
+<part name="C22" library="resistor" deviceset="C-EU" device="C0603" value="1uF"/>
 </parts>
 <sheets>
@@
 <instance part="GND5" gate="1" x="205.74" y="-86.36"/>
 <instance part="GND7" gate="1" x="256.54" y="-86.36"/>
+<instance part="C22" gate="G$1" x="58.42" y="167.64" rot="R180"/>
 </instances>
 <busses>
@@
 <wire x1="15.24" y1="162.56" x2="26.67" y2="162.56" width="0.1524" layer="91"/>
 <wire x1="26.67" y1="162.56" x2="36.83" y2="162.56" width="0.1524" layer="91"/>
-<wire x1="36.83" y1="162.56" x2="46.99" y2="162.56" width="0.1524" layer="91"/>
+<wire x1="36.83" y1="162.56" x2="45.72" y2="162.56" width="0.1524" layer="91"/>
+<wire x1="45.72" y1="162.56" x2="46.99" y2="162.56" width="0.1524" layer="91"/>
 <wire x1="3.81" y1="165.1" x2="3.81" y2="162.56" width="0.1524" layer="91"/>
 <pinref part="C6" gate="G$1" pin="1"/>
@@
 <pinref part="SUPPLY7" gate="GND" pin="GND"/>
 <junction x="-25.4" y="158.75"/>
+<wire x1="46.99" y1="162.56" x2="58.42" y2="162.56" width="0.1524" layer="91"/>
+<pinref part="C22" gate="G$1" pin="1"/>
+<wire x1="58.42" y1="162.56" x2="58.42" y2="165.1" width="0.1524" layer="91"/>
 </segment>
 <segment>
@@
 <junction x="36.83" y="172.72"/>
 <pinref part="C9" gate="G$1" pin="2"/>
-<wire x1="36.83" y1="172.72" x2="46.99" y2="172.72" width="0.1524" layer="91"/>
-</segment>
-<segment>
+<wire x1="36.83" y1="172.72" x2="45.72" y2="172.72" width="0.1524" layer="91"/>
+<pinref part="C22" gate="G$1" pin="2"/>
+<wire x1="45.72" y1="172.72" x2="46.99" y2="172.72" width="0.1524" layer="91"/>
+<wire x1="46.99" y1="172.72" x2="58.42" y2="172.72" width="0.1524" layer="91"/>
+</segment>
+<segment>
