File: Hardware/4/stm32hw03.brd (EAGLE design)
At the start: 54 x 55 mm, 50 parts, among them CN1 AC 9V, U1 STM32F303_334RXT

Commit message: v5 design
Parts:
- added C16: 100nF, resistor:C0603
- added LED1: Red 1.85V, adafruit:CHIP-LED0805
- added R1: 4.7k, resistor:R0603
- added R3: 1K, rcl:R0603
- R10, R12, R21, R8: value 1k -> 330R
Connections:
- net OSC_IN renamed LSE_IN
- net OSC_OUT renamed LSE_OUT
- removed net USB_DM: U1.44
- removed net USB_DP: U1.45
- new net DS18B20: R1.1, T2.1, U1.42
- new net LED: R3.2, U1.41
- new net N$41: LED1.A, R3.1
- new net N$7: T1.2
- new net N$9: T1.3
- new net PULSE: C16.2, T2.2, U1.43
- net +3V3: now also R1.2, T1.1
- net BIAS: now also U1.22; no longer U1.27
- net BIAS_IN: now also U1.23; no longer U1.26
- net CT1: now also U1.14
- net CT3: now also U1.16; no longer U1.14
- net GND: now also C16.1, LED1.C, T2.3
- net UART2_RX: no longer U1.17
- net UART2_TX: no longer U1.16
Routing:
- net BIAS: track 103.6 -> 97.4 mm
- net BIAS_IN: track 11.7 -> 10.4 mm
