File: Hardware/5/stm32hw05.brd (EAGLE design)
At the start: 54 x 55 mm, 46 parts

Commit message: gerbers
Connections:
- net +3V3: no longer RASPBERRYPI.2
- net +5V: now also RASPBERRYPI.1, RASPBERRYPI.3
Routing:
- net +5V: track 75.5 -> 95.0 mm
Other:
- board text added: "Designed in"
- board text added: "Made in UK"
- board text added: "North Wales"
