File: stm_may2019/v0.1.brd (EAGLE design)
At the start: 128.9 x 99.5 mm, 91 parts, among them J1 RJ45, J2 USB_A_SMT_FEMALE, J3 RJ45, J5 RJ45, Y1 32.768kHz

Commit message: COMMIT
Parts:
- added MODULE_HEADER: (no value), con-lsta-RFM69Pi:FE12-2
- moved GND 2.54 mm to (54.2, 66.6)
- moved SJ1 2.53 mm to (51.8, 63.0)
Routing:
- net +3V3: track 307.9 -> 306.2 mm
- net CT8: track 50.7 -> 52.2 mm
- net UART_TX: track 13.1 -> 11.8 mm
- net N$1: track 2.45 -> 3.26 mm
- net +5V: track 101.0 -> 101.7 mm
- net CT9: track 82.6 -> 83.3 mm
