File: stm_may2019/v0.1.sch (EAGLE design)
At the start: 90 parts, among them J1 RJ45, J2 USB_A_SMT_FEMALE, J3 RJ45, J5 RJ45, Y1 32.768kHz

Commit message: COMMIT
Parts:
- added MODULE_HEADER: (no value), con-lsta-RFM69Pi:FE12-2
Other:
- note added: "Expansion module interface. For vertically stacked modules."
Changed lines of the file:
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@@
 <part name="U$11" library="OMNIMATE_LSF" deviceset="OMNIMATE_LSF_2" device=""/>
 <part name="U$1" library="con-molex-usb" deviceset="MICRO-USB-RECEPTACLE" device="47589-0001"/>
+<part name="MODULE_HEADER" library="con-lsta-RFM69Pi" deviceset="FE12-2" device="" package3d_urn="urn:adsk.eagle:package:8178/1"/>
 </parts>
 <sheets>
@@
 <text x="-8.89" y="88.9" size="1.778" layer="91" rot="R90">Frequency 8MHZ to 32MHZ</text>
 <text x="240.792" y="-5.588" size="1.778" layer="95">Mbus</text>
+<text x="21.59" y="-182.245" size="1.778" layer="91">Expansion module interface.
+For vertically stacked modules.</text>
 </plain>
 <instances>
@@
 <attribute name="VALUE" x="309.88" y="-15.24" size="1.778" layer="96" font="vector" rot="R270"/>
 </instance>
+<instance part="MODULE_HEADER" gate="1" x="50.8" y="-200.66" smashed="yes" rot="R90">
+<attribute name="VALUE" x="71.12" y="-204.47" size="1.778" layer="96" rot="R90"/>
+<attribute name="NAME" x="34.798" y="-204.47" size="1.778" layer="95" rot="R90"/>
+</instance>
 </instances>
