File: stm_may2019/stm v0.1.brd (EAGLE design)
At the start: 128.9 x 99.5 mm, 92 parts, among them J1 RJ45, J2 USB_A_SMT_FEMALE, J3 RJ45, J5 RJ45, Y1 32.768kHz

Commit message: commit
Parts:
- removed J2: USB_A_SMT_FEMALE, SparkFun-Connectors:USB-A-S-SILK-FEMALE
- removed J3, J5: RJ45, SparkFun-Connectors:RJ45-8
- added LED2, LED3: Red 1.85V, adafruit:CHIP-LED0805
- added R4, R5: 220R, rcl:R0603
- moved J1 119.5 mm to (9.45, 23.9), turned to 270 degrees
- moved ESP12 73.9 mm to (114.2, 62.9), turned to 90 degrees
- moved RFM69HCW 36.5 mm to (111.6, 38.4), turned to 180 degrees
- moved LED1 18.1 mm to (82.3, 51.9)
- moved MCP1825 11.5 mm to (104.6, 22.0)
- moved C22 11.2 mm to (103.0, 30.5)
- moved C4 10.7 mm to (108.0, 30.9)
- moved C3 6.90 mm to (113.2, 15.9)
- moved R1 1.28 mm to (70.3, 52.3)
- moved C8 0.42 mm to (50.6, 59.7)
Connections:
- removed net VBUS: J2.VBUS
- new net LED2: R4.2, STM32F303VB.56
- new net LED3: R5.2, STM32F303VB.57
- new net N$5: LED2.A, R4.1
- new net N$6: LED3.A, R5.1
- net GND: now also LED2.C, LED3.C; no longer J2.GND
- net LED1: now also STM32F303VB.55; no longer STM32F303VB.53
Routing:
- net N$41: track 2.53 -> 64.3 mm, vias 0 -> 2
- net +3V3: track 306.2 -> 345.1 mm, vias 3 -> 4
- net LED3: track 0.00 -> 27.8 mm, vias 0 -> 4
- net N$6: track 0.00 -> 18.0 mm
- net LED2: track 0.00 -> 16.8 mm, vias 0 -> 4
- net N$5: track 0.00 -> 14.8 mm, vias 0 -> 2
- net DS18B20: track 101.9 -> 107.8 mm
- net CT8: track 52.2 -> 56.2 mm
- net +5V: track 101.7 -> 99.3 mm
- net N$9: track 17.7 -> 19.2 mm
- net CT9: track 83.3 -> 84.5 mm, vias 0 -> 2
- net LED1: track 4.12 -> 4.98 mm, vias 0 -> 2
- net CT5: track 35.1 -> 35.7 mm
- net GND: track 0.00 -> 0.35 mm, vias 33 -> 41
Other:
- outline, holes or cut-outs redrawn
- board text removed: "SJ1"
