File: stm_may2019/stm v0.1.sch (EAGLE design)
At the start: 91 parts, among them J1 RJ45, J2 USB_A_SMT_FEMALE, J3 RJ45, J5 RJ45, Y1 32.768kHz

Commit message: commit
Parts:
- removed J2: USB_A_SMT_FEMALE, SparkFun-Connectors:USB_A_SMT_FEMALE
- removed J3, J5: RJ45, SparkFun-Connectors:RJ45-8
- added LED2, LED3: Red 1.85V, adafruit:LEDCHIP-LED0805
- added R4, R5: 220R, rcl:R-EU_R0603
Connections:
- new net LED2: R4.2, STM32F303VB.PD9
- new net LED3: R5.2, STM32F303VB.PD10
- new net N$5: LED2.A, R4.1
- new net N$6: LED3.A, R5.1
- net GND: now also LED2.C, LED3.C
- net LED1: now also STM32F303VB.PD8; no longer STM32F303VB.PB14
Other:
- moved on the sheet: BOOT0, C10, LED1, R2, R3, S1
