File: stm_may2019/stm v0.3.brd (EAGLE design)
At the start: 128.9 x 100.7 mm, 127 parts, among them Q1 MMBT3906, Q2 MMBT3904, Q3 MMBT3904, Y1 32.768kHz

Commit message: v0.3 and notes
Parts:
- added U$2: BOOST_MODULE, BOOST MODULE CN6009:BOOST
- moved SV1 1.27 mm to (97.8, 43.1)
- moved SV2 1.27 mm to (97.8, 55.8)
- moved U$1 1.27 mm to (126.9, 24.7)
- moved SJ2 1.01 mm to (52.6, 47.1)
- moved C3 0.52 mm to (116.3, 21.2)
- moved C2 0.18 mm to (114.0, 17.0)
Connections:
- net +5V: now also U$2.IN+
- net 24V: now also U$2.OUT+
- net GND: now also U$2.P$1, U$2.P$2
