File: stm_may2019/stm v0.3.sch (EAGLE design)
At the start: 92 parts, among them J1 RJ45, Y1 32.768kHz

Commit message: v0.3
Parts:
- removed MODULE_HEADER: (no value), con-lsta-RFM69Pi:FE12-2
- removed PCB1: RPI3RPI3, e14_Rpi3_RevA+mirror-pcb copy:RPI3RPI3
- removed U$11: OMNIMATE_LSF_2, OMNIMATE_LSF:OMNIMATE_LSF_2
- added 2POLE_MBUS: OMNIMATE_LSF_2, OMNIMATE_LSF:OMNIMATE_LSF_2
- added 3POLE_4, 3POLE_5, 3POLE_6: OMNIMATE_LSF_3, OMNIMATE_LSF:OMNIMATE_LSF_3
- added BOOT_ESP: (no value), SparkFun:M02PTH
- added C1, C2: 100nF, resistor:C-EUC0603
- added J$1: SMA_EDGE, SparkFun-Connectors:SMA_EDGE
- added PCB2: RPI3YA, e14_Rpi3_RevA+mirror-pcb copy:RPI3YA
- added Q1: MMBT3906, Transistor:MMBT3906
- added Q2, Q3: MMBT3904, Transistor:MMBT3904
- added R11: 33K, rcl:R-EU_R0603
- added R14: 22K, rcl:R-EU_R0603
- added R15: 3k3, rcl:R-EU_R0603
- added R16: 82R, rcl:R-EU_R0603
- added R17: 220K, rcl:R-EU_R0603
- added R18, R19: 1K, rcl:R-EU_R0603
- added R6, R7: 10k, resistor:R-EU_R0603
- added R9: 39K, rcl:R-EU_R0603
- added SJ10, SJ11, SJ12, SJ2, SJ3, SJ4, SJ5, SJ6, SJ7, SJ8, SJ9: SOLDERJUMPERNO, SparkFun:SOLDERJUMPERNO
- added SV1, SV2: (no value), con-lsta-RFM69Pi:FE05-2
- added U$8: MCP1501T-33E, MCP1501T-33E:MCP1501T-33E
- added UART_ESP: (no value), con-lstb-db:MA06-1
- renumbered BOOT0 to BOOT_STM, J1 to RJ45_1, U$4 to 3POLE_1, U$5 to 3POLE_2, U$6 to 3POLE_3
Connections:
- removed net N$9: RFM69HCW.GND, RFM69HCW.GND@1
- new net +3V3_ADC: SJ2.2, STM32F303VB.VDDA, U$8.OUT
- new net 24V: 2POLE_MBUS.2, R11.2, R17.2, R9.2
- new net ADC_RJ45IN: RJ45_1.8, STM32F303VB.PA3
- new net ANT: J$1.SIGNAL, RFM69HCW.ANT
- new net CS_RFM69: PCB2.GPIO25, RFM69HCW.!SEL
- new net MBUS_RX: R18.2, SJ11.2
- new net MBUS_TX: R19.2, SJ12.2
- new net MISO: PCB2.GPIO9, RFM69HCW.SDO, SJ6.2
- new net MOSI: PCB2.GPIO10, RFM69HCW.SDI, SJ5.2
- new net N$11: ESP12.GPIO2, R6.1
- new net N$16: PCB2.GPIO12, SJ8.1
- new net N$19: ESP12.GPIO15, R7.1
- new net N$22: PCB2.3V3@1
- new net N$24: PCB2.3V3@17
- new net N$29: 2POLE_MBUS.1, Q1.E, R17.1
- new net N$30: Q1.C, Q2.B, R16.2
- new net N$31: Q1.B, Q3.C, R14.2, R9.1
- new net N$32: Q2.C, R11.1, R15.2, R19.1
- new net N$33: Q3.B, R18.1
- new net PUSHIN_3: 3POLE_3.2, STM32F303VB.PD0
- new net PUSHIN_4: 3POLE_4.2, STM32F303VB.PD1
- new net PUSHIN_5: 3POLE_5.2, STM32F303VB.PD2
- new net PUSHIN_6: 3POLE_6.2, STM32F303VB.PD3
- new net RST_ESP_1: C1.2, UART_ESP.6
- new net RST_ESP_2: C1.1, ESP12.RESET
- new net RXD0: PCB2.GPIO15, SJ12.1, SJ4.1
- new net SPI3_CLK: SJ7.1, STM32F303VB.PC10
- new net SPI3_CS: SJ8.2, STM32F303VB.PA15
- new net SPI3_MISO: SJ6.1, STM32F303VB.PC11
- new net SPI3_MOSI: SJ5.1, STM32F303VB.PC12
- new net SPI_CLK: PCB2.GPIO11, RFM69HCW.SCK, SJ7.2
- new net TXD0: PCB2.GPIO14, SJ11.1, SJ3.1
- new net UART_RX_ESP: ESP12.TX, SJ9.2, UART_ESP.4
- new net UART_TX_ESP: ESP12.RX, SJ10.1, UART_ESP.5
- new net USART3_RX: SJ3.2, SJ9.1, STM32F303VB.PB11
- new net USART3_TX: SJ10.2, SJ4.2, STM32F303VB.PB10
- net +3V3: now also 3POLE_3.1, 3POLE_4.1, 3POLE_5.1, 3POLE_6.1, C2.1, R6.2, RJ45_1.2, SJ2.1, U$8.SHT_DN, UART_ESP.2; no longer STM32F303VB.VDDA
- net +5V: now also PCB2.5V@2, PCB2.5V@4, RJ45_1.7, U$8.VDD, UART_ESP.3
- net DS18B20: now also RJ45_1.4, STM32F303VB.PB13; no longer STM32F303VB.PB10
- net GND: now also 3POLE_3.3, 3POLE_4.3, 3POLE_5.3, 3POLE_6.3, BOOT_ESP.2, C2.2, J$1.GND@0, J$1.GND@1, J$1.GND@2, J$1.GND@3, PCB2.GND@14, PCB2.GND@20, PCB2.GND@25, PCB2.GND@30, PCB2.GND@34, PCB2.GND@39, PCB2.GND@6, PCB2.GND@9, Q2.E, Q3.E, R14.1, R15.1, R16.1, R7.2, RFM69HCW.GND, RFM69HCW.GND@1, RJ45_1.1, RJ45_1.3, RJ45_1.5, U$8.GND, UART_ESP.1
- net N$7: now also BOOT_ESP.1, ESP12.GPIO0; no longer ESP12.RESET
- net PULSE: now also RJ45_1.6
Other:
- note removed: "Expansion module interface. For vertically stacked modules."

Commit message: v0.3 and notes
Parts:
- added U$2: BOOST_MODULE, BOOST MODULE CN6009:BOOST_MODULE
Connections:
- net +5V: now also U$2.+5V
- net 24V: now also U$2.24V
- net GND: now also U$2.GND, U$2.GND.
Changed lines of the file:
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@@
 <part name="RFM69HCW" library="rfm12b _ rfm69cw" deviceset="RFM12_SMD" device="SMD"/>
 <part name="SUPPLY33" library="supply2" library_urn="urn:adsk.eagle:library:372" deviceset="GND" device=""/>
+<part name="U$2" library="BOOST MODULE CN6009" deviceset="BOOST_MODULE" device=""/>
 </parts>
 <sheets>
@@
 <attribute name="VALUE" x="117.602" y="-94.742" size="1.778" layer="96"/>
 </instance>
+<instance part="U$2" gate="G$1" x="347.98" y="-175.26" smashed="yes"/>
 </instances>
 <busses>
@@
 <junction x="134.62" y="-134.62"/>
 </segment>
+<segment>
+<pinref part="U$2" gate="G$1" pin="GND."/>
+<wire x1="363.22" y1="-180.34" x2="368.3" y2="-180.34" width="0.1524" layer="91"/>
+<label x="365.76" y="-182.88" size="1.778" layer="95"/>
+</segment>
+<segment>
+<pinref part="U$2" gate="G$1" pin="GND"/>
+<wire x1="330.2" y1="-180.34" x2="325.12" y2="-180.34" width="0.1524" layer="91"/>
+<label x="325.12" y="-182.88" size="1.778" layer="95"/>
+</segment>
 </net>
 <net name="+5V" class="1">
@@
 <wire x1="325.12" y1="10.16" x2="302.26" y2="10.16" width="0.1524" layer="91"/>
 <label x="302.26" y="10.16" size="1.778" layer="95"/>
+</segment>
+<segment>
+<pinref part="U$2" gate="G$1" pin="+5V"/>
+<wire x1="330.2" y1="-165.1" x2="325.12" y2="-165.1" width="0.1524" layer="91"/>
+<label x="322.58" y="-165.1" size="1.778" layer="95"/>
 </segment>
 </net>
@@
 <wire x1="322.58" y1="-141.224" x2="322.58" y2="-137.16" width="0.1524" layer="91"/>
 </segment>
-</net>
+<segment>
+<pinref part="U$2" gate="G$1" pin="24V"/>
+<wire x1="363.22" y1="-165.1" x2="368.3" y2="-165.1" width="0.1524" layer="91"/>
+<label x="367.792" y="-163.83" size="1.778" layer="95"/>
+</segment>
+</net>
