File: stm32-pi/stm v0.4.sch (EAGLE design)
At the start: 139 parts, among them Q1 MMBT3906, Q2 MMBT3904, Q3 MMBT3904, Y1 32.768kHz

Commit message: update v0.4
Parts:
- removed C14: 18pF, resistor:C-EUC0603
- removed GND: UART, con-lsta:FE05-1
- removed SJ3, SJ4: SOLDERJUMPERNO, SparkFun:SOLDERJUMPERNO
- removed SV1, SV2: (no value), con-lsta-RFM69Pi:FE05-2
- removed U$1: MICRO-USB-RECEPTACLE47589-0001, con-molex-usb:MICRO-USB-RECEPTACLE47589-0001
- added C11, C13: 10nF, rcl:C-EUC0603
- added C12, C17: 1uF, resistor:C-EUC0603
- added C19, C20, C21: 100nF, resistor:C-EUC0603
- added C7: 1uF, rcl:C-EUC0805
- added EXPANSION: (no value), con-lstb:MA13-2
- added UART_STM: (no value), con-lstb:MA06-1
- added USB_CONN: MICRO-USB-RECEPTACLE47589-0001, con-molex-usb:MICRO-USB-RECEPTACLE47589-0001
- C15: value 18pF -> 100nF
- C22: value 1uF -> 100nF; device rcl:C-EUC1210 -> resistor:C-EUC0603
- C4: device rcl:C-EUC1210 -> rcl:C-EUC0805
- HSE: value 8MHZ -> 8MHZ ~15pFmax
Connections:
- removed net BIAS_SW1: CT1.1, CT1.4, RB1.2, RB10.2, S1.1
- removed net BIAS_SW2: CT2.1, CT2.4, RB11.2, RB2.2, S2.1
- removed net BIAS_SW3: CT3.1, CT3.4, RB12.2, RB3.2, S3.1
- removed net DS18B20: 3POLE_1.2, R1.1, RJ45_1.4, STM32F303VB.PB13
- removed net PC0: STM32F303VB.PC0, SV2.1
- removed net PC1: STM32F303VB.PC1, SV2.2
- removed net PC2: STM32F303VB.PC2, SV2.3
- removed net PC3: STM32F303VB.PC3, SV2.4
- removed net PE0: STM32F303VB.PE0, SV1.1
- removed net PE1: STM32F303VB.PE1, SV1.2
- removed net PE10: STM32F303VB.PE10, SV1.5
- removed net PE11: STM32F303VB.PE11, SV1.6
- removed net PE12: STM32F303VB.PE12, SV1.7
- removed net PE2: STM32F303VB.PE2, SV1.3
- removed net PE3: STM32F303VB.PE3, SV1.4
- removed net PE7: STM32F303VB.PE7, SV1.8
- removed net PE8: STM32F303VB.PE8, SV1.9
- removed net PE9: STM32F303VB.PE9, SV1.10
- removed net PUSHIN_5: 3POLE_5.2, STM32F303VB.PD2
- removed net PUSHIN_6: 3POLE_6.2, STM32F303VB.PD3
- removed net RXD0: PCB2.GPIO15, SJ12.1, SJ4.1
- removed net TXD0: PCB2.GPIO14, SJ11.1, SJ3.1
- new net CT1_EX: STM32F303VB.PA4
- new net CT2_EX: STM32F303VB.PA5
- new net CT3_EX: STM32F303VB.PA6
- new net CT4_EX: STM32F303VB.PA7
- new net CT5_EX: STM32F303VB.PC4
- new net CT6_EX: STM32F303VB.PC0
- new net CT7_EX: STM32F303VB.PC1
- new net DS18B20_1: R1.1, RJ45_1.4
- new net DS18B20_2: 3POLE_1.2
- new net N$13: EXPANSION.3
- new net N$14: EXPANSION.5
- new net N$15: EXPANSION.7
- new net N$17: EXPANSION.9
- new net N$18: EXPANSION.11
- new net N$19: EXPANSION.13
- new net N$20: EXPANSION.15
- new net N$21: EXPANSION.17
- new net N$23: EXPANSION.19
- new net N$25: EXPANSION.21
- new net N$26: RB18.2, RB9.2, S1.1
- new net N$27: RB17.2, RB8.2, S2.1
- new net N$28: RB16.2, RB7.2, S3.1
- new net N$9: EXPANSION.1
- new net PULSE1: C22.1, RJ45_1.6
- new net PULSE2: 3POLE_5.2, C20.1
- new net PUSHIN_1: 3POLE_6.2, C21.1
- new net PUSHIN_2: 3POLE_2.2, C10.1
- new net VSIG4: STM32F303VB.PC2
- new net VSIG5: STM32F303VB.PC3
- new net VSIG6: STM32F303VB.PF2
- net +3V3: now also C13.1, C17.1, STM32F303VB.VDDA; no longer C22.2, STM32F303VB.VREF+, SV2.10, SV2.9
- net +3V3_ADC: now also C11.1, C12.1, C7.1, STM32F303VB.VREF+; no longer STM32F303VB.VDDA
- net +5V: now also UART_STM.3, USB_CONN.1; no longer GND.3, SV2.6, U$1.1
- net ADC_RJ45IN: now also STM32F303VB.PB15; no longer STM32F303VB.PA3
- net BIAS: now also CT1.1, CT1.4, CT2.1, CT2.4, CT3.1, CT3.4, RB1.2, RB10.2, RB11.2, RB12.2, RB2.2, RB3.2, STM32F303VB.PB12; no longer RB16.2, RB17.2, RB18.2, RB7.2, RB8.2, RB9.2, STM32F303VB.PB0, SV2.5
- net BIAS_IN: now also STM32F303VB.PD11; no longer STM32F303VB.PB1
- net CT1: now also STM32F303VB.PE13; no longer STM32F303VB.PA4
- net CT2: now also STM32F303VB.PE12; no longer STM32F303VB.PA5
- net CT3: now also STM32F303VB.PE11; no longer STM32F303VB.PA6
- net CT4: now also STM32F303VB.PE10; no longer STM32F303VB.PA7
- net CT5: now also STM32F303VB.PE9; no longer STM32F303VB.PC4
- net CT6: now also STM32F303VB.PE8; no longer STM32F303VB.PC5
- net CT7: now also STM32F303VB.PE7; no longer STM32F303VB.PE14
- net CT8: now also STM32F303VB.PB1; no longer STM32F303VB.PE15
- net CT9: now also STM32F303VB.PB0; no longer STM32F303VB.PB12
- net D+: now also STM32F303VB.PA12, USB_CONN.3; no longer U$1.3
- net D-: now also STM32F303VB.PA11, USB_CONN.2; no longer U$1.2
- net GND: now also C10.2, C11.2, C12.2, C13.2, C17.2, C19.2, C20.2, C21.2, C22.2, C7.2, RST.P, UART_STM.1, USB_CONN.5, USB_CONN.GND1, USB_CONN.GND2, USB_CONN.GND3, USB_CONN.GND4; no longer C10.1, C14.2, C22.1, GND.1, RST.S, SV2.7, SV2.8, U$1.5, U$1.GND1, U$1.GND2, U$1.GND3, U$1.GND4
- net HSE_IN: no longer C14.1
- net HSE_OUT: no longer C15.1
- net MBUS_RX: now also PCB2.GPIO23
- net MBUS_TX: now also PCB2.GPIO24
- net N$1: now also UART_STM.2; no longer GND.2
- net N$10: now also CT7.2; no longer CT3.2
- net N$12: now also USB_CONN.4; no longer U$1.4
- net N$2: now also CT9.2; no longer CT1.2
- net N$38: now also CT6.2; no longer CT4.2
- net N$40: now also CT4.2; no longer CT6.2
- net N$42: now also CT3.2; no longer CT7.2
- net N$43: now also CT2.2; no longer CT8.2
- net N$44: now also CT1.2; no longer CT9.2
- net N$8: now also CT8.2; no longer CT2.2
- net NRST: now also RST.S, UART_STM.6; no longer C10.2, RST.P
- net PULSE: no longer 3POLE_2.2, RJ45_1.6, STM32F303VB.PB15
- net PUSHIN_3: now also C15.1; no longer STM32F303VB.PD0
- net PUSHIN_4: now also C19.1; no longer STM32F303VB.PD1
- net SPI3_CS_ESP: now also STM32F303VB.PD3; no longer STM32F303VB.PD5
- net UART_RX: now also STM32F303VB.PD5, UART_STM.4; no longer GND.4, STM32F303VB.PA10
- net UART_TX: now also STM32F303VB.PA3, UART_STM.5; no longer GND.5, STM32F303VB.PA9
- net USART3_RX: now also PCB2.GPIO14, SJ11.1; no longer SJ3.2
- net USART3_TX: now also PCB2.GPIO15, SJ12.1; no longer SJ4.2
Other:
- note added: "BOOT / RFM69 / ESP12"
- note added: "MBUS"
- note added: "STM32F303 OpenEnergyMonitor Concept"
- note added: "VT and CT inputs"
- note added: "Voltage Reference"
- note added: "rPi"
- note removed: "STM32F303xB OpenEnergyMonitor Concept"
- note removed: "VDDA"
- note removed: "VT and CT inputs to base board"
- moved on the sheet: C10, C15, C22, C8, C9, CT1, CT2, CT3, CT4, CT6, CT7, CT8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

Commit message: update v0.4
Parts:
- removed C16: 100nF, resistor:C-EUC0603
- added C14: 1uF, rcl:C-EUC0805
- added C23: 100nF, resistor:C-EUC0603
- added C24: 47uF, rcl:C-EUC0805
- added R8: 4.7k, resistor:R-EU_R0603
- added UART1: (no value), SparkFun:M02PTH
- C3: device rcl:C-EUC1210 -> rcl:C-EUC0805
- UART_STM: device con-lstb:MA06-1 -> con-lstb-db:MA06-1
Connections:
- removed net PULSE: C16.2
- new net UART1_RX: STM32F303VB.PA10, UART1.1
- new net UART1_TX: STM32F303VB.PA9, UART1.2
- net +3V3: now also C14.1, C23.1, C24.1, R8.2
- net DS18B20_1: now also 3POLE_1.2, STM32F303VB.PC6; no longer RJ45_1.4
- net DS18B20_2: now also R8.1, RJ45_1.4; no longer 3POLE_1.2
- net GND: now also C14.2, C23.2, C24.2; no longer C16.1
- net PULSE2: now also STM32F303VB.PA8
- net PUSHIN_1: now also STM32F303VB.PB8
- net PUSHIN_2: now also STM32F303VB.PC7
- net PUSHIN_3: now also STM32F303VB.PC8
- net PUSHIN_4: now also STM32F303VB.PC9
Other:
- note added: "EXPANSION MODULE WIRING PUSH BUTTONS TO STM32 & PI"

Commit message: v0.4 update
Parts:
- added BUTTON1: (no value), switch-omron:31-XX
- renumbered EXPANSION to EXPANSION_MODULE, U$8 to VREF_3V3
Connections:
- net N$18 renamed VT1_EX
- net N$19 renamed VT3_EX
- removed net DS18B20_1: 3POLE_1.2, R1.1, STM32F303VB.PC6
- removed net N$14: EXPANSION_MODULE.5
- removed net N$15: EXPANSION_MODULE.7
- removed net N$17: EXPANSION_MODULE.9
- removed net N$20: EXPANSION_MODULE.15
- removed net N$21: EXPANSION_MODULE.17
- removed net N$23: EXPANSION_MODULE.19
- removed net N$25: EXPANSION_MODULE.21
- removed net N$9: EXPANSION_MODULE.1
- removed net PULSE1: C22.1, RJ45_1.6
- new net BUTTON1: BUTTON1.S, PCB2.GPIO4, STM32F303VB.PB14
- new net DS18B20_RJ45: R1.1, RJ45_1.4, STM32F303VB.PC9
- new net I010_EX: EXPANSION_MODULE.24
- new net I011_EX: EXPANSION_MODULE.25
- new net IO11_EX: STM32F303VB.PB8
- new net IO1_EX: EXPANSION_MODULE.15, STM32F303VB.PE0
- new net IO2_EX: EXPANSION_MODULE.16, STM32F303VB.PE1
- new net IO3_EX: EXPANSION_MODULE.17, STM32F303VB.PE2
- new net IO4_EX: EXPANSION_MODULE.18, STM32F303VB.PE3
- new net IO5_EX: EXPANSION_MODULE.19, STM32F303VB.PE4
- new net IO6_EX: EXPANSION_MODULE.20, STM32F303VB.PE5
- new net IO7_EX: EXPANSION_MODULE.21, STM32F303VB.PE6
- new net IO8_EX: EXPANSION_MODULE.22, STM32F303VB.PB5
- new net PULSE1_RJ45: C22.1, RJ45_1.6, STM32F303VB.PA8
- new net RPI_GPIO16: PCB2.GPIO16, STM32F303VB.PD12
- new net RPI_GPIO20: PCB2.GPIO20, STM32F303VB.PD13
- new net SCK: ESP12.GPIO5, EXPANSION_MODULE.23, PCB2.ID_SC*, STM32F303VB.PB6
- new net SDA: ESP12.GPIO4, PCB2.ID_SD*, STM32F303VB.PB7
- new net VT2_EX: EXPANSION_MODULE.12
- net +3V3: now also EXPANSION_MODULE.4
- net +5V: now also EXPANSION_MODULE.2
- net CT1_EX: now also EXPANSION_MODULE.3
- net CT2_EX: now also EXPANSION_MODULE.6
- net CT3_EX: now also EXPANSION_MODULE.5
- net CT4_EX: now also EXPANSION_MODULE.8
- net CT5_EX: now also EXPANSION_MODULE.7
- net CT6_EX: now also EXPANSION_MODULE.10
- net CT7_EX: now also EXPANSION_MODULE.9
- net DS18B20_2: now also 3POLE_1.2, STM32F303VB.PD14; no longer RJ45_1.4
- net GND: now also BUTTON1.P, EXPANSION_MODULE.1, EXPANSION_MODULE.14, EXPANSION_MODULE.26
- net N$13: now also PCB2.GPIO7; no longer EXPANSION_MODULE.3
- net NRST: now also PCB2.GPIO5
- net PULSE2: now also STM32F303VB.PC8; no longer STM32F303VB.PA8
- net PUSHIN_1: now also STM32F303VB.PB9; no longer STM32F303VB.PB8
- net PUSHIN_2: now also STM32F303VB.PD15; no longer STM32F303VB.PC7
- net PUSHIN_3: now also STM32F303VB.PC6; no longer STM32F303VB.PC8
- net PUSHIN_4: now also STM32F303VB.PC7; no longer STM32F303VB.PC9
- net SPI3_CS: now also PCB2.GPIO8
- net UART1_RX: now also PCB2.GPIO14, SJ11.1
- net UART1_TX: now also PCB2.GPIO15, SJ12.1
- net USART3_RX: no longer PCB2.GPIO14, SJ11.1
- net USART3_TX: no longer PCB2.GPIO15, SJ12.1
Other:
- note removed: "EXPANSION MODULE WIRING PUSH BUTTONS TO STM32 & PI"
- moved on the sheet: C21
