File: Hardware/stm32-pi_full/stm v0.6.brd (EAGLE design)
At the start: 128.9 x 105.8 mm, 149 parts, among them Q1 MMBT3906, Q2 MMBT3904, Q3 MMBT3904, Y1 32.768kHz

Commit message: hardware changes
Parts:
- moved UART1 2.36 mm to (38.2, 52.3)
- moved C18 0.61 mm to (47.8, 59.1)
- moved C17 0.55 mm to (75.7, 62.4)
- renumbered Y1 to LSE
Connections:
- net +5V: no longer PCB2.P$2, PCB2.P$4
- net BUTTON1: no longer PCB2.P$7
- net CS_RFM69: no longer PCB2.P$22
- net GND: no longer PCB2.P$14, PCB2.P$20, PCB2.P$25, PCB2.P$30, PCB2.P$34, PCB2.P$39, PCB2.P$6, PCB2.P$9
- net MBUS_RX: no longer PCB2.P$16
- net MBUS_TX: no longer PCB2.P$18
- net MISO: no longer PCB2.P$21
- net MOSI: no longer PCB2.P$19
- net N$13: no longer PCB2.P$26
- net N$16: no longer PCB2.P$32
- net N$22: no longer PCB2.P$1
- net N$24: no longer PCB2.P$17
- net NRST: no longer PCB2.P$29
- net RPI_GPIO16: no longer PCB2.P$36
- net RPI_GPIO20: no longer PCB2.P$38
- net SCK: no longer PCB2.P$28
- net SDA: no longer PCB2.P$27
- net SPI3_CS: no longer PCB2.P$24
- net SPI_CLK: no longer PCB2.P$23
- net UART1_RX: no longer PCB2.P$8
- net UART1_TX: no longer PCB2.P$10
- net UART_RX: now also STM32F303VB.26; no longer STM32F303VB.86
- net UART_TX: now also STM32F303VB.86; no longer STM32F303VB.26
Routing:
- net UART_TX: track 18.4 -> 80.5 mm, vias 1 -> 7
- net UART_RX: track 41.7 -> 21.4 mm
- net D-: track 123.3 -> 131.4 mm
- net UART1_TX: track 45.5 -> 48.0 mm, vias 3 -> 4
- net +3V3: track 468.3 -> 470.6 mm
- net +3V3_ADC: track 24.4 -> 22.6 mm
- net N$22: track 1.58 -> 0.00 mm
- net N$16: track 3.80 -> 2.33 mm
- net N$13: track 1.47 -> 0.00 mm
- net RPI_GPIO16: track 64.6 -> 63.1 mm
- net N$24: track 1.58 -> 0.14 mm
- net IO1_EX: track 45.2 -> 45.9 mm
- net BIAS_IN: track 8.21 -> 8.74 mm
- net MISO: track 139.6 -> 139.7 mm, vias 7 -> 8
- net SPI3_CS: track 47.9 -> 48.0 mm, vias 1 -> 2
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
Commit message: update v0.6
Parts:
- added LED4: Green 1.85V, adafruit:CHIP-LED0805
- added R10: 220R, rcl:R0603
- LED1: value Red 1.85V -> Green 1.85V
- LED2: value Red 1.85V -> Orange 1.85V
- moved LED1 7.62 mm to (2.67, 96.4)
- moved LED3 7.62 mm to (2.67, 89.0)
- moved R3 7.62 mm to (7.02, 96.4)
- moved R5 7.62 mm to (6.89, 89.0)
- moved RB1 0.24 mm to (19.2, 89.5)
- moved RB10 0.20 mm to (19.3, 89.5)
Connections:
- net LED1 renamed LED1_GREEN
- net LED2 renamed LED2_YELLOW
- net LED3 renamed LED3_RED
- new net N$9: LED4.A, R10.1
- net +3V3: now also R10.2
- net GND: now also LED4.C
Routing:
- net N$9: track 0.00 -> 9.19 mm
- net +3V3: track 470.6 -> 478.2 mm
- net LED3_RED: track 80.2 -> 72.6 mm
- net LED1_GREEN: track 63.7 -> 67.9 mm
- net LED2_YELLOW: track 88.3 -> 85.6 mm
- net N$1: track 10.0 -> 10.9 mm
- net CT4: track 25.9 -> 26.4 mm
- net GND: track 32.2 -> 31.8 mm, vias 176 -> 182
- net NRST: track 217.4 -> 217.7 mm, vias 3 -> 4

Commit message: reorganise files and upload v0.6 brd
Parts:
- removed C24: 47uF, rcl:C0805
- removed ESP12: (no value), ESP8266 MODULES _ CORRECTED:ESP12-SMD
- removed R7: 10k, resistor:R0603
- removed UART1: (no value), SparkFun:1X02
- added C16: 100nF, resistor:C0603
- added D1, D10, D11, D12, D13, D2, D3, D4, D5, D6, D7, D8, D9: ESD5Z3.3T1G, microbuilder:SOD-523
- added Q4: (no value), microbuilder:SOT23-R
- added SJ13, SJ14, SJ15, SJ16, SJ17, SJ18, SJ3, SJ4: SOLDERJUMPERNO, SparkFun:SJ_2S-NO
- added U1: ESP32-WROOM-32D, ESP32-WROOM-32D:MODULE_ESP32-WROOM-32D
- added UART2: (no value), SparkFun:1X02
- C1: value 100nF -> 1uF; device resistor:C0603 -> rcl:C0805
- C23: value 100nF -> (none); device resistor:C0603 -> rcl:153CLV-1010
- R6: value 10k -> (none); device resistor:R0603 -> rcl:R0603
- moved C23 55.8 mm to (88.3, 62.5), turned to 180 degrees
- moved C1 48.6 mm to (77.6, 74.4), turned to 0 degrees
- moved LED4 33.8 mm to (127.9, 34.0), turned to 180 degrees
- moved SJ10 27.7 mm to (30.4, 42.8), turned to 0 degrees
- moved R10 25.3 mm to (125.2, 35.0), turned to 180 degrees
- moved SJ9 24.7 mm to (39.4, 47.5), flipped to the top, turned to 90 degrees
- moved R6 14.6 mm to (70.6, 35.0), turned to 90 degrees
- moved BOOT_ESP 12.6 mm to (64.3, 39.6), turned to 180 degrees
- moved SJ1 5.47 mm to (91.9, 69.9)
- moved VREF_3V3 4.51 mm to (85.0, 52.0)
- moved BOOT_STM 2.00 mm to (82.1, 43.7)
- moved J$1 2.00 mm to (104.2, 4.93)
- moved CF4 1.65 mm to (49.8, 85.5)
- moved CF3 1.42 mm to (36.6, 85.2)
- moved UART_STM 1.00 mm to (88.4, 74.4)
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- renumbered RST to RESET
Connections:
- removed net RST_ESP_1: C1.2, UART_ESP.6
- removed net RST_ESP_2: C1.1, ESP12.RESET
- removed net UART_RX: STM32F303VB.26, UART_STM.4
- removed net UART_RX_ESP: ESP12.TXD0, SJ9.2, UART_ESP.4
- removed net UART_TX: STM32F303VB.86, UART_STM.5
- removed net UART_TX_ESP: ESP12.RXD0, SJ10.1, UART_ESP.5
- new net DIO0: PCB2.P$58, RFM69HCW.2, STM32F303VB.89, U1.24
- new net HSPICS0: SJ13.1, U1.23
- new net HSPID: SJ9.1, U1.16
- new net HSPIQ: SJ4.1, U1.14
- new net HSPI_CLK: SJ10.1, U1.13
- new net N$12: C1.2, UART_STM.6
- new net N$14: C16.1, UART_ESP.6
- new net N$15: C16.2, U1.3
- new net N$17: BOOT_ESP.2, U1.25
- new net RPI_MISO: PCB2.P$61, SJ6.2
- new net RPI_MOSI: PCB2.P$59, SJ5.2
- new net RPI_SPI_CLK: PCB2.P$63, SJ7.2
- new net STM32_CS: SJ14.1, SJ8.2
- new net UART2_RX: STM32F303VB.26, UART2.2
- new net UART2_TX: STM32F303VB.86, UART2.1
- net +3V3: now also Q4.3, R6.1, U1.2; no longer C23.1, C24.1, ESP12.VCC, R6.2
- net BIAS: now also D1.K
- net CS_RFM69: now also PCB2.P$64, SJ13.2; no longer PCB2.P$62
- net D+: now also R6.2
- net GND: now also BOOT_ESP.1, C23.-, D1.A, D10.A, D11.A, D12.A, D13.A, D2.A, D3.A, D4.A, D5.A, D6.A, D7.A, D8.A, D9.A, Q4.1, U1.1, U1.15, U1.38, U1.39; no longer BOOT_ESP.2, C23.2, C24.2, ESP12.GND, R7.2
- net MBUS_TX: now also PCB2.P$52; no longer PCB2.P$58
- net MISO: now also SJ16.2, SJ4.2, SJ6.1; no longer PCB2.P$61, SJ6.2
- net MOSI: now also SJ17.2, SJ5.1, SJ9.2; no longer PCB2.P$59, SJ5.2
- net N$10: now also D7.K
- net N$11: now also SJ18.1, U1.34, UART_ESP.4; no longer ESP12.GPIO2, R6.1
- net N$2: now also D5.K
- net N$38: now also D8.K
- net N$39: now also D9.K
- net N$40: now also D10.K
- net N$42: now also D11.K
- net N$43: now also D12.K
- net N$44: now also D13.K
- net N$7: now also SJ3.1, U1.35, UART_ESP.5; no longer BOOT_ESP.1, ESP12.GPIO0
- net N$8: now also D6.K
- net NRST: now also C1.1, RFM69HCW.6; no longer UART_STM.6
- net SCK: no longer ESP12.GPIO5
- net SDA: no longer ESP12.GPIO4
- net SPI3_CLK: now also SJ15.1; no longer ESP12.GPIO14, SJ7.1
- net SPI3_CS: now also SJ14.2; no longer PCB2.P$64, SJ8.2
- net SPI3_CS_ESP: no longer ESP12.GPIO15, R7.1
- net SPI3_MISO: now also SJ16.1; no longer ESP12.GPIO12, SJ6.1
- net SPI3_MOSI: now also SJ17.1; no longer ESP12.GPIO13, SJ5.1
- net SPI_CLK: now also SJ10.2, SJ15.2, SJ7.1; no longer PCB2.P$63, SJ7.2
- net UART1_RX: now also UART_STM.4; no longer PCB2.P$48, SJ11.1, UART1.1
- net UART1_TX: now also UART_STM.5; no longer PCB2.P$50, SJ12.1, UART1.2
- net USART3_RX: now also PCB2.P$48, SJ11.1, SJ3.2; no longer SJ9.1
- net USART3_TX: now also PCB2.P$50, SJ12.1, SJ18.2; no longer SJ10.2
- net VBAT: now also C23.+, Q4.2
- net VSIG1: now also D2.K
- net VSIG2: now also D3.K
- net VSIG3: now also D4.K
Routing:
- net +3V3: track 478.2 -> 0.00 mm, vias 2 -> 0
- net BIAS: track 355.9 -> 0.00 mm, vias 1 -> 0
- net +5V: track 276.3 -> 0.00 mm
- net NRST: track 217.7 -> 0.00 mm, vias 4 -> 0
- net MISO: track 139.6 -> 0.00 mm, vias 8 -> 0
- net D-: track 131.4 -> 0.00 mm, vias 3 -> 0
- net DS18B20_2: track 122.6 -> 0.00 mm, vias 3 -> 0
- net DS18B20_RJ45: track 122.0 -> 0.00 mm, vias 4 -> 0
- net MOSI: track 111.0 -> 0.00 mm, vias 6 -> 0
- net CS_RFM69: track 110.7 -> 0.00 mm, vias 4 -> 0
- net PULSE2: track 104.5 -> 0.00 mm, vias 1 -> 0
- net PULSE1_RJ45: track 103.5 -> 0.00 mm, vias 1 -> 0
- net ADC_RJ45IN: track 101.2 -> 0.00 mm, vias 2 -> 0
- net SPI_CLK: track 99.4 -> 0.00 mm, vias 4 -> 0
- net D+: track 96.5 -> 0.00 mm, vias 2 -> 0
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Other:
- outline, holes or cut-outs redrawn
- board text added: "MCP1501T"
- board text removed: "5V"
- board text removed: "RX"
- board text removed: "TX"
- board text removed: "VREF 3V3"

Commit message: update v0.5
Parts:
- removed 2POLE_MBUS: OMNIMATE_LSF_2, OMNIMATE_LSF:OMNIMATE_LSF_2
- removed BUTTON1, RESET: (no value), switch-omron:B3F-31XX
- removed C1: 1uF, rcl:C0805
- removed STLINK: (no value), SparkFun:1X03
- removed UART2: (no value), SparkFun:1X02
- removed UART_ESP, UART_STM: (no value), con-lstb-db:MA06-1
- added 3POLE_7: OMNIMATE_LSF_3COMBICON_SMT_3, OMNIMATE_LSF:OMNIMATE_LSF_3_SMT
- added C24, C25, C27: 4.7uF, rcl:C0805
- added C26, C28, C29, C30: 100nF, resistor:C0603
- added C50*: 1uF, rcl:C0603
- added D14, D15, D16, D17, D18, D19, D22, D23, D24, D25, D40*, D41*: ESD5Z3.3T1G, microbuilder:SOD-523
- added JP1: (no value), pinhead+:1X06_SMT
- added JP3: (no value), pinhead+:1X08_SMT
- added S11, S22: SWS001, smd-special:SMS-001
- added SJ19, SJ20, SJ21: SOLDERJUMPERNO, SparkFun:SJ_2S-NO
- added SJ22: (no value), jumper-con_db:SJ-CON
- added TP1: TPB1,27, testpad:B1,27
- added UART1: (no value), SparkFun:1X02
- 3POLE_1, 3POLE_2, 3POLE_3, 3POLE_4, 3POLE_5, 3POLE_6: value OMNIMATE_LSF_3 -> OMNIMATE_LSF_3COMBICON_SMT_3; device OMNIMATE_LSF:OMNIMATE_LSF_3 -> OMNIMATE_LSF:OMNIMATE_LSF_3_SMT
- C18: value 10uF -> 4.7uF
- EXPANSION_MODULE: value (none) -> TSM-113-01-T-DV; device con-lstb:MA13-2 -> pinhead+:2X13_SMT
- R6: value (none) -> 1.5K
- RJ45_1: value RJ45 -> 95501-6889; device SparkFun-Connectors:RJ45-8 -> 95501-6889 rj45 smt:955016889
- S1, S2: value SWS001 -> KSS221GLFS; device smd-special:SMS-001 -> KSS221GLFS:KSS
- moved S1 119.2 mm to (2.16, 82.3), turned to 270 degrees
- moved S2 81.5 mm to (126.7, 13.8), turned to 90 degrees
- moved R8 52.5 mm to (17.5, 71.2), turned to 0 degrees
- moved R1 49.2 mm to (24.0, 24.0), turned to 180 degrees
- moved C18 33.7 mm to (19.4, 76.7), turned to 90 degrees
- moved 3POLE_5 3.76 mm to (7.23, 28.6)
- moved 3POLE_4 3.51 mm to (7.23, 40.0)
- moved 3POLE_6 3.30 mm to (91.4, 7.37)
- moved 3POLE_3 3.25 mm to (7.23, 51.5)
- moved 3POLE_2 3.00 mm to (7.23, 62.8)
- moved 3POLE_1 2.75 mm to (7.23, 74.3)
- moved VREF_3V3 1.80 mm to (85.3, 53.8)
- moved RJ45_1 1.53 mm to (15.5, 6.22)
- moved EXPANSION_MODULE 1.52 mm to (99.3, 52.8)
- moved CF4 1.35 mm to (48.9, 86.5)
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- renumbered S3 to S33
Connections:
- net ANT renamed N$20
- removed net I010_EX: EXPANSION_MODULE.24
- removed net I011_EX: EXPANSION_MODULE.25
- removed net N$29: 2POLE_MBUS.P$1, 2POLE_MBUS.P$2, Q1.2, R17.1
- removed net SCK: EXPANSION_MODULE.23, PCB2.P$68, STM32F303VB.92
- removed net STM32_CS: SJ14.1, SJ8.2
- new net CSESP_STM32: SJ19.1, U1.27
- new net CS_STM32: SJ14.1, SJ19.2, SJ8.2
- new net MBUS_INPUT: 3POLE_7.P$2, Q1.2, R17.1
- new net N$18: D24.A, D25.K
- new net N$19: D40*.A, D41*.K
- new net N$21: R6.1, SJ22.2
- new net N$23: STM32F303VB.69, UART1.1
- new net SCL: EXPANSION_MODULE.22, PCB2.P$68, STM32F303VB.92, U1.36
- net +3V3: now also C24.1, C25.1, C26.1, C29.1, D22.K, D23.K, EXPANSION_MODULE.24, JP1.2, SJ22.1; no longer 3POLE_1.P$2, 3POLE_2.P$2, 3POLE_3.P$2, 3POLE_4.P$2, 3POLE_5.P$2, 3POLE_6.P$2, R6.1, UART_ESP.2
- net +5V: now also C18.1, C27.1, C28.1, C30.1, D24.K, D40*.K, JP1.3, JP3.3; no longer UART_ESP.3, UART_STM.3
- net 24V: now also 3POLE_7.P$3; no longer 2POLE_MBUS.P$3, 2POLE_MBUS.P$4
- net BIAS: now also S11.2, S22.2; no longer S1.2, S2.2
- net BIAS_IN: now also C50*.2; no longer C18.2
- net BUTTON1: now also S1.2; no longer BUTTON1.2
- net DS18B20_2: now also 3POLE_1.P$2, D14.K; no longer 3POLE_1.P$3, 3POLE_1.P$4
- net GND: now also 3POLE_1.P$3, 3POLE_2.P$3, 3POLE_3.P$3, 3POLE_4.P$3, 3POLE_5.P$3, 3POLE_6.P$3, 3POLE_7.P$1, C18.2, C24.2, C25.2, C26.2, C27.2, C28.2, C29.2, C30.2, C50*.1, D14.A, D15.A, D16.A, D17.A, D18.A, D19.A, D22.A, D23.A, D25.A, D41*.A, JP1.1, JP3.1, S1.1, S2.1; no longer 3POLE_1.P$5, 3POLE_1.P$6, 3POLE_2.P$5, 3POLE_2.P$6, 3POLE_3.P$5, 3POLE_3.P$6, 3POLE_4.P$5, 3POLE_4.P$6, 3POLE_5.P$5, 3POLE_5.P$6, 3POLE_6.P$5, 3POLE_6.P$6, BUTTON1.1, C18.1, RESET.1, UART_ESP.1, UART_STM.1
- net IO6_EX: now also EXPANSION_MODULE.21; no longer EXPANSION_MODULE.20
- net IO7_EX: now also EXPANSION_MODULE.23; no longer EXPANSION_MODULE.21
- net IO8_EX: now also EXPANSION_MODULE.25; no longer EXPANSION_MODULE.22
- net N$1: now also JP3.2; no longer UART_STM.2
- net N$11: now also JP1.4, SJ21.2; no longer UART_ESP.4
- net N$12: now also STM32F303VB.68, UART1.2; no longer C1.2, UART_STM.6
- net N$14: now also JP1.6; no longer UART_ESP.6
- net N$26: now also S11.1; no longer S1.1
- net N$27: now also S22.1; no longer S2.1
- net N$7: now also JP1.5, SJ20.2; no longer UART_ESP.5
- net NRST: now also JP3.6, S2.2; no longer C1.1, RESET.2, STLINK.3
- net PULSE2: now also 3POLE_5.P$2, D18.K; no longer 3POLE_5.P$3, 3POLE_5.P$4
- net PUSHIN_1: now also 3POLE_6.P$2, D19.K; no longer 3POLE_6.P$3, 3POLE_6.P$4
- net PUSHIN_2: now also 3POLE_2.P$2, D15.K; no longer 3POLE_2.P$3, 3POLE_2.P$4
- net PUSHIN_3: now also 3POLE_3.P$2, D16.K; no longer 3POLE_3.P$3, 3POLE_3.P$4
- net PUSHIN_4: now also 3POLE_4.P$2, D17.K; no longer 3POLE_4.P$3, 3POLE_4.P$4
- net SDA: now also EXPANSION_MODULE.20, U1.33
- net SWCLK: now also JP3.7; no longer STLINK.2
- net SWDIO: now also JP3.8; no longer STLINK.1
- net UART1_RX: now also PCB2.P$48, SJ11.1, SJ20.1; no longer STM32F303VB.69, UART_STM.4
- net UART1_TX: now also PCB2.P$50, SJ12.1, SJ21.1; no longer STM32F303VB.68, UART_STM.5
- net UART2_RX: now also JP3.4; no longer UART2.2
- net UART2_TX: now also JP3.5, STM32F303VB.25; no longer UART2.1
- net USART3_RX: no longer PCB2.P$48, SJ11.1
- net USART3_TX: no longer PCB2.P$50, SJ12.1
- net VSIG3: now also STM32F303VB.27; no longer STM32F303VB.25
Other:
- outline, holes or cut-outs redrawn

Commit message: commit
Parts:
- removed TP1: TPB1,27, testpad:B1,27
- moved UART1 101.3 mm to (40.6, 53.3), turned to 90 degrees
Changed lines of the file:
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@@
 <?xml version="1.0" encoding="utf-8"?>
 <!DOCTYPE eagle SYSTEM "eagle.dtd">
-<eagle version="9.4.2">
+<eagle version="9.5.0">
 <drawing>
 <settings>
@@
 <layer number="17" name="Pads" color="2" fill="1" visible="yes" active="yes"/>
 <layer number="18" name="Vias" color="2" fill="1" visible="yes" active="yes"/>
-<layer number="19" name="Unrouted" color="6" fill="1" visible="yes" active="yes"/>
+<layer number="19" name="Unrouted" color="6" fill="1" visible="no" active="yes"/>
 <layer number="20" name="Dimension" color="15" fill="1" visible="yes" active="yes"/>
 <layer number="21" name="tPlace" color="7" fill="1" visible="yes" active="yes"/>
@@
 <attribute name="VALUE" x="99.002228125" y="78.48321875" size="0.4064" layer="27" ratio="10" rot="R180"/>
 </element>
-<element name="UART1" library="SparkFun" package="1X02" value="" x="-10.16" y="-34.29" smashed="yes">
-<attribute name="NAME" x="-11.5062" y="-32.4612" size="1.27" layer="25" ratio="10"/>
-<attribute name="VALUE" x="-11.43" y="-37.465" size="1.27" layer="27"/>
-</element>
-<element name="TP1" library="testpad" library_urn="urn:adsk.eagle:library:385" package="B1,27" package3d_urn="urn:adsk.eagle:package:27944/2" value="TPB1,27" x="-11.43" y="-39.37" smashed="yes">
-<attribute name="NAME" x="-12.065" y="-38.354" size="1.27" layer="25" ratio="10"/>
-<attribute name="TP_SIGNAL_NAME" value="" x="-11.43" y="-39.37" size="1.778" layer="27" display="off"/>
-<attribute name="VALUE" x="-12.065" y="-40.132" size="0.0254" layer="27"/>
+<element name="UART1" library="SparkFun" package="1X02" value="" x="40.64" y="53.34" smashed="yes" rot="R90">
+<attribute name="NAME" x="38.8112" y="51.9938" size="1.27" layer="25" ratio="10" rot="R90"/>
+<attribute name="VALUE" x="43.815" y="52.07" size="1.27" layer="27" rot="R90"/>
 </element>
 </elements>
@@
 <contactref element="STM32F303VB" pad="68"/>
 <contactref element="UART1" pad="2"/>
-<wire x1="-7.62" y1="-34.29" x2="55.75049375" y2="53.936425" width="0" layer="19" extent="1-1"/>
+<wire x1="40.64" y1="55.88" x2="55.75049375" y2="53.936425" width="0" layer="19" extent="1-1"/>
 </signal>
 <signal name="N$23">
 <contactref element="STM32F303VB" pad="69"/>
 <contactref element="UART1" pad="1"/>
-<wire x1="-10.16" y1="-34.29" x2="55.75049375" y2="53.436425" width="0" layer="19" extent="1-1"/>
+<wire x1="40.64" y1="53.34" x2="55.75049375" y2="53.436425" width="0" layer="19" extent="1-1"/>
 </signal>
 <signal name="UART2_RX">
