File: Hardware/stm32-pi_full/stm v0.6.sch (EAGLE design)
At the start: 148 parts, among them Q1 MMBT3906, Q2 MMBT3904, Q3 MMBT3904, Y1 32.768kHz

Commit message: hardware changes
Parts:
- renumbered Y1 to LSE
Connections:
- net UART_RX: now also STM32F303VB.PA3; no longer STM32F303VB.PD5
- net UART_TX: now also STM32F303VB.PD5; no longer STM32F303VB.PA3
Changed lines of the file:
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@@
 <part name="CF9" library="resistor" deviceset="C-EU" device="C0603" value="100nF"/>
 <part name="SUPPLY18" library="supply2" library_urn="urn:adsk.eagle:library:372" deviceset="GND" device=""/>
-<part name="Y1" library="microbuilder" deviceset="CRYSTAL" device="8X3.8SMT" value="32.768kHz"/>
+<part name="LSE" library="microbuilder" deviceset="CRYSTAL" device="8X3.8SMT" value="32.768kHz"/>
 <part name="SUPPLY4" library="supply2" library_urn="urn:adsk.eagle:library:372" deviceset="GND" device=""/>
 <part name="SUPPLY19" library="supply2" library_urn="urn:adsk.eagle:library:372" deviceset="GND" device=""/>
@@
 <attribute name="VALUE" x="356.235" y="45.085" size="1.778" layer="96"/>
 </instance>
-<instance part="Y1" gate="G$1" x="53.34" y="15.24" smashed="yes" rot="R270">
+<instance part="LSE" gate="G$1" x="53.34" y="15.24" smashed="yes" rot="R270">
 <attribute name="NAME" x="55.88" y="17.78" size="1.27" layer="95" rot="R270"/>
 <attribute name="VALUE" x="49.53" y="17.78" size="1.27" layer="96" rot="R270"/>
@@
 </segment>
 <segment>
+<pinref part="STM32F303VB" gate="G$1" pin="PA3"/>
+<wire x1="63.5" y1="-2.54" x2="53.34" y2="-2.54" width="0.1524" layer="91"/>
+<label x="45.72" y="-2.54" size="1.778" layer="95"/>
+</segment>
+</net>
+<net name="UART_TX" class="0">
+<segment>
+<label x="0" y="-119.38" size="1.778" layer="95"/>
+<pinref part="UART_STM" gate="1" pin="5"/>
+<wire x1="0" y1="-119.38" x2="-30.48" y2="-119.38" width="0.1524" layer="91"/>
+</segment>
+<segment>
 <pinref part="STM32F303VB" gate="G$1" pin="PD5"/>
 <wire x1="114.3" y1="22.86" x2="127" y2="22.86" width="0.1524" layer="91"/>
 <label x="121.92" y="22.86" size="1.778" layer="95"/>
-</segment>
-</net>
-<net name="UART_TX" class="0">
-<segment>
-<label x="0" y="-119.38" size="1.778" layer="95"/>
-<pinref part="UART_STM" gate="1" pin="5"/>
-<wire x1="0" y1="-119.38" x2="-30.48" y2="-119.38" width="0.1524" layer="91"/>
-</segment>
-<segment>
-<pinref part="STM32F303VB" gate="G$1" pin="PA3"/>
-<wire x1="63.5" y1="-2.54" x2="53.34" y2="-2.54" width="0.1524" layer="91"/>
-<label x="45.72" y="-2.54" size="1.778" layer="95"/>
 </segment>
 </net>
@@
 <pinref part="STM32F303VB" gate="G$1" pin="PC14/OSC32_IN"/>
 <label x="53.34" y="20.32" size="1.778" layer="95"/>
-<pinref part="Y1" gate="G$1" pin="1"/>
+<pinref part="LSE" gate="G$1" pin="1"/>
 <wire x1="53.34" y1="20.32" x2="53.34" y2="17.78" width="0.1524" layer="91"/>
 </segment>
@@
 <pinref part="STM32F303VB" gate="G$1" pin="PC15/OSC32_OUT"/>
 <label x="53.34" y="10.16" size="1.778" layer="95"/>
-<pinref part="Y1" gate="G$1" pin="2"/>
+<pinref part="LSE" gate="G$1" pin="2"/>
 <wire x1="53.34" y1="10.16" x2="53.34" y2="12.7" width="0.1524" layer="91"/>
 </segment>

Commit message: update v0.6
Parts:
- added LED4: Green 1.85V, adafruit:LEDCHIP-LED0805
- added R10: 220R, rcl:R-EU_R0603
- LED1: value Red 1.85V -> Green 1.85V
- LED2: value Red 1.85V -> Orange 1.85V
Connections:
- net LED1 renamed LED1_GREEN
- net LED2 renamed LED2_YELLOW
- net LED3 renamed LED3_RED
- new net N$9: LED4.A, R10.1
- net +3V3: now also R10.2
- net GND: now also LED4.C
Other:
- note added: "OLED"
Changed lines of the file:
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@@
 <part name="R3" library="rcl" library_urn="urn:adsk.eagle:library:334" deviceset="R-EU_" device="R0603" package3d_urn="urn:adsk.eagle:package:23555/3" value="220R"/>
 <part name="SUPPLY25" library="supply2" library_urn="urn:adsk.eagle:library:372" deviceset="GND" device=""/>
-<part name="LED1" library="adafruit" deviceset="LED" device="CHIP-LED0805" value="Red 1.85V"/>
+<part name="LED1" library="adafruit" deviceset="LED" device="CHIP-LED0805" value="Green 1.85V"/>
 <part name="VT3" library="adafruit" deviceset="2.1MMJACK" device="SMT"/>
 <part name="SJ1" library="SparkFun" deviceset="SOLDERJUMPER" device="NO"/>
@@
 <part name="R4" library="rcl" library_urn="urn:adsk.eagle:library:334" deviceset="R-EU_" device="R0603" package3d_urn="urn:adsk.eagle:package:23555/3" value="220R"/>
 <part name="SUPPLY20" library="supply2" library_urn="urn:adsk.eagle:library:372" deviceset="GND" device=""/>
-<part name="LED2" library="adafruit" deviceset="LED" device="CHIP-LED0805" value="Red 1.85V"/>
+<part name="LED2" library="adafruit" deviceset="LED" device="CHIP-LED0805" value="Orange 1.85V"/>
 <part name="R5" library="rcl" library_urn="urn:adsk.eagle:library:334" deviceset="R-EU_" device="R0603" package3d_urn="urn:adsk.eagle:package:23555/3" value="220R"/>
 <part name="SUPPLY21" library="supply2" library_urn="urn:adsk.eagle:library:372" deviceset="GND" device=""/>
@@
 <part name="SUPPLY35" library="supply2" library_urn="urn:adsk.eagle:library:372" deviceset="GND" device=""/>
 <part name="P+1" library="supply1" library_urn="urn:adsk.eagle:library:371" deviceset="+5V" device=""/>
+<part name="R10" library="rcl" library_urn="urn:adsk.eagle:library:334" deviceset="R-EU_" device="R0603" package3d_urn="urn:adsk.eagle:package:23555/3" value="220R"/>
+<part name="SUPPLY36" library="supply2" library_urn="urn:adsk.eagle:library:372" deviceset="GND" device=""/>
+<part name="LED4" library="adafruit" deviceset="LED" device="CHIP-LED0805" value="Green 1.85V"/>
 </parts>
 <sheets>
@@
 <text x="241.3" y="-99.06" size="3.81" layer="91">MBUS</text>
 <text x="-223.52" y="129.54" size="3.81" layer="91">rPi</text>
+<text x="-53.34" y="-55.88" size="25.4" layer="91">OLED</text>
 </plain>
 <instances>
@@
 <attribute name="VALUE" x="403.86" y="-15.24" size="1.778" layer="96" rot="R90"/>
 </instance>
+<instance part="R10" gate="G$1" x="92.964" y="171.704" smashed="yes" rot="R90">
+<attribute name="NAME" x="96.5454" y="170.434" size="1.778" layer="95" rot="R90"/>
+<attribute name="VALUE" x="91.186" y="167.894" size="1.778" layer="96" rot="R90"/>
+</instance>
+<instance part="SUPPLY36" gate="GND" x="92.964" y="153.924" smashed="yes">
+<attribute name="VALUE" x="91.059" y="150.749" size="1.778" layer="96"/>
+</instance>
+<instance part="LED4" gate="G$1" x="92.964" y="161.544" smashed="yes">
+<attribute name="NAME" x="96.52" y="156.972" size="1.778" layer="95" rot="R90"/>
+<attribute name="VALUE" x="99.441" y="156.972" size="1.778" layer="96" rot="R90"/>
+</instance>
 </instances>
 <busses>
@@
 <pinref part="SUPPLY35" gate="GND" pin="GND"/>
 </segment>
+<segment>
+<pinref part="SUPPLY36" gate="GND" pin="GND"/>
+<pinref part="LED4" gate="G$1" pin="C"/>
+</segment>
 </net>
 <net name="+5V" class="1">
@@
 <pinref part="C9" gate="G$1" pin="2"/>
 <wire x1="29.21" y1="172.72" x2="41.91" y2="172.72" width="0.1524" layer="91"/>
+<wire x1="41.91" y1="172.72" x2="81.28" y2="172.72" width="0.1524" layer="91"/>
+<wire x1="81.28" y1="172.72" x2="81.28" y2="180.34" width="0.1524" layer="91"/>
+<junction x="41.91" y="172.72"/>
+<pinref part="R10" gate="G$1" pin="2"/>
+<wire x1="92.964" y1="176.784" x2="92.964" y2="180.34" width="0.1524" layer="91"/>
+<label x="93.472" y="179.832" size="1.778" layer="95"/>
+<wire x1="81.28" y1="180.34" x2="92.964" y2="180.34" width="0.1524" layer="91"/>
 </segment>
 <segment>
@@
 </segment>
 <segment>
+<wire x1="-30.48" y1="-116.84" x2="-7.62" y2="-116.84" width="0.1524" layer="91"/>
 <pinref part="UART_STM" gate="1" pin="6"/>
-<wire x1="-30.48" y1="-116.84" x2="-22.86" y2="-116.84" width="0.1524" layer="91"/>
-<label x="-25.4" y="-116.84" size="1.778" layer="95"/>
 </segment>
 <segment>
@@
 </segment>
 </net>
-<net name="LED1" class="0">
+<net name="LED1_GREEN" class="0">
 <segment>
 <pinref part="R3" gate="G$1" pin="2"/>
@@
 </segment>
 </net>
-<net name="LED2" class="0">
+<net name="LED2_YELLOW" class="0">
 <segment>
 <pinref part="R4" gate="G$1" pin="2"/>
@@
 </segment>
 </net>
-<net name="LED3" class="0">
+<net name="LED3_RED" class="0">
 <segment>
 <pinref part="R5" gate="G$1" pin="2"/>
@@
 </segment>
 </net>
+<net name="N$9" class="0">
+<segment>
+<pinref part="R10" gate="G$1" pin="1"/>
+<pinref part="LED4" gate="G$1" pin="A"/>
+<wire x1="92.964" y1="166.624" x2="92.964" y2="164.084" width="0.1524" layer="91"/>
+</segment>
+</net>

Commit message: reorganise files and upload v0.6 brd
Parts:
- removed C24: 47uF, rcl:C-EUC0805
- removed ESP12: (no value), ESP8266 MODULES _ CORRECTED:ESP12SMD
- removed R7: 10k, resistor:R-EU_R0603
- removed UART1: (no value), SparkFun:M02PTH
- added C16: 100nF, resistor:C-EUC0603
- added D1, D10, D11, D12, D13, D2, D3, D4, D5, D6, D7, D8, D9: ESD5Z3.3T1G, microbuilder:DIODESOD-523
- added Q4: (no value), microbuilder:MOSFET-P
- added SJ13, SJ14, SJ15, SJ16, SJ17, SJ18, SJ3, SJ4: SOLDERJUMPERNO, SparkFun:SOLDERJUMPERNO
- added U1: ESP32-WROOM-32D, ESP32-WROOM-32D:ESP32-WROOM-32D
- added UART2: (no value), SparkFun:M02PTH
- C1: value 100nF -> 1uF; device resistor:C-EUC0603 -> rcl:C-EUC0805
- C23: value 100nF -> (none); device resistor:C-EUC0603 -> rcl:CPOL-EU153CLV-1010
- R6: value 10k -> (none); device resistor:R-EU_R0603 -> rcl:R-EU_R0603
- renumbered RST to RESET
Connections:
- removed net RST_ESP_1: C1.2, UART_ESP.6
- removed net RST_ESP_2: C1.1, ESP12.RESET
- removed net UART_RX: STM32F303VB.PA3, UART_STM.4
- removed net UART_RX_ESP: ESP12.TX, SJ9.2, UART_ESP.4
- removed net UART_TX: STM32F303VB.PD5, UART_STM.5
- removed net UART_TX_ESP: ESP12.RX, SJ10.1, UART_ESP.5
- new net DIO0: PCB2.GPIO24, RFM69HCW.!IRQ, STM32F303VB.PB3, U1.IO2
- new net HSPICS0: SJ13.1, U1.IO15
- new net HSPID: SJ9.1, U1.IO13
- new net HSPIQ: SJ4.1, U1.IO12
- new net HSPI_CLK: SJ10.1, U1.IO14
- new net N$12: C1.2, UART_STM.6
- new net N$14: C16.1, UART_ESP.6
- new net N$15: C16.2, U1.EN
- new net N$17: BOOT_ESP.2, U1.IO0
- new net RPI_MISO: PCB2.GPIO9, SJ6.2
- new net RPI_MOSI: PCB2.GPIO10, SJ5.2
- new net RPI_SPI_CLK: PCB2.GPIO11, SJ7.2
- new net STM32_CS: SJ14.1, SJ8.2
- new net UART2_RX: STM32F303VB.PA3, UART2.2
- new net UART2_TX: STM32F303VB.PD5, UART2.1
- net +3V3: now also Q4.D, R6.1, U1.3V3; no longer C23.1, C24.1, ESP12.VCC, R6.2
- net BIAS: now also D1.C
- net CS_RFM69: now also PCB2.GPIO8, SJ13.2; no longer PCB2.GPIO25
- net D+: now also R6.2
- net GND: now also BOOT_ESP.1, C23.-, D1.A, D10.A, D11.A, D12.A, D13.A, D2.A, D3.A, D4.A, D5.A, D6.A, D7.A, D8.A, D9.A, Q4.G, U1.GND; no longer BOOT_ESP.2, C23.2, C24.2, ESP12.GND, R7.2
- net MBUS_TX: now also PCB2.GPIO18; no longer PCB2.GPIO24
- net MISO: now also SJ16.2, SJ4.2, SJ6.1; no longer PCB2.GPIO9, SJ6.2
- net MOSI: now also SJ17.2, SJ5.1, SJ9.2; no longer PCB2.GPIO10, SJ5.2
- net N$10: now also D7.C
- net N$11: now also SJ18.1, U1.RXD0, UART_ESP.4; no longer ESP12.GPIO2, R6.1
- net N$2: now also D5.C
- net N$38: now also D8.C
- net N$39: now also D9.C
- net N$40: now also D10.C
- net N$42: now also D11.C
- net N$43: now also D12.C
- net N$44: now also D13.C
- net N$7: now also SJ3.1, U1.TXD0, UART_ESP.5; no longer BOOT_ESP.1, ESP12.GPIO0
- net N$8: now also D6.C
- net NRST: now also C1.1, RFM69HCW.!RES; no longer UART_STM.6
- net SCK: no longer ESP12.GPIO5
- net SDA: no longer ESP12.GPIO4
- net SPI3_CLK: now also SJ15.1; no longer ESP12.GPIO14, SJ7.1
- net SPI3_CS: now also SJ14.2; no longer PCB2.GPIO8, SJ8.2
- net SPI3_CS_ESP: no longer ESP12.GPIO15, R7.1
- net SPI3_MISO: now also SJ16.1; no longer ESP12.GPIO12, SJ6.1
- net SPI3_MOSI: now also SJ17.1; no longer ESP12.GPIO13, SJ5.1
- net SPI_CLK: now also SJ10.2, SJ15.2, SJ7.1; no longer PCB2.GPIO11, SJ7.2
- net UART1_RX: now also UART_STM.4; no longer PCB2.GPIO14, SJ11.1, UART1.1
- net UART1_TX: now also UART_STM.5; no longer PCB2.GPIO15, SJ12.1, UART1.2
- net USART3_RX: now also PCB2.GPIO14, SJ11.1, SJ3.2; no longer SJ9.1
- net USART3_TX: now also PCB2.GPIO15, SJ12.1, SJ18.2; no longer SJ10.2
- net VBAT: now also C23.+, Q4.S
- net VSIG1: now also D2.C
- net VSIG2: now also D3.C
- net VSIG3: now also D4.C
Other:
- note added: "BOOT_STM"
- note added: "ESP32"
- note added: "RFM69CW"
- note removed: "BOOT / RFM69 / ESP12"
- moved on the sheet: BOOT_ESP, C1, C14, C2, R6, SJ1, SJ10, SJ9, STLINK, UART_ESP, UART_STM

Commit message: update v0.5
Parts:
- removed 2POLE_MBUS: OMNIMATE_LSF_2, OMNIMATE_LSF:OMNIMATE_LSF_2
- removed BUTTON1, RESET: (no value), switch-omron:31-XX
- removed C1: 1uF, rcl:C-EUC0805
- removed STLINK: (no value), SparkFun:M03PTH
- removed UART2: (no value), SparkFun:M02PTH
- removed UART_ESP, UART_STM: (no value), con-lstb-db:MA06-1
- added 3POLE_7: OMNIMATE_LSF_3COMBICON_SMT_3, OMNIMATE_LSF:OMNIMATE_LSF_3COMBICON_SMT_3
- added C24, C25, C27: 4.7uF, rcl:C-EUC0805
- added C26, C28, C29, C30: 100nF, resistor:C-EUC0603
- added C50*: 1uF, rcl:C-EUC0603
- added D14, D15, D16, D17, D18, D19, D22, D23, D24, D25, D40*, D41*: ESD5Z3.3T1G, microbuilder:DIODESOD-523
- added JP1: (no value), pinhead+:PINHD-1X61X06_SMT
- added JP3: (no value), pinhead+:PINHD-1X81X08_SMT
- added S11, S22: SWS001, smd-special:SWS001
- added SJ19, SJ20, SJ21: SOLDERJUMPERNO, SparkFun:SOLDERJUMPERNO
- added SJ22: (no value), jumper-con_db:SJ-CONCON
- added TP1: TPB1,27, testpad:TPB1,27
- added UART1: (no value), SparkFun:M02PTH
- 3POLE_1, 3POLE_2, 3POLE_3, 3POLE_4, 3POLE_5, 3POLE_6: value OMNIMATE_LSF_3 -> OMNIMATE_LSF_3COMBICON_SMT_3; device OMNIMATE_LSF:OMNIMATE_LSF_3 -> OMNIMATE_LSF:OMNIMATE_LSF_3COMBICON_SMT_3
- C18: value 10uF -> 4.7uF
- EXPANSION_MODULE: value (none) -> TSM-113-01-T-DV; device con-lstb:MA13-2 -> pinhead+:PINHD-2X13SMT
- R6: value (none) -> 1.5K
- RJ45_1: value RJ45 -> 95501-6889; device SparkFun-Connectors:RJ45-8 -> 95501-6889 rj45 smt:95501-6889
- S1, S2: value SWS001 -> KSS221GLFS; device smd-special:SWS001 -> KSS221GLFS:KSS221GLFS
- renumbered S3 to S33
Connections:
- net ANT renamed N$20
- removed net I010_EX: EXPANSION_MODULE.24
- removed net I011_EX: EXPANSION_MODULE.25
- removed net N$29: 2POLE_MBUS.1, Q1.E, R17.1
- removed net SCK: EXPANSION_MODULE.23, PCB2.ID_SC*, STM32F303VB.PB6
- removed net STM32_CS: SJ14.1, SJ8.2
- new net CSESP_STM32: SJ19.1, U1.IO16
- new net CS_STM32: SJ14.1, SJ19.2, SJ8.2
- new net MBUS_INPUT: 3POLE_7.2, Q1.E, R17.1
- new net N$18: D24.A, D25.C
- new net N$19: D40*.A, D41*.C
- new net N$21: R6.1, SJ22.2
- new net N$23: STM32F303VB.PA10, UART1.1
- new net SCL: EXPANSION_MODULE.22, PCB2.ID_SC*, STM32F303VB.PB6, U1.IO22
- net +3V3: now also C24.1, C25.1, C26.1, C29.1, D22.C, D23.C, EXPANSION_MODULE.24, JP1.2, SJ22.1; no longer R6.1, UART_ESP.2
- net +5V: now also C18.1, C27.1, C28.1, C30.1, D24.C, D40*.C, JP1.3, JP3.3; no longer UART_ESP.3, UART_STM.3
- net 24V: now also 3POLE_7.3; no longer 2POLE_MBUS.2
- net BIAS: now also S11.2, S22.2; no longer S1.2, S2.2
- net BIAS_IN: now also C50*.2; no longer C18.2
- net BUTTON1: now also S1.2; no longer BUTTON1.S
- net DS18B20_2: now also D14.C
- net GND: now also 3POLE_7.1, C18.2, C24.2, C25.2, C26.2, C27.2, C28.2, C29.2, C30.2, C50*.1, D14.A, D15.A, D16.A, D17.A, D18.A, D19.A, D22.A, D23.A, D25.A, D41*.A, JP1.1, JP3.1, S1.1, S2.1; no longer BUTTON1.P, C18.1, RESET.P, UART_ESP.1, UART_STM.1
- net IO6_EX: now also EXPANSION_MODULE.21; no longer EXPANSION_MODULE.20
- net IO7_EX: now also EXPANSION_MODULE.23; no longer EXPANSION_MODULE.21
- net IO8_EX: now also EXPANSION_MODULE.25; no longer EXPANSION_MODULE.22
- net N$1: now also JP3.2; no longer UART_STM.2
- net N$11: now also JP1.4, SJ21.2; no longer UART_ESP.4
- net N$12: now also STM32F303VB.PA9, UART1.2; no longer C1.2, UART_STM.6
- net N$14: now also JP1.6; no longer UART_ESP.6
- net N$26: now also S11.1; no longer S1.1
- net N$27: now also S22.1; no longer S2.1
- net N$7: now also JP1.5, SJ20.2; no longer UART_ESP.5
- net NRST: now also JP3.6, S2.2; no longer C1.1, RESET.S, STLINK.3
- net PULSE2: now also D18.C
- net PUSHIN_1: now also D19.C
- net PUSHIN_2: now also D15.C
- net PUSHIN_3: now also D16.C
- net PUSHIN_4: now also D17.C
- net SDA: now also EXPANSION_MODULE.20, U1.IO21
- net SWCLK: now also JP3.7; no longer STLINK.2
- net SWDIO: now also JP3.8; no longer STLINK.1
- net UART1_RX: now also PCB2.GPIO14, SJ11.1, SJ20.1; no longer STM32F303VB.PA10, UART_STM.4
- net UART1_TX: now also PCB2.GPIO15, SJ12.1, SJ21.1; no longer STM32F303VB.PA9, UART_STM.5
- net UART2_RX: now also JP3.4; no longer UART2.2
- net UART2_TX: now also JP3.5, STM32F303VB.PA2; no longer UART2.1
- net USART3_RX: no longer PCB2.GPIO14, SJ11.1
- net USART3_TX: no longer PCB2.GPIO15, SJ12.1
- net VSIG3: now also STM32F303VB.PF4; no longer STM32F303VB.PA2
Other:
- note removed: "OLED"
- moved on the sheet: C18, SJ1

Commit message: commit
Parts:
- removed TP1: TPB1,27, testpad:TPB1,27
Changed lines of the file:
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@@
 <?xml version="1.0" encoding="utf-8"?>
 <!DOCTYPE eagle SYSTEM "eagle.dtd">
-<eagle version="9.4.2">
+<eagle version="9.5.0">
 <drawing>
 <settings>
@@
 <part name="JP3" library="pinhead+" deviceset="PINHD-1X8" device="1X08_SMT"/>
 <part name="UART1" library="SparkFun" deviceset="M02" device="PTH"/>
-<part name="TP1" library="testpad" library_urn="urn:adsk.eagle:library:385" deviceset="TP" device="B1,27" package3d_urn="urn:adsk.eagle:package:27944/2"/>
 </parts>
 <sheets>
@@
 <attribute name="NAME" x="29.464" y="-14.478" size="1.778" layer="95"/>
 </instance>
-<instance part="TP1" gate="G$1" x="25.4" y="5.08" smashed="yes">
-<attribute name="NAME" x="24.13" y="6.35" size="1.778" layer="95"/>
-<attribute name="TP_SIGNAL_NAME" x="26.67" y="3.81" size="1.778" layer="97"/>
-</instance>
 </instances>
