File: Hardware/stm32-pi_full/stm v0.7.brd (EAGLE design)
At the start: 128.9 x 105.8 mm, 198 parts, among them Q1 MMBT3906, Q2 MMBT3904, Q3 MMBT3904, U1 ESP32-WROOM-32D

Commit message: adc retest
Parts:
- removed 3POLE_4, 3POLE_5: OMNIMATE_LSF_3COMBICON_SMT_3, OMNIMATE_LSF:OMNIMATE_LSF_3_SMT
- removed C19, C20, C22, C29, C30: 100nF, resistor:C0603
- removed D17, D18: ESD5Z3.3T1G, microbuilder:SOD-523
- removed EXPANSION_MODULE: TSM-113-01-T-DV, pinhead+:2X13_SMT
- removed R8: 4.7k, resistor:R0603
- added C40, C41, C42, C45, C46, C47: 100nF, resistor:C0603
- added EXPANSION: TSM-113-01-T-DV, pinhead+:2X13_SMT
- added RJ45_2: 95501-6889, 95501-6889 rj45 smt:955016889
- moved RJ45_1 62.9 mm to (7.62, 68.6), turned to 270 degrees
- moved 3POLE_3 44.8 mm to (14.6, 7.23), turned to 0 degrees
- moved C10 40.7 mm to (16.7, 18.3)
- moved D15 40.6 mm to (16.7, 21.3)
- moved 3POLE_2 39.4 mm to (7.23, 23.5)
- moved 3POLE_1 36.8 mm to (7.23, 37.4)
- moved D14 35.8 mm to (16.8, 33.2)
- moved D16 34.3 mm to (20.4, 16.3), turned to 90 degrees
- moved C15 29.3 mm to (20.8, 18.5), turned to 0 degrees
- moved R1 28.8 mm to (21.9, 52.7), turned to 90 degrees
- moved 3POLE_6 2.54 mm to (94.0, 7.37)
- moved BOOT_ESP 2.54 mm to (66.9, 39.6)
- moved BOOT_STM 2.54 mm to (84.7, 43.7)
- moved C11 2.54 mm to (78.4, 58.8)
- moved C12 2.54 mm to (78.4, 56.7)
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Connections:
- removed net DS18B20_2: 3POLE_1.P$2, D14.K, R8.1, STM32F303VB.61
- removed net PULSE2: 3POLE_5.P$2, C20.1, D18.K, STM32F303VB.65
- removed net PUSHIN_4: 3POLE_4.P$2, C19.1, D17.K, STM32F303VB.64
- new net ADC_2_RJ45IN: RJ45_2.8
- new net DS18B20_2_RJ45: RJ45_2.4
- new net PULSE_2_RJ45: C46.1, RJ45_2.6
- new net PUSHIN_BYANT: 3POLE_6.P$2, C21.1, D19.K, STM32F303VB.96
- net +3V3: now also C40.1, C45.1, EXPANSION.24, EXPANSION.4, RJ45_2.2; no longer 3POLE_4.P$1, 3POLE_5.P$1, C29.1, EXPANSION_MODULE.24, EXPANSION_MODULE.4, R8.2
- net +5V: now also C42.1, C47.1, EXPANSION.2, RJ45_2.7; no longer C30.1, EXPANSION_MODULE.2
- net CT1_EX: now also EXPANSION.3; no longer EXPANSION_MODULE.3
- net CT2_EX: now also EXPANSION.6; no longer EXPANSION_MODULE.6
- net CT3_EX: now also EXPANSION.5; no longer EXPANSION_MODULE.5
- net CT4_EX: now also EXPANSION.8; no longer EXPANSION_MODULE.8
- net CT5_EX: now also EXPANSION.7; no longer EXPANSION_MODULE.7
- net CT6_EX: now also EXPANSION.10; no longer EXPANSION_MODULE.10
- net CT7_EX: now also EXPANSION.9; no longer EXPANSION_MODULE.9
- net GND: now also C40.2, C41.2, C42.2, C45.2, C46.2, C47.2, EXPANSION.1, EXPANSION.14, EXPANSION.26, RJ45_2.1, RJ45_2.3, RJ45_2.5; no longer 3POLE_4.P$3, 3POLE_5.P$3, C19.2, C20.2, C22.2, C29.2, C30.2, D17.A, D18.A, EXPANSION_MODULE.1, EXPANSION_MODULE.14, EXPANSION_MODULE.26
- net IO1_EX: now also EXPANSION.15; no longer EXPANSION_MODULE.15
- net IO2_EX: now also EXPANSION.16; no longer EXPANSION_MODULE.16
- net IO3_EX: now also EXPANSION.17; no longer EXPANSION_MODULE.17
- net IO4_EX: now also EXPANSION.18; no longer EXPANSION_MODULE.18
- net IO5_EX: now also EXPANSION.19; no longer EXPANSION_MODULE.19
- net IO6_EX: now also EXPANSION.21; no longer EXPANSION_MODULE.21
- net IO7_EX: now also EXPANSION.23; no longer EXPANSION_MODULE.23
- net IO8_EX: now also EXPANSION.25; no longer EXPANSION_MODULE.25
- net PULSE1_RJ45: now also C41.1; no longer C22.1
- net PUSHIN_1: now also 3POLE_1.P$2, D14.K, STM32F303VB.63; no longer 3POLE_6.P$2, C21.1, D19.K, STM32F303VB.96
- net PUSHIN_2: now also STM32F303VB.64; no longer STM32F303VB.62
- net PUSHIN_3: now also STM32F303VB.65; no longer STM32F303VB.63
- net SCL: now also EXPANSION.22; no longer EXPANSION_MODULE.22
- net SDA: now also EXPANSION.20; no longer EXPANSION_MODULE.20
- net VT1_EX: now also EXPANSION.11; no longer EXPANSION_MODULE.11
- net VT2_EX: now also EXPANSION.12; no longer EXPANSION_MODULE.12
- net VT3_EX: now also EXPANSION.13; no longer EXPANSION_MODULE.13
Routing:
- net +3V3: track 494.8 -> 352.3 mm, vias 31 -> 28
- net ADC_RJ45IN: track 124.4 -> 0.00 mm, vias 6 -> 0
- net DS18B20_RJ45: track 124.0 -> 0.00 mm, vias 2 -> 0
- net PULSE1_RJ45: track 115.8 -> 0.00 mm, vias 2 -> 0
- net LED1_GREEN: track 114.7 -> 0.00 mm, vias 4 -> 0
- net PULSE2: track 114.5 -> 0.00 mm, vias 6 -> 0
- net PUSHIN_2: track 79.9 -> 0.00 mm, vias 4 -> 0
- net RPI_GPIO20: track 74.7 -> 0.00 mm, vias 4 -> 0
- net LED3_RED: track 74.7 -> 0.00 mm, vias 4 -> 0
- net PUSHIN_1: track 74.5 -> 0.00 mm, vias 2 -> 0
- net PUSHIN_BYANT: track 0.00 -> 74.5 mm, vias 0 -> 2
- net PUSHIN_4: track 66.8 -> 0.00 mm, vias 6 -> 0
- net PUSHIN_3: track 57.5 -> 0.00 mm, vias 4 -> 0
- net DS18B20_2: track 55.3 -> 0.00 mm, vias 2 -> 0
- net MBUS_RX: track 79.2 -> 66.9 mm
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Other:
- board size 128.9 x 105.8 mm -> 131.4 x 105.8 mm
- board text added: "131.445 x 105.791 y"
- board text removed: "128.905 x 105.791 y"
- board text removed: "CLMP_4"
- board text removed: "CLMP_5"
