File: Hardware/stm32-pi_full/stm v0.7.sch (EAGLE design)
At the start: 197 parts, among them Q1 MMBT3906, Q2 MMBT3904, Q3 MMBT3904, U1 ESP32-WROOM-32D

Commit message: adc retest
Parts:
- removed 3POLE_4, 3POLE_5: OMNIMATE_LSF_3COMBICON_SMT_3, OMNIMATE_LSF:OMNIMATE_LSF_3COMBICON_SMT_3
- removed C19, C20, C22, C29, C30: 100nF, resistor:C-EUC0603
- removed D17, D18: ESD5Z3.3T1G, microbuilder:DIODESOD-523
- removed EXPANSION_MODULE: TSM-113-01-T-DV, pinhead+:PINHD-2X13SMT
- removed R8: 4.7k, resistor:R-EU_R0603
- added C40, C41, C42, C45, C46, C47: 100nF, resistor:C-EUC0603
- added EXPANSION: TSM-113-01-T-DV, pinhead+:PINHD-2X13SMT
- added RJ45_2: 95501-6889, 95501-6889 rj45 smt:95501-6889
Connections:
- removed net DS18B20_2: 3POLE_1.2, D14.C, R8.1, STM32F303VB.PD14
- removed net PULSE2: 3POLE_5.2, C20.1, D18.C, STM32F303VB.PC8
- removed net PUSHIN_4: 3POLE_4.2, C19.1, D17.C, STM32F303VB.PC7
- new net ADC_2_RJ45IN: RJ45_2.8
- new net DS18B20_2_RJ45: RJ45_2.4
- new net PULSE_2_RJ45: C46.1, RJ45_2.6
- new net PUSHIN_BYANT: 3POLE_6.2, C21.1, D19.C, STM32F303VB.PB9
- net +3V3: now also C40.1, C45.1, EXPANSION.24, EXPANSION.4, RJ45_2.2; no longer 3POLE_4.1, 3POLE_5.1, C29.1, EXPANSION_MODULE.24, EXPANSION_MODULE.4, R8.2
- net +5V: now also C42.1, C47.1, EXPANSION.2, RJ45_2.7; no longer C30.1, EXPANSION_MODULE.2
- net CT1_EX: now also EXPANSION.3; no longer EXPANSION_MODULE.3
- net CT2_EX: now also EXPANSION.6; no longer EXPANSION_MODULE.6
- net CT3_EX: now also EXPANSION.5; no longer EXPANSION_MODULE.5
- net CT4_EX: now also EXPANSION.8; no longer EXPANSION_MODULE.8
- net CT5_EX: now also EXPANSION.7; no longer EXPANSION_MODULE.7
- net CT6_EX: now also EXPANSION.10; no longer EXPANSION_MODULE.10
- net CT7_EX: now also EXPANSION.9; no longer EXPANSION_MODULE.9
- net GND: now also C40.2, C41.2, C42.2, C45.2, C46.2, C47.2, EXPANSION.1, EXPANSION.14, EXPANSION.26, RJ45_2.1, RJ45_2.3, RJ45_2.5; no longer 3POLE_4.3, 3POLE_5.3, C19.2, C20.2, C22.2, C29.2, C30.2, D17.A, D18.A, EXPANSION_MODULE.1, EXPANSION_MODULE.14, EXPANSION_MODULE.26
- net IO1_EX: now also EXPANSION.15; no longer EXPANSION_MODULE.15
- net IO2_EX: now also EXPANSION.16; no longer EXPANSION_MODULE.16
- net IO3_EX: now also EXPANSION.17; no longer EXPANSION_MODULE.17
- net IO4_EX: now also EXPANSION.18; no longer EXPANSION_MODULE.18
- net IO5_EX: now also EXPANSION.19; no longer EXPANSION_MODULE.19
- net IO6_EX: now also EXPANSION.21; no longer EXPANSION_MODULE.21
- net IO7_EX: now also EXPANSION.23; no longer EXPANSION_MODULE.23
- net IO8_EX: now also EXPANSION.25; no longer EXPANSION_MODULE.25
- net PULSE1_RJ45: now also C41.1; no longer C22.1
- net PUSHIN_1: now also 3POLE_1.2, D14.C, STM32F303VB.PC6; no longer 3POLE_6.2, C21.1, D19.C, STM32F303VB.PB9
- net PUSHIN_2: now also STM32F303VB.PC7; no longer STM32F303VB.PD15
- net PUSHIN_3: now also STM32F303VB.PC8; no longer STM32F303VB.PC6
- net SCL: now also EXPANSION.22; no longer EXPANSION_MODULE.22
- net SDA: now also EXPANSION.20; no longer EXPANSION_MODULE.20
- net VT1_EX: now also EXPANSION.11; no longer EXPANSION_MODULE.11
- net VT2_EX: now also EXPANSION.12; no longer EXPANSION_MODULE.12
- net VT3_EX: now also EXPANSION.13; no longer EXPANSION_MODULE.13
Other:
- moved on the sheet: BOOT_ESP, C14, C16, C18, C2, C24, C25, C26, C27, C28, JP1, Q1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
