File: Hardware/stm32-pi_full/stm32 v0.8.brd (EAGLE design)
At the start: 131.4 x 105.8 mm, 252 parts, among them IC1 MCP23017T-E_SO, J1 SOLDERJUMPERNO, Q1 MMBT3906, Q2 MMBT3904, Q3 MMBT3904, U1 ESP32-WROOM-32D

Commit message: minor commit
Parts:
- added Q10, Q8, Q9: (no value), adafruit:SOT23
Connections:
- net N$20 renamed SDA_
- net N$21 renamed SCL_
- new net GPB3: IC1.4, Q8.1
- new net GPB4: IC1.5, Q9.1
- new net GPB5: IC1.6, Q10.1
- net AC1: now also Q8.3
- net AC2: now also Q9.3
- net AC3: now also Q10.3
- net VSIG1: now also Q8.2
- net VSIG2: now also Q9.2
- net VSIG3: now also Q10.2
Changed lines of the file:
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@@
 </element>
 <element name="R16" library="rcl" library_urn="urn:adsk.eagle:library:334" package="R0603" package3d_urn="urn:adsk.eagle:package:23555/3" value="82R" x="91.4" y="29.1" smashed="yes" rot="R180">
-<attribute name="NAME" x="92.158459375" y="27.8046" size="0.9906" layer="25" ratio="10" rot="R180"/>
+<attribute name="NAME" x="91.396459375" y="27.6776" size="0.9906" layer="25" ratio="10" rot="R180"/>
 <attribute name="POPULARITY" value="70" x="91.4" y="29.1" size="1.778" layer="27" rot="R180" display="off"/>
 <attribute name="SPICEPREFIX" value="R" x="91.4" y="29.1" size="1.778" layer="27" rot="R180" display="off"/>
@@
 <attribute name="VALUE" x="-41.275" y="-121.285" size="1.27" layer="27"/>
 </element>
+<element name="Q8" library="adafruit" library_urn="urn:adsk.eagle:library:420" package="SOT23" package3d_urn="urn:adsk.eagle:package:6240836/1" value="" x="-39.37" y="-130.81" smashed="yes">
+<attribute name="MPN" value="FDV303N" x="-39.37" y="-124.46" size="1.778" layer="27" display="off"/>
+<attribute name="NAME" x="-41.275" y="-128.905" size="1.27" layer="25"/>
+<attribute name="VALUE" x="-41.275" y="-133.985" size="1.27" layer="27"/>
+</element>
+<element name="Q9" library="adafruit" library_urn="urn:adsk.eagle:library:420" package="SOT23" package3d_urn="urn:adsk.eagle:package:6240836/1" value="" x="-39.37" y="-137.16" smashed="yes">
+<attribute name="MPN" value="FDV303N" x="-39.37" y="-130.81" size="1.778" layer="27" display="off"/>
+<attribute name="NAME" x="-41.275" y="-135.255" size="1.27" layer="25"/>
+<attribute name="VALUE" x="-41.275" y="-140.335" size="1.27" layer="27"/>
+</element>
+<element name="Q10" library="adafruit" library_urn="urn:adsk.eagle:library:420" package="SOT23" package3d_urn="urn:adsk.eagle:package:6240836/1" value="" x="-39.37" y="-124.46" smashed="yes">
+<attribute name="MPN" value="FDV303N" x="-39.37" y="-137.16" size="1.778" layer="27" display="off"/>
+<attribute name="NAME" x="-41.275" y="-122.555" size="1.27" layer="25"/>
+<attribute name="VALUE" x="-41.275" y="-127.635" size="1.27" layer="27"/>
+</element>
 </elements>
 <signals>
@@
 <wire x1="120.036690625" y1="69.318640625" x2="116.390890625" y2="72.33026875" width="0.4064" layer="1"/>
 <wire x1="116.390890625" y1="72.33026875" x2="115.990890625" y2="74.471971875" width="0.4064" layer="1"/>
+<contactref element="Q10" pad="3"/>
+<wire x1="-39.37" y1="-123.36" x2="120.036690625" y2="69.318640625" width="0" layer="19" extent="1-1"/>
 </signal>
 <signal name="VSIG1" class="4">
@@
 <wire x1="109.726459375" y1="44.372003125" x2="110.379725" y2="43.7187375" width="0.3048" layer="1"/>
 <wire x1="110.379725" y1="43.7187375" x2="110.379725" y2="43.143825" width="0.3048" layer="1"/>
+<contactref element="Q8" pad="2"/>
+<wire x1="70.5" y1="64.15" x2="-38.42" y2="-131.91" width="0" layer="19" extent="1-1"/>
 </signal>
 <signal name="CT1" class="4">
@@
 <wire x1="120.12466875" y1="55.4" x2="120.036690625" y2="55.394921875" width="0.4064" layer="1"/>
 <wire x1="120.12466875" y1="55.4" x2="123.8" y2="55.4" width="0.4064" layer="1"/>
+<contactref element="Q9" pad="3"/>
+<wire x1="-39.37" y1="-136.06" x2="120.036690625" y2="55.394921875" width="0" layer="19" extent="1-1"/>
 </signal>
 <signal name="AC1">
@@
 <wire x1="120.036690625" y1="41.4729" x2="116.390890625" y2="44.62795625" width="0.4064" layer="1"/>
 <wire x1="116.390890625" y1="44.62795625" x2="115.990890625" y2="46.5963625" width="0.4064" layer="1"/>
+<contactref element="Q8" pad="3"/>
+<wire x1="116.390890625" y1="44.62795625" x2="-39.37" y2="-129.71" width="0" layer="19" extent="1-1"/>
 </signal>
 <signal name="VSIG2" class="4">
@@
 <wire x1="112.565525" y1="52.51344375" x2="112.969125" y2="52.51344375" width="0.3048" layer="1"/>
 <wire x1="112.969125" y1="52.51344375" x2="113.9630625" y2="51.51950625" width="0.3048" layer="1"/>
+<contactref element="Q9" pad="2"/>
+<wire x1="70" y1="64.15" x2="-38.42" y2="-138.26" width="0" layer="19" extent="1-1"/>
 </signal>
 <signal name="VSIG3" class="4">
@@
 <wire x1="114.690890625" y1="72.33026875" x2="114.364984375" y2="72.02625625" width="0.254" layer="1"/>
 <contactref element="D30" pad="K"/>
+<contactref element="Q10" pad="2"/>
 <wire x1="112.846134375" y1="66.59191875" x2="114.212953125" y2="65.543084375" width="0" layer="19" extent="1-1"/>
+<wire x1="-38.42" y1="-125.56" x2="69.5" y2="64.15" width="0" layer="19" extent="1-1"/>
 </signal>
 <signal name="N$38">
@@
 <wire x1="26.78001875" y1="25.78606875" x2="26.78111875" y2="25.78716875" width="0.3048" layer="16"/>
 </signal>
-<signal name="N$20">
+<signal name="SDA_">
 <contactref element="SJ26" pad="2"/>
 <contactref element="PCB2" pad="P$43"/>
 <wire x1="33.056609375" y1="42.7028125" x2="31.7299125" y2="73.177296875" width="0" layer="19" extent="1-1"/>
 </signal>
-<signal name="N$21">
+<signal name="SCL_">
 <contactref element="PCB2" pad="P$45"/>
 <contactref element="SJ27" pad="1"/>
@@
 <contactref element="IC1" pad="1"/>
 <contactref element="Q5" pad="1"/>
-<wire x1="67.564" y1="84.05" x2="-40.32" y2="-37.93" width="0" layer="19" extent="1-1"/>
+<wire x1="-40.32" y1="-37.93" x2="67.564" y2="84.05" width="0" layer="19" extent="1-16"/>
 </signal>
 <signal name="GPB1">
 <contactref element="IC1" pad="2"/>
 <contactref element="Q6" pad="1"/>
-<wire x1="68.834" y1="84.05" x2="-40.32" y2="-44.28" width="0" layer="19" extent="1-1"/>
+<wire x1="-40.32" y1="-44.28" x2="68.834" y2="84.05" width="0" layer="19" extent="1-16"/>
 </signal>
 <signal name="GPB2">
 <contactref element="IC1" pad="3"/>
 <contactref element="Q7" pad="1"/>
-<wire x1="70.104" y1="84.05" x2="-40.32" y2="-119.21" width="0" layer="19" extent="1-1"/>
+<wire x1="70.104" y1="84.05" x2="-40.32" y2="-119.21" width="0" layer="19" extent="1-16"/>
+</signal>
+<signal name="GPB3">
+<contactref element="IC1" pad="4"/>
+<contactref element="Q8" pad="1"/>
+<wire x1="71.374" y1="84.05" x2="-40.32" y2="-131.91" width="0" layer="19" extent="1-16"/>
+</signal>
+<signal name="GPB4">
+<contactref element="IC1" pad="5"/>
+<contactref element="Q9" pad="1"/>
+<wire x1="72.644" y1="84.05" x2="-40.32" y2="-138.26" width="0" layer="19" extent="1-16"/>
+</signal>
+<signal name="GPB5">
+<contactref element="IC1" pad="6"/>
+<contactref element="Q10" pad="1"/>
+<wire x1="73.914" y1="84.05" x2="-40.32" y2="-125.56" width="0" layer="19" extent="1-16"/>
 </signal>
 </signals>
