File: Hardware/stm32-pi_full/stm32 v0.8.sch (EAGLE design)
At the start: 218 parts, among them J1 SOLDERJUMPERNO, Q1 MMBT3906, Q2 MMBT3904, Q3 MMBT3904, U1 ESP32-WROOM-32D

Commit message: update
Parts:
- added JP2, JP3: JUMPER-SMT_3_1-NC_TRACE_NO-SILK, SparkFun-Jumpers:JUMPER-SMT_3_1-NC_TRACE_NO-SILK
- R43: value 120k -> 120k 0.1%
- R53: value 10k -> 10k 0.1%
- RB9, RB9_: value 22r -> 22r 0.1%
- RF9, RV1: value 330R -> 330R 0.1%
- S1: value KSS221GLFS -> (none); device KSS221GLFS:KSS221GLFS -> switch-omron:31-XX
- renumbered RB10 to RB9_, RB11 to RB8_, RB12 to RB7_, RB13 to RB4_, RB14 to RB5_, RB15 to RB6_, RB16 to RB3_, RB17 to RB2_, RB18 to RB1_
Connections:
- removed net CT1_EX: EXPANSION.3, STM32F303VE.PA4
- removed net CT2_EX: EXPANSION.6, STM32F303VE.PA5
- removed net CT3_EX: EXPANSION.5, STM32F303VE.PA6
- removed net CT4_EX: EXPANSION.8, STM32F303VE.PA7
- removed net CT5_EX: EXPANSION.7, STM32F303VE.PC4
- removed net CT6_EX: EXPANSION.10, STM32F303VE.PC0
- removed net CT7_EX: EXPANSION.9, STM32F303VE.PC1
- new net CT_EX1: EXPANSION.3, STM32F303VE.PA0
- new net CT_EX2: EXPANSION.6, STM32F303VE.PA1
- new net CT_EX3: EXPANSION.5, STM32F303VE.PC0
- new net CT_EX4: EXPANSION.8, STM32F303VE.PC1
- new net CT_EX5: EXPANSION.7, STM32F303VE.PC2
- new net CT_EX6: EXPANSION.10, STM32F303VE.PC3
- new net PUSHIN_1_PRE: C1.1, D17.C, JP2.3, STM32F303VE.PC6
- new net PUSHIN_2_PRE: C19.1, D18.C, JP3.3, STM32F303VE.PC7
- net ADC_2_RJ45IN: now also STM32F303VE.PD14
- net BIAS: now also RB7.2, RB8.2, RB9.2; no longer RB1.2, RB2.2, RB3.2
- net BUTTON1: now also S1.S; no longer S1.2
- net CT1: now also CF9.2, STM32F303VE.PB0; no longer CF1.2, STM32F303VE.PE13
- net CT2: now also CF8.2, STM32F303VE.PB1; no longer CF2.2, STM32F303VE.PE12
- net CT3: now also CF7.2, STM32F303VE.PE7; no longer CF3.2, STM32F303VE.PE11
- net CT4: now also CF6.2, STM32F303VE.PE8; no longer CF4.2, STM32F303VE.PE10
- net CT6: now also CF4.2, STM32F303VE.PE10; no longer CF6.2, STM32F303VE.PE8
- net CT7: now also CF3.2, STM32F303VE.PE11; no longer CF7.2, STM32F303VE.PE7
- net CT8: now also CF2.2, STM32F303VE.PE12; no longer CF8.2, STM32F303VE.PB1
- net CT9: now also CF1.2, STM32F303VE.PE13; no longer CF9.2, STM32F303VE.PB0
- net GND: now also EXPANSION.9, S1.P; no longer S1.1
- net N$10: now also RB7.1, RF7.1; no longer RB3.1, RF3.1
- net N$2: now also RB9.1, RF9.1; no longer RB1.1, RF1.1
- net N$26: now also RB1.2; no longer RB9.2
- net N$27: now also RB2.2; no longer RB8.2
- net N$28: now also RB3.2; no longer RB7.2
- net N$38: now also RB6.1, RF6.1; no longer RB4.1, RF4.1
- net N$40: now also RB4.1, RF4.1; no longer RB6.1, RF6.1
- net N$42: now also RB3.1, RF3.1; no longer RB7.1, RF7.1
- net N$43: now also RB2.1, RF2.1; no longer RB8.1, RF8.1
- net N$44: now also RB1.1, RF1.1; no longer RB9.1, RF9.1
- net N$8: now also RB8.1, RF8.1; no longer RB2.1, RF2.1
- net PULSE_2_RJ45: now also STM32F303VE.PF6
- net PUSHIN_1: now also JP2.2; no longer C1.1, D17.C, STM32F303VE.PC6
- net PUSHIN_2: now also JP3.2; no longer C19.1, D18.C, STM32F303VE.PC7
- net SCL: now also JP2.1
- net SDA: now also JP3.1
- net UART2_TX: no longer STM32F303VE.PD5
- net VSIG1: now also STM32F303VE.PA4; no longer STM32F303VE.PA0
- net VSIG2: now also STM32F303VE.PA5; no longer STM32F303VE.PA1
- net VSIG3: now also STM32F303VE.PA6; no longer STM32F303VE.PF4
- net VSIG4: now also STM32F303VE.PA7; no longer STM32F303VE.PC2
- net VSIG5: now also STM32F303VE.PC4; no longer STM32F303VE.PC3
- net VSIG6: now also STM32F303VE.PC5; no longer STM32F303VE.PF2
Other:
- note added: "BATTERY/RTC"
- note added: "RFM69"
- note removed: "BATTERY_BACKUP"
- note removed: "RFM69CW"
- moved on the sheet: G1, Q4, R8, RB1, RB2, RB3, RB4, RB6, RB7, RB8, RB9, RF1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

Commit message: commit
Parts:
- removed R6: 1.5k, rcl:R-EU_R0603
- removed RV1: 330R 0.1%, resistor:R-EU_R0603
- removed RV2, RV3: 330R, resistor:R-EU_R0603
- removed TP5, TP6: TPB1,27, testpad:TPB1,27
- added C33: 47uF, rcl:C-EUC0805
- added IC1: AD8603UJ, analog-devices:AD8603UJ
- added SJ22, SJ34, SJ35, SJ36, SJ37: SOLDERJUMPERNO, SparkFun:SOLDERJUMPERNO
- added SVT1, SVT2, SVT3: SWS001, smd-special:SWS001
- C12, C21: value 2.2uF -> 47uF
- CF1, CF2, CF3, CF4, CF5, CF6, CF7, CF8, CF9, CV1, CV2, CV3: value 100nF -> 10nF
- R21: value 200k -> 0R
- R43: value 120k 0.1% -> 120k
- R53: value 10k 0.1% -> 10k
- RB1, RB2, RB3, RB4, RB5, RB6, RB7, RB8, RB9: device rcl:R-EU_R1206 -> rcl:R-EU_R1210
- RF1, RF2, RF3, RF4, RF5, RF6, RF7, RF8: value 330R -> 9k1 0.1%
- RF9: value 330R 0.1% -> 9k1 0.1%
Connections:
- net SPI3_CS renamed SPI1_NSS
- removed net ADC0: R41.2, R51.1, RV3.1
- removed net D+: R6.2, STM32F303VE.PA12, TP5.TP, USB-C.D1+
- removed net D-: STM32F303VE.PA11, TP6.TP, USB-C.D1-
- removed net DIO0: PCB2.GPIO24, RFM69HCW.!IRQ, STM32F303VE.PB3, U1.IO2
- removed net IO11_EX: STM32F303VE.PB8
- removed net IO8_EX: STM32F303VE.PB5
- removed net N$34: R42.1, R52.1, RV2.1
- removed net N$37: R43.1, R53.1, RV1.1
- removed net SPI3_CLK: SJ15.1, STM32F303VE.PC10
- removed net SPI3_MISO: SJ16.1, STM32F303VE.PC11
- removed net SPI3_MOSI: SJ17.1, STM32F303VE.PC12
- new net DIO0_RFM: PCB2.GPIO24, RFM69HCW.!IRQ, STM32F303VE.PD7, U1.IO2
- new net N$18: STM32F303VE.PC12
- new net SPI1_CLK: SJ15.1, STM32F303VE.PB3
- new net SPI1_MISO: SJ16.1, STM32F303VE.PB4
- new net SPI1_MOSI: SJ17.1, STM32F303VE.PB5
- new net UART4_RX: SJ3.2, STM32F303VE.PC11
- new net UART4_TX: SJ18.2, STM32F303VE.PC10
- new net VREF+_: IC1.IN-, IC1.OUT, JP1.3, SJ2.2, STM32F303VE.VREF+
- net +3V3: now also C33.1; no longer R6.1
- net +5V: now also IC1.+VS
- net AC1: now also SJ37.2, SVT1.2
- net AC2: now also SJ36.2, SVT2.2
- net AC3: now also SJ35.2, SVT3.2
- net GND: now also C33.2, IC1.-VS
- net IO1_EX: no longer STM32F303VE.PE0
- net MBUS_RX: now also SJ34.2
- net MBUS_TX: now also SJ22.2
- net PUSHIN_BYANT: now also STM32F303VE.PE0; no longer STM32F303VE.PB9
- net USART3_RX: now also SJ22.1, STM32F303VE.PB8; no longer SJ3.2, STM32F303VE.PB11
- net USART3_TX: now also SJ34.1, STM32F303VE.PB9; no longer SJ18.2, STM32F303VE.PB10
- net VREF+: now also IC1.IN+; no longer JP1.3, SJ2.2, STM32F303VE.VREF+
- net VSIG1: now also R43.1, R53.1, SJ37.1, SVT1.1; no longer RV1.2
- net VSIG2: now also R42.1, R52.1, SJ36.1, SVT2.1; no longer RV2.2
- net VSIG3: now also R41.2, R51.1, SJ35.1, SVT3.1; no longer RV3.2

Commit message: rPi_RFM additions
Parts:
- removed IC1: AD8603UJ, analog-devices:AD8603UJ
- removed VREF_3V3: MCP1501T-33E, MCP1501T-33E:MCP1501T-33E
- added D14, D15, D16, D19, D20, D24, D25, D27, D28, D29, D30, D31, D32: ESD5Z3.3T1G, microbuilder:DIODESOD-523
- added PS1: LT1461AIS8-3.3#PBF, LT1461AIS8:LT1461AIS8-3.3#PBF
- added R6: 0R, resistor:R-EU_R0603
- added U$7: 47219-2001_MICROSD, MOLEX 47219-2001:47219-2001_MICROSD
- C23: value 200pF* -> 2.2uF; device rcl:C-EUC0603 -> rcl:C-EUC0805
Connections:
- removed net CS_STM32_RPI: PCB2.GPIO12, SJ8.1
- removed net RST_RFM_RPI: PCB2.GPIO5, SJ28.2
- removed net SCL_RPI: PCB2.ID_SC*, SJ27.1
- removed net SDA_RPI: PCB2.ID_SD*, SJ26.2
- removed net SPI1_CLK: SJ15.1, STM32F303VE.PB3
- removed net SPI1_MISO: SJ16.1, STM32F303VE.PB4
- removed net SPI1_MOSI: SJ17.1, STM32F303VE.PB5
- removed net VREF+_: IC1.IN-, IC1.OUT, JP1.3, SJ2.2, STM32F303VE.VREF+
- new net BIAS_: R6.2, STM32F303VE.PB12
- new net N$11: PCB2.GPIO8, SJ8.1
- new net N$19: SJ8.2
- new net N$20: PCB2.GPIO2, SJ26.2
- new net N$21: PCB2.GPIO3, SJ27.1
- new net N$7: STM32F303VE.PD6
- new net SD_CLK: SJ17.1, U$7.CLK
- new net SD_CS: SJ15.2, STM32F303VE.PD2
- new net SD_CS_: SJ15.1, U$7.CD/DAT3
- new net SD_MISO: SJ28.1, U$7.DAT0
- new net SD_MOSI: SJ16.1, U$7.CMD
- net +3V3: now also D1.C, D15.C, D16.C, D19.C, D20.C, D24.C, D25.C, D27.C, D28.C, D29.C, D30.A, D31.A, D32.A, SJ2.2, U$7.VDD; no longer SJ2.1
- net +5V: now also PS1.VIN; no longer IC1.+VS, VREF_3V3.SHT_DN, VREF_3V3.VDD
- net BIAS: now also D1.A, D14.C, R6.1; no longer D1.C, STM32F303VE.PB12
- net CS_RFM69: now also STM32F303VE.PD5; no longer PCB2.GPIO8
- net CS_STM32: no longer SJ14.1, SJ8.2
- net GND: now also D14.A, PS1.GND, U$7.GND, U$7.VSS; no longer D1.A, IC1.-VS, VREF_3V3.GND
- net MISO: now also SJ28.2, STM32F303VE.PB4; no longer SJ16.2
- net MOSI: now also SJ16.2, STM32F303VE.PB5; no longer SJ17.2
- net N$10: now also D19.A
- net N$13: now also SJ14.1
- net N$2: now also D15.A
- net N$38: now also D24.A
- net N$39: now also D20.A
- net N$40: now also D25.A
- net N$42: now also D27.A
- net N$43: now also D28.A
- net N$44: now also D29.A
- net N$8: now also D16.A
- net RST_RFM: now also STM32F303VE.PD4; no longer SJ28.1
- net SPI_CLK: now also SJ17.2, STM32F303VE.PB3; no longer SJ15.2
- net VREF+: now also JP1.3, PS1.VOUT, SJ2.1, STM32F303VE.VREF+; no longer IC1.IN+, VREF_3V3.OUT
- net VSIG1: now also D32.C
- net VSIG2: now also D31.C
- net VSIG3: now also D30.C
Other:
- note added: "i2c pullups"
- moved on the sheet: C23, D1, R13, R20

Commit message: commit
RFM69
PULSE input
started on bringing in ds18b20 code from dBC's work.
Parts:
- removed SJ29, SJ30: SOLDERJUMPERNO, SparkFun:SOLDERJUMPERNO
- added IC1: MCP23017T-E_SO, MCP23017T-E_SO:MCP23017T-E_SO
- added Q5, Q6, Q7: (no value), adafruit:MOSFET-NREFLOW
- added R12, R24: 0R, rcl:R-EU_R0603
- added RB10: 22r 0.1%, rcl:R-EU_R1210
- added RB11, RB12, RB13, RB14, RB15, RB16, RB17, RB18: 22r, rcl:R-EU_R1210
Connections:
- removed net N$42: CT3.2, D11.C, D27.A, RB3.1, RB3_.1, RF3.1
- removed net N$43: CT2.2, D12.C, D28.A, RB2.1, RB2_.1, RF2.1
- removed net N$44: CT1.2, D13.C, D29.A, RB1.1, RB1_.1, RF1.1
- new net CT_IN1: CT1.2, D13.C, D29.A, Q5.D, RB1.1, RB1_.1, RF1.1
- new net CT_IN2: CT2.2, D12.C, D28.A, Q6.D, RB2.1, RB2_.1, RF2.1
- new net CT_IN3: CT3.2, D11.C, D27.A, Q7.D, RB3.1, RB3_.1, RF3.1
- new net GPB0: IC1.GPB0, Q5.G
- new net GPB1: IC1.GPB1, Q6.G
- new net GPB2: IC1.GPB2, Q7.G
- new net MOS0: Q5.S, RB18.2
- new net MOS1: Q6.S, RB17.2
- new net MOS2: Q7.S, RB16.2
- new net N$37: RB15.2
- new net N$45: RB10.2
- new net N$46: RB11.2
- new net N$47: RB14.2
- new net N$48: RB13.2
- new net N$49: RB12.2
- net +3V3: now also IC1.VDD
- net BIAS: now also RB10.1, RB11.1, RB12.1, RB13.1, RB14.1, RB15.1, RB16.1, RB17.1, RB18.1
- net GND: now also IC1.A0, IC1.A2_1, IC1.A2_2, IC1.VSS
- net NRST_STM: now also IC1.!RESET
- net RPI_GPIO16: now also R12.2; no longer SJ29.2
- net RPI_GPIO16_RPI: now also R12.1; no longer SJ29.1
- net RPI_GPIO20: now also R24.2; no longer SJ30.2
- net RPI_GPIO20_RPI: now also R24.1; no longer SJ30.1
- net SCL: now also IC1.SCK
- net SDA: now also IC1.SDA

Commit message: minor commit
Parts:
- added Q10, Q8, Q9: (no value), adafruit:MOSFET-NREFLOW
Connections:
- net N$20 renamed SDA_
- net N$21 renamed SCL_
- new net GPB3: IC1.GPB3, Q8.G
- new net GPB4: IC1.GPB4, Q9.G
- new net GPB5: IC1.GPB5, Q10.G
- net AC1: now also Q8.D
- net AC2: now also Q9.D
- net AC3: now also Q10.D
- net VSIG1: now also Q8.S
- net VSIG2: now also Q9.S
- net VSIG3: now also Q10.S
Changed lines of the file:
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@@
 </part>
 <part name="SUPPLY30" library="supply2" deviceset="GND" device=""/>
+<part name="Q8" library="adafruit" library_urn="urn:adsk.eagle:library:420" deviceset="MOSFET-N" device="REFLOW" package3d_urn="urn:adsk.eagle:package:6240836/1">
+<attribute name="MPN" value="FDV303N"/>
+</part>
+<part name="Q9" library="adafruit" library_urn="urn:adsk.eagle:library:420" deviceset="MOSFET-N" device="REFLOW" package3d_urn="urn:adsk.eagle:package:6240836/1">
+<attribute name="MPN" value="FDV303N"/>
+</part>
+<part name="Q10" library="adafruit" library_urn="urn:adsk.eagle:library:420" deviceset="MOSFET-N" device="REFLOW" package3d_urn="urn:adsk.eagle:package:6240836/1">
+<attribute name="MPN" value="FDV303N"/>
+</part>
 </parts>
 <sheets>
@@
 <attribute name="VALUE" x="414.655" y="-128.905" size="1.778" layer="96"/>
 </instance>
+<instance part="Q8" gate="G$1" x="327.66" y="-99.06" smashed="yes">
+<attribute name="NAME" x="332.74" y="-98.425" size="1.27" layer="95"/>
+<attribute name="VALUE" x="332.74" y="-100.33" size="1.27" layer="96"/>
+<attribute name="MPN" x="327.66" y="-99.06" size="1.778" layer="96" display="off"/>
+</instance>
+<instance part="Q9" gate="G$1" x="340.36" y="-99.06" smashed="yes">
+<attribute name="NAME" x="345.44" y="-98.425" size="1.27" layer="95"/>
+<attribute name="VALUE" x="345.44" y="-100.33" size="1.27" layer="96"/>
+<attribute name="MPN" x="340.36" y="-99.06" size="1.778" layer="96" display="off"/>
+</instance>
+<instance part="Q10" gate="G$1" x="353.06" y="-99.06" smashed="yes">
+<attribute name="NAME" x="358.14" y="-98.425" size="1.27" layer="95"/>
+<attribute name="VALUE" x="358.14" y="-100.33" size="1.27" layer="96"/>
+<attribute name="MPN" x="317.754" y="-90.424" size="1.778" layer="96"/>
+</instance>
 </instances>
 <busses>
@@
 <junction x="273.05" y="203.2"/>
 </segment>
+<segment>
+<pinref part="Q10" gate="G$1" pin="D"/>
+<wire x1="355.6" y1="-93.98" x2="355.6" y2="-91.44" width="0.1524" layer="91"/>
+<label x="355.6" y="-91.44" size="1.778" layer="95" rot="R180"/>
+</segment>
 </net>
 <net name="VSIG1" class="4">
@@
 <label x="53.34" y="-5.08" size="1.778" layer="95"/>
 </segment>
+<segment>
+<pinref part="Q8" gate="G$1" pin="S"/>
+<wire x1="330.2" y1="-104.14" x2="330.2" y2="-106.68" width="0.1524" layer="91"/>
+<label x="330.2" y="-106.68" size="1.778" layer="95" rot="R180"/>
+</segment>
 </net>
 <net name="CT1" class="4">
@@
 <junction x="295.91" y="203.2"/>
 </segment>
+<segment>
+<pinref part="Q9" gate="G$1" pin="D"/>
+<wire x1="342.9" y1="-93.98" x2="342.9" y2="-91.44" width="0.1524" layer="91"/>
+<label x="342.9" y="-91.44" size="1.778" layer="95" rot="R180"/>
+</segment>
 </net>
 <net name="AC1" class="0">
@@
 <junction x="318.77" y="203.2"/>
 </segment>
+<segment>
+<pinref part="Q8" gate="G$1" pin="D"/>
+<wire x1="330.2" y1="-93.98" x2="330.2" y2="-91.44" width="0.1524" layer="91"/>
+<label x="330.2" y="-91.44" size="1.778" layer="95" rot="R180"/>
+</segment>
 </net>
 <net name="VSIG2" class="4">
@@
 <label x="53.34" y="-7.62" size="1.778" layer="95"/>
 </segment>
+<segment>
+<pinref part="Q9" gate="G$1" pin="S"/>
+<wire x1="342.9" y1="-104.14" x2="342.9" y2="-106.68" width="0.1524" layer="91"/>
+<label x="342.9" y="-106.68" size="1.778" layer="95" rot="R180"/>
+</segment>
 </net>
 <net name="VSIG3" class="4">
@@
 <label x="53.34" y="-10.16" size="1.778" layer="95"/>
 </segment>
+<segment>
+<pinref part="Q10" gate="G$1" pin="S"/>
+<wire x1="355.6" y1="-104.14" x2="355.6" y2="-106.68" width="0.1524" layer="91"/>
+<label x="355.6" y="-106.68" size="1.778" layer="95" rot="R180"/>
+</segment>
 </net>
 <net name="N$38" class="0">
@@
 </segment>
 </net>
-<net name="N$20" class="0">
+<net name="SDA_" class="0">
 <segment>
 <pinref part="SJ26" gate="1" pin="2"/>
@@
 </segment>
 </net>
-<net name="N$21" class="0">
+<net name="SCL_" class="0">
 <segment>
 <pinref part="PCB2" gate="G$1" pin="GPIO3"/>
@@
 </segment>
 </net>
+<net name="GPB3" class="0">
+<segment>
+<pinref part="IC1" gate="G$1" pin="GPB3"/>
+<wire x1="378.46" y1="-96.52" x2="370.84" y2="-96.52" width="0.1524" layer="91"/>
+<label x="370.84" y="-96.52" size="1.778" layer="95"/>
+</segment>
+<segment>
+<pinref part="Q8" gate="G$1" pin="G"/>
+<wire x1="325.12" y1="-101.6" x2="322.58" y2="-101.6" width="0.1524" layer="91"/>
+<wire x1="322.58" y1="-101.6" x2="322.58" y2="-104.14" width="0.1524" layer="91"/>
+<label x="325.12" y="-101.6" size="1.778" layer="95" rot="R90"/>
+</segment>
+</net>
+<net name="GPB4" class="0">
+<segment>
+<pinref part="IC1" gate="G$1" pin="GPB4"/>
+<wire x1="378.46" y1="-99.06" x2="370.84" y2="-99.06" width="0.1524" layer="91"/>
+<label x="370.84" y="-99.06" size="1.778" layer="95"/>
+</segment>
+<segment>
+<pinref part="Q9" gate="G$1" pin="G"/>
+<wire x1="337.82" y1="-101.6" x2="335.28" y2="-101.6" width="0.1524" layer="91"/>
+<wire x1="335.28" y1="-101.6" x2="335.28" y2="-104.14" width="0.1524" layer="91"/>
+<label x="337.82" y="-101.6" size="1.778" layer="95" rot="R90"/>
+</segment>
+</net>
+<net name="GPB5" class="0">
+<segment>
+<pinref part="IC1" gate="G$1" pin="GPB5"/>
+<wire x1="378.46" y1="-101.6" x2="370.84" y2="-101.6" width="0.1524" layer="91"/>
+<label x="370.84" y="-101.6" size="1.778" layer="95"/>
+</segment>
+<segment>
+<pinref part="Q10" gate="G$1" pin="G"/>
+<wire x1="350.52" y1="-101.6" x2="347.98" y2="-101.6" width="0.1524" layer="91"/>
+<wire x1="347.98" y1="-101.6" x2="347.98" y2="-104.14" width="0.1524" layer="91"/>
+<label x="350.52" y="-101.6" size="1.778" layer="95" rot="R90"/>
+</segment>
+</net>

Commit message: working4 to use internal oscillator
just debugging something
Parts:
- removed IC1: MCP23017T-E_SO, MCP23017T-E_SO:MCP23017T-E_SO
- removed Q10, Q6, Q7, Q8, Q9: (no value), adafruit:MOSFET-NREFLOW
- removed SVT1, SVT2, SVT3: SWS001, smd-special:SWS001
- added Q11, Q12, Q13, Q14, Q15, Q16, Q17, Q18, Q19, Q20, Q21: (no value), adafruit:MOSFET-NREFLOW
- added R25, R26, R27: 1k, resistor:R-EU_R0603
Connections:
- removed net GPB0: IC1.GPB0, Q5.G
- removed net GPB1: IC1.GPB1, Q6.G
- removed net GPB2: IC1.GPB2, Q7.G
- removed net GPB3: IC1.GPB3, Q8.G
- removed net GPB4: IC1.GPB4, Q9.G
- removed net GPB5: IC1.GPB5, Q10.G
- new net MOS3: Q19.G, STM32F303VE.PE9
- new net MOS4: Q17.G, STM32F303VE.PE10
- new net MOS5: Q18.G, STM32F303VE.PE11
- new net MOS6: Q5.G, STM32F303VE.PE12
- new net MOS7: Q14.G, STM32F303VE.PE13
- new net MOS8: Q15.G, STM32F303VE.PE14
- new net MOS9: Q16.G, STM32F303VE.PE15
- new net VMOS1: Q11.G, STM32F303VE.PC0
- new net VMOS2: Q12.G, STM32F303VE.PC1
- new net VMOS3: Q13.G, STM32F303VE.PC2
- new net _AC1: CV1.1, Q11.S, R25.1, R43.1, R53.1, SJ37.1
- new net _AC2: CV2.1, Q12.S, R26.1, R42.1, R52.1, SJ36.1
- new net _AC3: Q13.S, R27.1, R41.2, R51.1, SJ35.1
- net +3V3: no longer IC1.VDD
- net AC1: now also Q11.D; no longer Q8.D, SVT1.2
- net AC2: now also Q12.D; no longer Q9.D, SVT2.2
- net AC3: now also Q13.D; no longer Q10.D, SVT3.2
- net CT1: now also STM32F303VE.PC3
- net CT2: now also STM32F303VE.PA4
- net CT3: now also STM32F303VE.PA5; no longer STM32F303VE.PE7
- net CT4: now also STM32F303VE.PA6; no longer STM32F303VE.PE8
- net CT5: now also STM32F303VE.PA7; no longer STM32F303VE.PE9
- net CT6: now also STM32F303VE.PC4; no longer STM32F303VE.PE10
- net CT7: now also STM32F303VE.PC5; no longer STM32F303VE.PE11
- net CT8: now also STM32F303VE.PB2; no longer STM32F303VE.PE12
- net CT9: now also STM32F303VE.PB11; no longer STM32F303VE.PE13
- net CT_EX1: no longer STM32F303VE.PA0
- net CT_EX2: no longer STM32F303VE.PA1
- net CT_EX3: no longer STM32F303VE.PC0
- net CT_EX4: no longer STM32F303VE.PC1
- net CT_EX5: no longer STM32F303VE.PC2
- net CT_EX6: no longer STM32F303VE.PC3
- net CT_IN1: now also Q21.S; no longer Q5.D
- net CT_IN2: now also Q20.S; no longer Q6.D
- net CT_IN3: now also Q19.S; no longer Q7.D
- net GND: no longer IC1.A0, IC1.A2_1, IC1.A2_2, IC1.VSS
- net MOS0: now also Q21.D; no longer Q5.S
- net MOS1: now also Q20.D, Q21.G, STM32F303VE.PE7; no longer Q6.S
- net MOS2: now also Q19.D, Q20.G, STM32F303VE.PE8; no longer Q7.S
- net N$10: now also Q14.S
- net N$2: now also Q16.S
- net N$37: now also Q17.D
- net N$38: now also Q5.S
- net N$39: now also Q18.S
- net N$40: now also Q17.S
- net N$45: now also Q16.D
- net N$46: now also Q15.D
- net N$47: now also Q18.D
- net N$48: now also Q5.D
- net N$49: now also Q14.D
- net N$8: now also Q15.S
- net NRST_STM: no longer IC1.!RESET
- net SCL: no longer IC1.SCK
- net SDA: no longer IC1.SDA
- net VSIG1: now also R25.2, STM32F303VE.PA0; no longer CV1.1, Q8.S, R43.1, R53.1, SJ37.1, STM32F303VE.PA4, SVT1.1
- net VSIG2: now also R26.2, STM32F303VE.PA1; no longer CV2.1, Q9.S, R42.1, R52.1, SJ36.1, STM32F303VE.PA5, SVT2.1
- net VSIG3: now also R27.2, STM32F303VE.PF2; no longer Q10.S, R41.2, R51.1, SJ35.1, STM32F303VE.PA6, SVT3.1
- net VSIG4: no longer STM32F303VE.PA7
- net VSIG5: no longer STM32F303VE.PC4
- net VSIG6: no longer STM32F303VE.PC5
Other:
- moved on the sheet: Q5
