File: Hardware/stm32-pi_full/stm32 v0.8.sch (EAGLE design)
At the start: 255 parts, among them J1 SOLDERJUMPERNO, Q1 MMBT3906, Q2 MMBT3904, Q3 MMBT3904, U1 ESP32-WROOM-32D

Commit message: update, minor board revision
Parts:
- removed RB1__, RB2__, RB3__: 22r, rcl:R-EU_R1210
- removed SJ11, SJ12, SJ15, SJ16, SJ17, SJ18, SJ19, SJ22, SJ24, SJ28, SJ31, SJ33, SJ34, SJ8: SOLDERJUMPERNO, SparkFun:SOLDERJUMPERNO
- removed U$5, U$6: 3.5MM_TERMINAL_BLOCK, 3.5mm terminal block rs pro:3.5MM_TERMINAL_BLOCK
- removed U$9: 3.5MM_TB_X4, 3.5mm terminal block rs pro:3.5MM_TB_X4
- added D21, D33, D34, D35: ESD5Z3.3T1G, microbuilder:DIODESOD-523
- added FB1: (no value), microbuilder:FERRITE
- added GOLD_ORB_SM1: OSHWLOGOLOGO8MM, oshw:OSHWLOGOLOGO8MM
- added JP7, JP8: JUMPER-SMT_3_1-NC_TRACE_SILK, SparkFun-Jumpers:JUMPER-SMT_3_1-NC_TRACE_SILK
- added R28, R29: 10K, rcl:R-EU_R0603
- added RB1Q, RB2Q, RB3Q: 22r, rcl:R-EU_R1210
- added TERM2: 3.5MM_TB_X6, 3.5mm terminal block rs pro:3.5MM_TB_X6
- added TP1, TP11, TP12, TP13, TP14, TP15, TP16, TP2, TP21, TP3: TEST-POINT3, SparkFun-Connectors:TEST-POINT3
- added TP10, TP17, TP18, TP19, TP20, TP5, TP6, TP7, TP9: TEST-POINTPOGO_PTH, SparkFun-Connectors:TEST-POINTPOGO_PTH
- added UART_STM: (no value), con-lstb-db:MA06-1
- C29, C30: value 5nF -> 15pF
- C31, C32: value 2.2uF -> 10pF; device rcl:C-EUC0805 -> rcl:C-EUC0603
- JP2, JP3: value JUMPER-SMT_3_1-NC_TRACE_NO-SILK -> JUMPER-SMT_3_1-NC_TRACE_SILK; device SparkFun-Jumpers:JUMPER-SMT_3_1-NC_TRACE_NO-SILK -> SparkFun-Jumpers:JUMPER-SMT_3_1-NC_TRACE_SILK
- JP4, JP5, JP6: value JUMPER-SMT_2_NC_TRACE_NO-SILK -> (none); device SparkFun-Jumpers:JUMPER-SMT_2_NC_TRACE_NO-SILK -> rcl:R-EU_R0603
- MCP1825: MPN (none) -> MCP1825S-3302E/DB
- PCB2: value TSM-120-01-T-DV -> RPI3YA; MPN (none) -> M20-7872042
- R12, R24: value 0R -> 10K
- RB9, RB9_: value 22r 0.1% -> 100R 0.1%
- RB9Q: value 22r 0.1% -> 22R 0.1%
- SJ10, SJ13, SJ4, SJ9: value SOLDERJUMPERNO -> JUMPER-SMT_2_NO_SILK; device SparkFun:SOLDERJUMPERNO -> SparkFun-Jumpers:JUMPER-SMT_2_NO_SILK
- STM32F303VET6: MPN (none) -> STM32F303VET6
- ST_LINK: value (none) -> 455-1750-1-ND; device SparkFun:M02PTH -> SparkFun-Connectors:CONN_03
- renumbered Q16]_ to Q16_, RB4__ to RB4Q, RB5__ to RB5Q, RB6__ to RB6Q, RB7__ to RB7Q, RB8__ to RB8Q, RB9__ to RB9Q, RJ45_1 to RJ1, RJ45_2 to RJ2, STM32F303VE to STM32F303VET6, U$10 to TERM3, U$4 to TERM1
Connections:
- removed net +3V3_ESP: SJ23.1, U1.3V3
- removed net 24V: R11.2, R17.2, R9.2, U$2.24V, U$6.P$3
- removed net CSESP_STM32: SJ19.1, U1.IO16
- removed net CS_RFM69: RFM69HCW.!SEL, SJ13.2, STM32F303VET6.PD5
- removed net CS_STM32: SJ19.2
- removed net DS18B20_2_RJ45: R7.1, RJ2.4, STM32F303VET6.PD0
- removed net HSPICS0: SJ13.1, U1.IO15
- removed net HSPID: SJ9.1, U1.IO13
- removed net HSPIQ: SJ4.1, U1.IO12
- removed net MBUS_RX: R18.2, SJ11.2, SJ33.2, SJ34.2
- removed net MBUS_RX_RPI: PCB2.GPIO23, SJ33.1
- removed net MBUS_TX: R19.2, SJ12.2, SJ22.2, SJ31.2
- removed net MBUS_TX_RPI: PCB2.GPIO18, SJ31.1
- removed net MISO: RFM69HCW.SDO, SJ28.2, SJ4.2, SJ6.1, STM32F303VET6.PB4
- removed net MOS0: Q11_.D, RB1__.2
- removed net MOSI: RFM69HCW.SDI, SJ16.2, SJ5.1, SJ9.2, STM32F303VET6.PB5
- removed net N$13: PCB2.GPIO7, SJ14.1
- removed net N$19: SJ8.2
- removed net N$22: PCB2.3V3@1
- removed net N$24: PCB2.3V3@17
- removed net PUSHIN_1: JP2.2, TERM1.P$2
- removed net PUSHIN_1_PRE: C1.1, D17.C, JP2.3, STM32F303VET6.PC6
- removed net PUSHIN_2: JP3.2, TERM1.P$6
- removed net PUSHIN_2_PRE: C19.1, D18.C, JP3.3, STM32F303VET6.PC7
- removed net PUSHIN_3: STM32F303VET6.PC8
- removed net PUSHIN_BYANT: C22.1, D26.C, STM32F303VET6.PE0, U$5.P$2
- removed net RST_RFM_ESP: SJ24.1, U1.IO17
- removed net SD_CS: SJ15.2, STM32F303VET6.PD2
- removed net SPI1_NSS: SJ14.2, STM32F303VET6.PA15
- removed net SPI3_CS_ESP: STM32F303VET6.PD3
- removed net SPI_CLK: RFM69HCW.SCK, SJ10.2, SJ17.2, SJ7.1, STM32F303VET6.PB3
- removed net UART4_RX: SJ3.2, STM32F303VET6.PC11
- removed net UART4_TX: SJ18.2, STM32F303VET6.PC10
- removed net VSIG4: EXPANSION.11
- removed net VSIG5: EXPANSION.12
- removed net VSIG6: EXPANSION.13
- removed net _AC3: R27.1, R41.2, R51.1, SJ35.1
- new net +24V: R11.2, R17.2, R9.2, TERM2.P$1, U$2.24V
- new net BUTTON1_STM: SJ3.2, STM32F303VET6.PB14
- new net ESP_PWR: R29.2, STM32F303VET6.PC11
- new net ESP_PWR_PRE: R29.1, SJ23.1, U1.3V3
- new net EXT_TERM1: C1.1, D17.C, STM32F303VET6.PC6, TERM1.P$2
- new net EXT_TERM2: C19.1, D18.C, STM32F303VET6.PC7, TERM1.P$3
- new net EXT_TERM3: C22.1, D26.C, STM32F303VET6.PD6, TERM2.P$4
- new net HSPI_CS0: JP2.3, SJ13.1, U1.IO15
- new net HSPI_ID/MOSI: JP3.3, SJ9.1, U1.IO13
- new net HSPI_Q/MISO: JP7.3, SJ4.1, U1.IO12
- new net N$20: Q11_.D, RB1Q.2
- new net N$21: Q12_.D, RB2Q.2
- new net N$23: Q13_.D, RB3Q.2
- new net RPI_PWR: R28.1, STM32F303VET6.PD15, TP11.1
- new net SPI1_CLK_SLAVE: SJ10.2, SJ7.1, STM32F303VET6.PB3, TP1.1
- new net SPI1_MISO_SLAVE: SJ4.2, SJ6.1, STM32F303VET6.PB4, TP2.1
- new net SPI1_MOSI_SLAVE: SJ5.1, SJ9.2, STM32F303VET6.PB5, TP3.1
- new net SPI1_NSS_SLAVE: SJ13.2, SJ14.2, STM32F303VET6.PA15, TP21.1
- new net SPI4_CLK_MASTER: JP8.1, RFM69HCW.SCK, STM32F303VET6.PE2, TP12.1
- new net SPI4_CS_RFM69_MASTER: RFM69HCW.!SEL, STM32F303VET6.PE4, TP14.1
- new net SPI4_CS_SDCARD_MASTER: JP2.1, STM32F303VET6.PE3, TP13.1
- new net SPI4_MISO_MASTER: JP7.1, RFM69HCW.SDO, STM32F303VET6.PE5, TP15.1
- new net SPI4_MOSI_MASTER: JP3.1, RFM69HCW.SDI, STM32F303VET6.PE6, TP16.1
- new net UART5_RX: SJ20.1, STM32F303VET6.PD2
- new net UART5_TX: SJ21.1, STM32F303VET6.PC12
- net +3V3: now also D21.C, D34.C, TERM1.P$1, TERM2.P$5, UART_STM.2; no longer TERM1.P$3, U$5.P$3
- net +5V: now also FB1.P$2, TERM2.P$6, UART_STM.3; no longer USB-C.VBUS1, USB-C.VBUS2
- net AC1_MOS: no longer CV1.1
- net AC2_MOS: no longer CV2.1
- net AC3_MOS: now also R27.1, R41.2, R51.1, SJ35.1
- net BIAS: now also TP5.1; no longer CT1.4, CT2.4, CT3.4, RB1__.1, RB2__.1, RB3__.1
- net BIAS_IN: now also TP10.1
- net BUTTON1: now also SJ3.1; no longer STM32F303VET6.PB14
- net CT1: now also CF1.2, TP18.1; no longer CF9.2, STM32F303VET6.PB0
- net CT2: now also CF2.2; no longer CF8.2, STM32F303VET6.PB1
- net CT3: now also CF3.2; no longer CF7.2
- net CT4: now also CF4.2; no longer CF6.2
- net CT6: now also CF6.2; no longer CF4.2
- net CT7: now also CF7.2, TP19.1; no longer CF3.2
- net CT8: now also CF8.2; no longer CF2.2
- net CT9: now also CF9.2; no longer CF1.2
- net DIO0_RFM: now also STM32F303VET6.PE1; no longer PCB2.GPIO24, STM32F303VET6.PD7, U1.IO2
- net DS18B20_RJ45: now also R7.1, RJ2.4, STM32F303VET6.PC10, TP9.1; no longer STM32F303VET6.PC9
- net GND: now also D33.A, D35.A, TERM1.P$6, TERM2.P$3, UART_STM.1; no longer TERM1.P$1, TERM1.P$4, TERM1.P$5, U$5.P$1, U$6.P$1
- net HSPI_CLK: now also JP8.3
- net IO2_EX: no longer STM32F303VET6.PE1
- net IO3_EX: no longer STM32F303VET6.PE2
- net IO4_EX: no longer STM32F303VET6.PE3
- net IO5_EX: no longer STM32F303VET6.PE4
- net IO6_EX: no longer STM32F303VET6.PE5
- net IO7_EX: no longer STM32F303VET6.PE6
- net MBUS_I/O: now also TERM2.P$2; no longer U$6.P$2
- net MOS1: now also TP17.1; no longer Q12_.D, RB2__.2
- net MOS2: no longer Q13_.D, RB3__.2
- net N$11: now also SJ14.1; no longer SJ8.1
- net N$18: now also PCB2.3V3@17, R28.2; no longer STM32F303VET6.PC12
- net N$26: now also CT1.4, RB1Q.1
- net N$27: now also CT2.4, RB2Q.1
- net N$28: now also CT3.4, RB3Q.1
- net N$7: now also FB1.P$1, USB-C.VBUS1, USB-C.VBUS2; no longer STM32F303VET6.PD6
- net NRST_STM: now also ST_LINK.3, UART_STM.6
- net PULSE1_RJ45: now also STM32F303VET6.PA12; no longer STM32F303VET6.PA8
- net RST_RFM: now also STM32F303VET6.PE0; no longer SJ24.2, STM32F303VET6.PD4
- net RXD0_ESP: no longer SJ18.1
- net SCL: now also D34.A, D35.C, STM32F303VET6.PC8, TERM1.P$5; no longer JP2.1, STM32F303VET6.PB6
- net SDA: now also D21.A, D33.C, STM32F303VET6.PC9, TERM1.P$4; no longer JP3.1, STM32F303VET6.PB7
- net SD_CLK: now also JP8.2; no longer SJ17.1
- net SD_CS_: now also JP2.2; no longer SJ15.1
- net SD_MISO: now also JP7.2; no longer SJ28.1
- net SD_MOSI: now also JP3.2; no longer SJ16.1
- net TXD0_ESP: no longer SJ3.1
- net UART1_RX: now also UART_STM.4; no longer SJ11.1, SJ20.1
- net UART1_TX: now also UART_STM.5; no longer SJ12.1, SJ21.1
- net USART3_RX: now also R19.2; no longer SJ22.1
- net USART3_TX: now also R18.2; no longer SJ34.1
- net VMOS1: now also TP6.1
- net VREF+: now also TP7.1
- net VSIG1: now also CV1.1, TP20.1
- net VSIG2: now also CV2.1
Other:
- note added: "SD card normally conn'd to ESP32"
- moved on the sheet: C1, C19, C22, CF1, CF2, CF3, CF4, CF6, CF7, CF8, CF9, D17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
