File: Hardware/stm32-pi_full/stm32 v0.9b.sch (EAGLE design)
At the start: 271 parts, among them J1 SOLDERJUMPERNO, J2 5-1814400-1, U1 ESP32-WROOM-32D, Y1 6MM_3.5MM_CRYSTAL

Commit message: bias changed to inverting op-amp with in-the-loop compensator
Parts:
- removed R23: 10k, resistor:R-EU_R0603
- removed TP10: TEST-POINTPOGO_PTH, SparkFun-Connectors:TEST-POINTPOGO_PTH
- added Q4: (no value), microbuilder:TRANSISTOR_NPNWIDE
- added SJ1: (no value), jumper-con_db:SJ-CONCON
- added TP3, TP6: TEST-POINTPOGO_PTH, SparkFun-Connectors:TEST-POINTPOGO_PTH
- added X1: OPAMP, ngspice-simulation:OPAMP
- C20: value 2.2uF -> 2nF
- C50: value (none) -> 1nF
- R22: value 10k -> 1k
- R37: value 0R -> 1k
- R6: value 0R -> 5R
Connections:
- removed net BIAS_: R6.2, STM32F303VE.PB12
- removed net BIAS_IN: C50.2, R22.1, R23.2, STM32F303VE.PD11, TP10.1
- new net OPAMP_FB2: C50.1, Q4.B, R38.1, R6.2, TP3.1
- new net OPAMP_NON-INVERT+: SJ1.1, STM32F303VE.PD11
- new net OPAMP_OUT: C20.2, R6.1, STM32F303VE.PB12, TP5.1, X1.VOUT
- net +3V3ANA: now also Q4.C, R37.1
- net AGND: now also C50.2, R22.1, SJ1.2, X1.P; no longer C50.1, R23.1, R38.2
- net BIAS: now also Q4.E, R22.2; no longer C20.1, R37.1, R6.1, TP5.1
- net LED2: now also STM32F303VE.PD12; no longer STM32F303VE.PD9
- net LED3: now also STM32F303VE.PD13; no longer STM32F303VE.PD10
- net OPAMP_INVERT-: now also C20.1, R38.2, TP6.1, X1.N; no longer C20.2, R38.1
- net VREF+: no longer R22.2
Other:
- note added: "BIAS"
- note removed: "BIAS IN"
- note removed: "BIAS OUT"
- note removed: "FEEDBACK"
- moved on the sheet: C20, C35, C36, C50, D1, D14, R22, R37, R38, R6

Commit message: update readme.md
including link for the enclosure CAD
Parts:
- removed CANBUS: TX/RX, con-lstb-db:MA02-1
- removed R35, R36: 0R, rcl:R-EU_R0603
- added C51: 22uF, rcl:C-EUC0805
- added JP2: JUMPER-SMT_2_NO_NO-SILK, SparkFun-Jumpers:JUMPER-SMT_2_NO_NO-SILK
- added JP20, JP21, JP22, JP23, JP5, JP6, JP7, JP8, JP9: (no value), jumper-con_db:JP1E
- added JP3: JUMPER-SMT_3_NO_NO-SILK, SparkFun-Jumpers:JUMPER-SMT_3_NO_NO-SILK
- added R23: 1k, resistor:R-EU_R0603
- added TP1: TEST-POINTPOGO_PTH, SparkFun-Connectors:TEST-POINTPOGO_PTH
- C20: value 2nF -> 2.2nF
- C31, C32: device rcl:C-EUC0805 -> rcl:C-EUC0603
- C48: value 100nF -> (none)
- C49: value 10pF -> 1nF; device rcl:C-EUC0805 -> rcl:C-EUC0603
- C50: value 1nF -> 1uf
- C7: value 2.2uF -> 22uF
- CF1, CF2, CF3, CF4, CF5, CF6, CF7, CF8, CF9, CV1, CV2, CV3, CV4: value 10nF -> 10nF 5%
- JP1: value JUMPER-SMT_2_NC_TRACE_NO-SILK -> JUMPER-SMT_2_NO_NO-SILK; device SparkFun-Jumpers:JUMPER-SMT_2_NC_TRACE_NO-SILK -> SparkFun-Jumpers:JUMPER-SMT_2_NO_NO-SILK
- PS1: value LT1461AIS8-3.3#PBF -> REF191ESZ; MPN REF196GSZ -> REF191ESZ
- R22: value 1k -> 10k
- R25, R26, R27: value 9k1 -> 9k1 0.1%
- R34: value 0R -> (none); device rcl:R-EU_R0603 -> rcl:R-EU_R1210
- R37: value 1k -> 2k
- R6: value 5R -> 20R
- RB1A, RB1B: value 22r 0.3W 1% -> 22r
- RB1_: value 22r 0.5W -> (none)
- RB2_, RB3_, RB4_, RB5_, RB6_, RB7_, RB8_: value 22r -> (none)
- RB9A, RB9B: value 100R 0.1% -> 22r
- RB9_: value 100R 0.1% -> (none)
- renumbered TERM1 to TB1
Connections:
- removed net IO3_EX: EXPANSION.17
- removed net IO5_EX: EXPANSION.19
- removed net N$28: JP14.1, R36.1, RB3A.2, RB3B.2, RB3_.2
- new net N$12: JP3.2, R37.1
- new net N$24: JP20.2, RB5A.2, RB5B.2, RB5_.2
- new net N$25: JP22.2, RB6A.2, RB6B.2, RB6_.2
- new net N$29: JP21.2, RB8A.2, RB8B.2, RB8_.2
- new net N$34: JP23.2, RB9A.2, RB9B.2, RB9_.2
- new net N$35: JP8.2, RB4A.2, RB4B.2, RB4_.2
- new net N$36: JP9.2, RB7A.2, RB7B.2, RB7_.2
- new net N$37: JP7.2, RB3A.2, RB3B.2, RB3_.2
- new net N$7: C50.1, R23.1
- net +3V3ANA: now also JP3.3, TP1.1; no longer R37.1
- net +5V: now also C51.1
- net AC1: now also R34.1
- net BIAS: now also JP10.1, JP12.1, JP14.1, JP2.2, JP20.1, JP21.1, JP22.1, JP23.1, JP5.1, JP6.1, JP7.1, JP8.1, JP9.1; no longer R35.2, R36.2, RB4A.2, RB4B.2, RB4_.2, RB5A.2, RB5B.2, RB5_.2, RB6A.2, RB6B.2, RB6_.2, RB7A.2, RB7B.2, RB7_.2, RB8A.2, RB8B.2, RB8_.2, RB9A.2, RB9B.2, RB9_.2
- net CAN_RX: now also EXPANSION.17; no longer CANBUS.1
- net CAN_TX: now also EXPANSION.19; no longer CANBUS.2
- net DGND: now also C51.2
- net HSPI_CLK: now also U$7.CLK
- net HSPI_ID/MOSI: now also U$7.CMD
- net HSPI_Q/MISO: now also U$7.DAT0
- net N$26: now also JP5.2; no longer JP10.1, R34.1
- net N$27: now also JP6.2; no longer JP12.1, R35.1
- net OPAMP_FB2: now also JP2.1, R23.2; no longer C50.1
- net SPI1_CLK_SLAVE: no longer U$7.CLK
- net SPI1_MISO_SLAVE: no longer U$7.DAT0
- net SPI1_MOSI_SLAVE: no longer U$7.CMD
- net VREF+: now also JP3.1
Other:
- note added: "GPIO"
- note removed: "check transistor part numbers"
- note removed: "gpio - literally"
- moved on the sheet: C19, C20, C22, C35, C36, C40, C41, C42, C45, C46, C47, C50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
