File: Hardware/stm32-pi_full/stm32 v1.1.brd (EAGLE design)
At the start: 131.4 x 105.8 mm, 289 parts, among them IC2 AD8519KS, J1 JUMPER-SMT_2_NC_TRACE_NO-SILK, Q1 PNP, Q2 NPN, Q3 NPN, U1 ESP32-WROOM-32D

Commit message: commit
Parts:
- removed FB6: (no value), microbuilder:_0603
- removed SJ1: JUMPER-SMT_2_NC_TRACE_NO-SILK, SparkFun-Jumpers:SMT-JUMPER_2_NC_TRACE_NO-SILK
- removed SJ2: JUMPER-SMT_2_NO_SILK, SparkFun-Jumpers:SMT-JUMPER_2_NO_SILK
- added TP12: TEST-POINT3, SparkFun-Connectors:PAD.03X.03
- C11: value 22uF -> 1uF
- moved TP11 6.56 mm to (91.3, 64.8)
- moved C11 5.80 mm to (93.7, 67.0), turned to 90 degrees
- moved TP10 2.08 mm to (91.2, 67.9)
- moved C37 1.93 mm to (92.6, 62.2)
- moved REF19X 1.59 mm to (86.7, 64.8)
Connections:
- removed net +5V_REF: C11.1, C37.1, FB6.1, REF19X.2, REF19X.3, TP11.1
- removed net N$12: REF19X.4, SJ1.2, SJ2.2, TP10.1
- net +3V3ANA: now also C11.1, C37.1, REF19X.2, REF19X.3, TP11.1
- net +5V: no longer FB6.2
- net AGND: now also C11.2, C37.2, REF19X.4, TP10.1; no longer SJ1.1
- net DGND: no longer C11.2, C37.2, SJ2.1
- net VBAT: now also TP12.P$1
Routing:
- net +5V: track 344.6 -> 323.4 mm
- net +3V3ANA: track 57.2 -> 73.2 mm, vias 20 -> 23
- net +5V_REF: track 13.8 -> 0.00 mm
- net N$12: track 4.40 -> 0.00 mm
- net VREF+: track 49.6 -> 53.1 mm
- net OPAMP_OUT: track 19.6 -> 17.4 mm
- net OPAMP_NON-INVERT+: track 19.9 -> 18.4 mm
- net VBAT: track 21.7 -> 22.3 mm
- net AGND: track 16.3 -> 16.6 mm, vias 117 -> 118
- net DGND: vias 104 -> 100
Other:
- board text removed: "TB1"

Commit message: changed lmv824 3-phase feedback resistor values
Parts:
- R39, R40, R41: value 620R -> 330R
Changed lines of the file:
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@@
 <attribute name="VALUE" x="119.919240625" y="73.7925" size="1.27" layer="27" align="center"/>
 </element>
-<element name="R40" library="rcl" library_urn="urn:adsk.eagle:library:334" package="R0603" package3d_urn="urn:adsk.eagle:package:23555/3" value="620R" x="119.807334375" y="65.701946875" smashed="yes">
+<element name="R40" library="rcl" library_urn="urn:adsk.eagle:library:334" package="R0603" package3d_urn="urn:adsk.eagle:package:23555/3" value="330R" x="119.807334375" y="65.701946875" smashed="yes">
 <attribute name="NAME" x="121.49270625" y="65.072025" size="1.016" layer="25"/>
 <attribute name="POPULARITY" value="70" x="119.807334375" y="65.701946875" size="1.778" layer="27" display="off"/>
@@
 <attribute name="VALUE" x="119.172334375" y="63.796946875" size="1.27" layer="27"/>
 </element>
-<element name="R39" library="rcl" library_urn="urn:adsk.eagle:library:334" package="R0603" package3d_urn="urn:adsk.eagle:package:23555/3" value="620R" x="119.8196" y="63.59000625" smashed="yes">
+<element name="R39" library="rcl" library_urn="urn:adsk.eagle:library:334" package="R0603" package3d_urn="urn:adsk.eagle:package:23555/3" value="330R" x="119.8196" y="63.59000625" smashed="yes">
 <attribute name="NAME" x="121.52795" y="62.9581625" size="1.016" layer="25"/>
 <attribute name="POPULARITY" value="70" x="119.8196" y="63.59000625" size="1.778" layer="27" display="off"/>
@@
 <attribute name="VALUE" x="119.1846" y="61.68500625" size="1.27" layer="27"/>
 </element>
-<element name="R41" library="rcl" library_urn="urn:adsk.eagle:library:334" package="R0603" package3d_urn="urn:adsk.eagle:package:23555/3" value="620R" x="119.789375" y="67.807859375" smashed="yes" rot="R180">
+<element name="R41" library="rcl" library_urn="urn:adsk.eagle:library:334" package="R0603" package3d_urn="urn:adsk.eagle:package:23555/3" value="330R" x="119.789375" y="67.807859375" smashed="yes" rot="R180">
 <attribute name="NAME" x="121.569375" y="67.145325" size="1.016" layer="25"/>
 <attribute name="POPULARITY" value="70" x="119.789375" y="67.807859375" size="1.778" layer="27" rot="R180" display="off"/>
