File: Hardware/stm32-pi_full/stm32 v1.1_backup.sch (EAGLE design)
At the start: 264 parts, among them IC1 TS461CLT, J1 JUMPER-SMT_2_NC_TRACE_NO-SILK, Q1 PNP, Q2 NPN, Q3 NPN, U1 ESP32-WROOM-32D, U2 RFM69HCW/RFM95W

Commit message: tidy
Parts:
- removed FB10, FB11, FB6: (no value), microbuilder:FERRITE_0603
- removed IC1: TS461CLT, TS461CLT:TS461CLT
- removed JP3, JP5: JUMPER-SMT_3_1-NC_TRACE_NO-SILK, SparkFun-Jumpers:JUMPER-SMT_3_1-NC_TRACE_NO-SILK
- removed JP6: JUMPER-SMT_2_NC_PASTE_SILK, SparkFun-Jumpers:JUMPER-SMT_2_NC_PASTE_SILK
- removed LMV1, LMV2, LMV3: LMV824IDG4, LMV824IDG4:LMV824IDG4
- removed RB10, RB11, RB12, RB13, RB14, RB15, RB16, RB17, RB18: 510R 0.1%, rcl:R-EU_R0805
- removed RB19, RB20, RB21, RB22, RB23, RB24, RB44, RB55, RB66: 680R | 681R 0.1%, rcl:R-EU_R0805
- removed SJ1: JUMPER-SMT_2_NC_TRACE_NO-SILK, SparkFun-Jumpers:JUMPER-SMT_2_NC_TRACE_NO-SILK
- removed U2: RFM69HCW/RFM95W, microbuilder:RFM69HCW_SMT
- added C36: (no value), rcl:C-EUC0603
- added C50: 1uF, rcl:C-EUC0603
- added C53: 22uF, rcl:C-EUC0805
- added D10, D11, D12, D13, D15, D16, D19, D20, D24, D25, D27, D28, D29, D5, D6, D7, D8, D9: ESD5Z3.3T1G, microbuilder:DIODESOD-523
- added IC2: AD8519KS, analog-devices:AD8519KS
- added JP10, JP11, JP12, JP13, JP14, JP15, JP16, JP17, JP18: JUMPER-SMT_2_NO_NO-SILK_ROUND, SparkFun-Jumpers:JUMPER-SMT_2_NO_NO-SILK_ROUND
- added R23: 1k, resistor:R-EU_R0603
- added R38: 39k, resistor:R-EU_R0603
- added R42, R44, R45, R46, R47, R48, R49, R50, R51: 0R, rcl:R-EU_R0603
- added R54: 10k, resistor:R-EU_R0603
- added RB1B, RB2B, RB3B, RB4B, RB5B, RB6B, RB7B, RB8B, RB9B: (no value), rcl:R-EU_R0805
- C11, C23: value 22uf -> 1uF
- C20: value 22uF -> 2.2nF; device rcl:C-EUC0805 -> rcl:C-EUC0603
- C35: value 22uF -> (none); device rcl:C-EUC0805 -> rcl:C-EUC0603
- FB1: value 1600R -> (none)
- FB2: value 0R -> (none)
- R55: value 10k -> 91k
- R6: value 20R -> 0R; device rcl:R-EU_R0603 -> resistor:R-EU_R0603
- RB1A, RB2A, RB3A, RB4A, RB5A, RB6A, RB7A, RB8A, RB9A: value 6R81 -> 6R8
- renumbered RB1 to RB1A, RB2 to RB2A, RB3 to RB3A, RB4 to RB4A, RB5 to RB5A, RB6 to RB6A, RB7 to RB7A, RB8 to RB8A, RB9 to RB9A
Connections:
- net CT1_ADC renamed CT1
- net CT2_ADC renamed CT2
- net CT3_ADC renamed CT3
- net CT4_ADC renamed CT4
- net CT5_ADC renamed CT5
- net CT6_ADC renamed CT6
- removed net ANT_LORA: JP6.1, U2.ANT
- removed net BIAS123: LMV1.1IN+, LMV1.2IN+, LMV1.3IN+, LMV1.4IN-, LMV1.4OUT, RB19.2, RB20.2, RB21.2
- removed net BIAS456: LMV2.1IN+, LMV2.2IN+, LMV2.3IN+, LMV2.4IN-, LMV2.4OUT, RB44.2, RB55.2, RB66.2
- removed net BIAS789: LMV3.1IN+, LMV3.2IN+, LMV3.3IN+, LMV3.4IN-, LMV3.4OUT, RB22.2, RB23.2, RB24.2
- removed net BIAS_SOT23: IC1.-V, IC1.OUT, JP5.2
- removed net CT1_OUT: LMV1.1OUT, RB10.1, RF1.1
- removed net CT2_OUT: LMV1.2OUT, RB14.1, RF2.1
- removed net CT3_OUT: LMV1.3OUT, RB15.2, RF3.1
- removed net CT4_OUT: LMV2.1OUT, RB11.1, RF4.1
- removed net CT5_OUT: LMV2.2OUT, RB12.1, RF5.1
- removed net CT6_OUT: LMV2.3OUT, RB13.2, RF6.1
- removed net CT7_OUT: LMV3.1OUT, RB16.1, RF7.1
- removed net CT8_OUT: LMV3.2OUT, RB17.1, RF8.1
- removed net CT9_OUT: LMV3.3OUT, RB18.2, RF9.1
- removed net DIO1_RFM: STM32F303VE.PE4, U2.DIO1
- removed net N$12: CT5.3
- removed net N$38: CT4.3
- removed net N$39: C20.1, IC1.+V, JP3.3, TP6.1
- removed net N$40: CT6.1, RB66.1, RB6A.2, RB6_.2
- removed net N$42: JP5.3, R6.1, TP3.1
- removed net N$43: CT9.1, RB24.1, RB9A.2, RB9_.2
- removed net N$45: CT8.1, RB23.1, RB8A.2, RB8_.2
- removed net N$46: CT7.1, RB22.1, RB7A.2, RB7_.2
- removed net STM32_OPAMP_NON-INVERT+: C35.1, JP3.1, STM32F303VE.PD11
- removed net STM32_OPAMP_OUT: JP5.1, STM32F303VE.PB12, TP2.1
- new net OPAMP_NON-INVERT+: C53.1, IC2.IN+, R55.1, R56.2, STM32F303VE.PD11, TP2.1
- net +3V3: now also MCP1825.+3V3; no longer FB10.P$2
- net +3V3ANA: now also C11.1, C37.1, D15.C, D16.C, D19.C, D20.C, D24.C, D25.C, D27.C, D28.C, D29.C, IC2.+VS, MCP1825(ANALOG).+3V3, REF19X.!SHDN, REF19X.VIN, TP11.1; no longer FB11.P$2, FB6.P$2, IC1.VDD, LMV1.VCC+, LMV2.VCC+, LMV3.VCC+
- net AGND: now also C36.2, C50.2, C53.2, D10.A, D11.A, D12.A, D13.A, D5.A, D6.A, D7.A, D8.A, D9.A, IC2.-VS, R54.2; no longer C20.2, IC1.VCC, LMV1.GND/VCC-, LMV2.GND/VCC-, LMV3.GND/VCC-
- net ANT: no longer JP6.2
- net BIAS: now also C35.1, C36.1, CT1.1, CT2.1, CT3.1, CT4.1, CT5.1, CT6.1, CT7.1, CT8.1, CT9.1, JP10.1, JP11.1, JP12.1, JP13.1, JP14.1, JP15.1, JP16.1, JP17.1, JP18.1, R23.2, R38.1, R42.1, R44.1, R45.1, R46.1, R47.1, R48.1, R49.1, R50.1, R51.1, TP3.1; no longer LMV1.4IN+, LMV2.4IN+, LMV3.4IN+, TP5.1
- net CT_IN1: now also D13.C, D29.A, RB1B.1, RF1.1; no longer LMV1.1IN-, RB10.2
- net CT_IN2: now also D12.C, D28.A, RB2B.1, RF2.1; no longer LMV1.2IN-, RB14.2
- net CT_IN3: now also D11.C, D27.A, RB3B.1, RF3.1; no longer LMV1.3IN-, RB15.1
- net CT_IN4: now also D10.C, D25.A, RB4B.1, RF4.1; no longer LMV2.1IN-, RB11.2
- net CT_IN5: now also D20.A, D9.C, RB5B.1, RF5.1; no longer LMV2.2IN-, RB12.2
- net CT_IN6: now also D24.A, D8.C, RB6B.1, RF6.1; no longer LMV2.3IN-, RB13.1
- net CT_IN7: now also D19.A, D7.C, RB7B.1, RF7.1; no longer LMV3.1IN-, RB16.2
- net CT_IN8: now also D16.A, D6.C, RB8B.1, RF8.1; no longer LMV3.2IN-, RB17.2
- net CT_IN9: now also D15.A, D5.C, RB9B.1, RF9.1; no longer LMV3.3IN-, RB18.1
- net DGND: no longer U2.GND@2
- net DIO0_RFM: no longer U2.DIO0
- net N$1: now also JP10.2
- net N$10: now also JP13.2
- net N$13: now also JP14.2
- net N$2: now also JP11.2
- net N$20: now also JP15.2
- net N$21: now also JP16.2
- net N$22: now also JP17.2
- net N$23: now also JP18.2
- net N$24: now also R47.2, RB5A.2, RB5B.2, RB5_.2; no longer CT6.3
- net N$25: now also R46.2, RB6A.2, RB6B.2, RB6_.2; no longer FB10.P$1, MCP1825.+3V3
- net N$26: now also R42.2, RB1B.2; no longer CT1.1, RB19.1
- net N$27: now also R44.2, RB2B.2; no longer CT2.1, RB20.1
- net N$29: now also R50.2, RB8A.2, RB8B.2, RB8_.2; no longer C11.1, C37.1, FB6.P$1, REF19X.!SHDN, REF19X.VIN, TP11.1
- net N$34: now also R51.2, RB9A.2, RB9B.2, RB9_.2; no longer FB11.P$1, MCP1825(ANALOG).+3V3
- net N$35: now also R48.2, RB4B.2; no longer CT4.1, RB44.1
- net N$36: now also R49.2, RB7A.2, RB7B.2, RB7_.2; no longer CT3.1, RB21.1, RB3A.2, RB3_.2
- net N$37: now also R45.2, RB3A.2, RB3B.2, RB3_.2; no longer JP3.2, R55.1, R56.2
- net N$7: now also C50.1, R23.1; no longer CT5.1, RB55.1, RB5A.2, RB5_.2
- net N$8: now also JP12.2
- net OPAMP_INVERT-: now also C20.1, IC2.IN-, R38.2, R54.1, TP6.1; no longer SJ1.1
- net OPAMP_OUT: now also C20.2, IC2.OUT, R6.1, STM32F303VE.PB12, TP5.1; no longer SJ1.2
- net RGND: no longer U2.GND@1, U2.GND@3
- net RST_RFM: no longer U2.RESET
- net SPI4_CLK_MASTER: no longer U2.SCK
- net SPI4_CS_RFM69_MASTER: no longer U2.NSS
- net SPI4_MISO_MASTER: no longer U2.MISO
- net SPI4_MOSI_MASTER: no longer U2.MOSI
- net VDD: no longer U2.VDD
Other:
- note added: "RFM69"
- note added: "maybe DNGA comes off the ana supply with FB in series"
- note removed: "RFMxx"
- note removed: "maybe DNGA comes off the ANA supply with FB in series"
- moved on the sheet: C20, C33, C35, C43, CF1, CF2, CF3, CF4, CF5, CF6, CF7, CF8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
