File: Hardware/stm32-pi_full/stm32 v1.1.sch (EAGLE design)
At the start: 286 parts, among them IC2 AD8519KS, J1 JUMPER-SMT_2_NC_TRACE_NO-SILK, Q1 PNP, Q2 NPN, Q3 NPN, U1 ESP32-WROOM-32D

Commit message: tidy
Parts:
- removed C36: (no value), rcl:C-EUC0603
- removed C50: 1uF, rcl:C-EUC0603
- removed C53: 22uF, rcl:C-EUC0805
- removed D10, D11, D12, D13, D15, D16, D19, D20, D24, D25, D27, D28, D29, D5, D6, D7, D8, D9: ESD5Z3.3T1G, microbuilder:DIODESOD-523
- removed IC2: AD8519KS, analog-devices:AD8519KS
- removed JP10, JP11, JP12, JP13, JP14, JP15, JP16, JP17, JP18: JUMPER-SMT_2_NO_NO-SILK_ROUND, SparkFun-Jumpers:JUMPER-SMT_2_NO_NO-SILK_ROUND
- removed R23: 1k, resistor:R-EU_R0603
- removed R38: 39k, resistor:R-EU_R0603
- removed R42, R44, R45, R46, R47, R48, R49, R50, R51: 0R, rcl:R-EU_R0603
- removed R54: 10k, resistor:R-EU_R0603
- removed RB1B, RB2B, RB3B, RB4B, RB5B, RB6B, RB7B, RB8B, RB9B: (no value), rcl:R-EU_R0805
- added FB10, FB11, FB6: (no value), microbuilder:FERRITE_0603
- added IC1: TS461CLT, TS461CLT:TS461CLT
- added JP3, JP5: JUMPER-SMT_3_1-NC_TRACE_NO-SILK, SparkFun-Jumpers:JUMPER-SMT_3_1-NC_TRACE_NO-SILK
- added JP6: JUMPER-SMT_2_NC_PASTE_SILK, SparkFun-Jumpers:JUMPER-SMT_2_NC_PASTE_SILK
- added LMV1, LMV2, LMV3: LMV824IDG4, LMV824IDG4:LMV824IDG4
- added RB10, RB11, RB12, RB13, RB14, RB15, RB16, RB17, RB18: 510R 0.1%, rcl:R-EU_R0805
- added RB19, RB20, RB21, RB22, RB23, RB24, RB44, RB55, RB66: 680R | 681R 0.1%, rcl:R-EU_R0805
- added SJ1: JUMPER-SMT_2_NC_TRACE_NO-SILK, SparkFun-Jumpers:JUMPER-SMT_2_NC_TRACE_NO-SILK
- added U2: RFM69HCW/RFM95W, microbuilder:RFM69HCW_SMT
- C11, C23: value 1uF -> 22uf
- C20: value 2.2nF -> 22uF; device rcl:C-EUC0603 -> rcl:C-EUC0805
- C35: value (none) -> 22uF; device rcl:C-EUC0603 -> rcl:C-EUC0805
- FB1: value (none) -> 1600R
- FB2: value (none) -> 0R
- R55: value 91k -> 10k
- R6: value 0R -> 20R; device resistor:R-EU_R0603 -> rcl:R-EU_R0603
- RB1, RB2, RB3, RB4, RB5, RB6, RB7, RB8, RB9: value 6R8 -> 6R81
- renumbered RB1A to RB1, RB2A to RB2, RB3A to RB3, RB4A to RB4, RB5A to RB5, RB6A to RB6, RB7A to RB7, RB8A to RB8, RB9A to RB9
Connections:
- net CT1 renamed CT1_ADC
- net CT2 renamed CT2_ADC
- net CT3 renamed CT3_ADC
- net CT4 renamed CT4_ADC
- net CT5 renamed CT5_ADC
- net CT6 renamed CT6_ADC
- removed net OPAMP_NON-INVERT+: C53.1, IC2.IN+, R55.1, R56.2, STM32F303VE.PD11, TP2.1
- new net ANT_LORA: JP6.1, U2.ANT
- new net BIAS123: LMV1.1IN+, LMV1.2IN+, LMV1.3IN+, LMV1.4IN-, LMV1.4OUT, RB19.2, RB20.2, RB21.2
- new net BIAS456: LMV2.1IN+, LMV2.2IN+, LMV2.3IN+, LMV2.4IN-, LMV2.4OUT, RB44.2, RB55.2, RB66.2
- new net BIAS789: LMV3.1IN+, LMV3.2IN+, LMV3.3IN+, LMV3.4IN-, LMV3.4OUT, RB22.2, RB23.2, RB24.2
- new net BIAS_SOT23: IC1.-V, IC1.OUT, JP5.2
- new net CT1_OUT: LMV1.1OUT, RB10.1, RF1.1
- new net CT2_OUT: LMV1.2OUT, RB14.1, RF2.1
- new net CT3_OUT: LMV1.3OUT, RB15.2, RF3.1
- new net CT4_OUT: LMV2.1OUT, RB11.1, RF4.1
- new net CT5_OUT: LMV2.2OUT, RB12.1, RF5.1
- new net CT6_OUT: LMV2.3OUT, RB13.2, RF6.1
- new net CT7_OUT: LMV3.1OUT, RB16.1, RF7.1
- new net CT8_OUT: LMV3.2OUT, RB17.1, RF8.1
- new net CT9_OUT: LMV3.3OUT, RB18.2, RF9.1
- new net DIO1_RFM: STM32F303VE.PE4, U2.DIO1
- new net N$12: CT5.3
- new net N$38: CT4.3
- new net N$39: C20.1, IC1.+V, JP3.3, TP6.1
- new net N$40: CT6.1, RB6.2, RB66.1, RB6_.2
- new net N$42: JP5.3, R6.1, TP3.1
- new net N$43: CT9.1, RB24.1, RB9.2, RB9_.2
- new net N$45: CT8.1, RB23.1, RB8.2, RB8_.2
- new net N$46: CT7.1, RB22.1, RB7.2, RB7_.2
- new net STM32_OPAMP_NON-INVERT+: C35.1, JP3.1, STM32F303VE.PD11
- new net STM32_OPAMP_OUT: JP5.1, STM32F303VE.PB12, TP2.1
- net +3V3: now also FB10.P$2; no longer MCP1825.+3V3
- net +3V3ANA: now also FB11.P$2, FB6.P$2, IC1.VDD, LMV1.VCC+, LMV2.VCC+, LMV3.VCC+; no longer C11.1, C37.1, D15.C, D16.C, D19.C, D20.C, D24.C, D25.C, D27.C, D28.C, D29.C, IC2.+VS, MCP1825(ANALOG).+3V3, REF19X.!SHDN, REF19X.VIN, TP11.1
- net AGND: now also C20.2, IC1.VCC, LMV1.GND/VCC-, LMV2.GND/VCC-, LMV3.GND/VCC-; no longer C36.2, C50.2, C53.2, D10.A, D11.A, D12.A, D13.A, D5.A, D6.A, D7.A, D8.A, D9.A, IC2.-VS, R54.2
- net ANT: now also JP6.2
- net BIAS: now also LMV1.4IN+, LMV2.4IN+, LMV3.4IN+, TP5.1; no longer C35.1, C36.1, CT1.1, CT2.1, CT3.1, CT4.1, CT5.1, CT6.1, CT7.1, CT8.1, CT9.1, JP10.1, JP11.1, JP12.1, JP13.1, JP14.1, JP15.1, JP16.1, JP17.1, JP18.1, R23.2, R38.1, R42.1, R44.1, R45.1, R46.1, R47.1, R48.1, R49.1, R50.1, R51.1, TP3.1
- net CT_IN1: now also LMV1.1IN-, RB10.2; no longer D13.C, D29.A, RB1B.1, RF1.1
- net CT_IN2: now also LMV1.2IN-, RB14.2; no longer D12.C, D28.A, RB2B.1, RF2.1
- net CT_IN3: now also LMV1.3IN-, RB15.1; no longer D11.C, D27.A, RB3B.1, RF3.1
- net CT_IN4: now also LMV2.1IN-, RB11.2; no longer D10.C, D25.A, RB4B.1, RF4.1
- net CT_IN5: now also LMV2.2IN-, RB12.2; no longer D20.A, D9.C, RB5B.1, RF5.1
- net CT_IN6: now also LMV2.3IN-, RB13.1; no longer D24.A, D8.C, RB6B.1, RF6.1
- net CT_IN7: now also LMV3.1IN-, RB16.2; no longer D19.A, D7.C, RB7B.1, RF7.1
- net CT_IN8: now also LMV3.2IN-, RB17.2; no longer D16.A, D6.C, RB8B.1, RF8.1
- net CT_IN9: now also LMV3.3IN-, RB18.1; no longer D15.A, D5.C, RB9B.1, RF9.1
- net DGND: now also U2.GND@2
- net DIO0_RFM: now also U2.DIO0
- net N$1: no longer JP10.2
- net N$10: no longer JP13.2
- net N$13: no longer JP14.2
- net N$2: no longer JP11.2
- net N$20: no longer JP15.2
- net N$21: no longer JP16.2
- net N$22: no longer JP17.2
- net N$23: no longer JP18.2
- net N$24: now also CT6.3; no longer R47.2, RB5.2, RB5B.2, RB5_.2
- net N$25: now also FB10.P$1, MCP1825.+3V3; no longer R46.2, RB6.2, RB6B.2, RB6_.2
- net N$26: now also CT1.1, RB19.1; no longer R42.2, RB1B.2
- net N$27: now also CT2.1, RB20.1; no longer R44.2, RB2B.2
- net N$29: now also C11.1, C37.1, FB6.P$1, REF19X.!SHDN, REF19X.VIN, TP11.1; no longer R50.2, RB8.2, RB8B.2, RB8_.2
- net N$34: now also FB11.P$1, MCP1825(ANALOG).+3V3; no longer R51.2, RB9.2, RB9B.2, RB9_.2
- net N$35: now also CT4.1, RB44.1; no longer R48.2, RB4B.2
- net N$36: now also CT3.1, RB21.1, RB3.2, RB3_.2; no longer R49.2, RB7.2, RB7B.2, RB7_.2
- net N$37: now also JP3.2, R55.1, R56.2; no longer R45.2, RB3.2, RB3B.2, RB3_.2
- net N$7: now also CT5.1, RB5.2, RB55.1, RB5_.2; no longer C50.1, R23.1
- net N$8: no longer JP12.2
- net OPAMP_INVERT-: now also SJ1.1; no longer C20.1, IC2.IN-, R38.2, R54.1, TP6.1
- net OPAMP_OUT: now also SJ1.2; no longer C20.2, IC2.OUT, R6.1, STM32F303VE.PB12, TP5.1
- net RGND: now also U2.GND@1, U2.GND@3
- net RST_RFM: now also U2.RESET
- net SPI4_CLK_MASTER: now also U2.SCK
- net SPI4_CS_RFM69_MASTER: now also U2.NSS
- net SPI4_MISO_MASTER: now also U2.MISO
- net SPI4_MOSI_MASTER: now also U2.MOSI
- net VDD: now also U2.VDD
Other:
- note added: "RFMxx"
- note added: "maybe DNGA comes off the ANA supply with FB in series"
- note removed: "RFM69"
- note removed: "maybe DNGA comes off the ana supply with FB in series"
- moved on the sheet: C20, C33, C35, C43, CF1, CF2, CF3, CF4, CF5, CF6, CF7, CF8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

Commit message: sync
Parts:
- removed BOOT_STM: (no value), con-lstb-db:MA02-1
- removed IC1: TS461CLT, TS461CLT:TS461CLT
- removed JP3, JP5: JUMPER-SMT_3_1-NC_TRACE_NO-SILK, SparkFun-Jumpers:JUMPER-SMT_3_1-NC_TRACE_NO-SILK
- removed TERM3: 3.5MM_TB_X6, 3.5mm terminal block rs pro:3.5MM_TB_X6
- removed TP3, TP4, TP5, TP6: TEST-POINTPOGO_PTH, SparkFun-Connectors:TEST-POINTPOGO_PTH
- added BOOT, RST_STM: (no value), SparkFun:M02PTH
- added C36, C50, C53, C56: 100nF, resistor:C-EUC0603
- added D10, D5, D6, D7, D8, D9: (no value), adafruit:DIODESOD-523
- added D11: ESD5Z3.3T1G, adafruit:DIODESOD-523
- added S3: KSC222JLFS, Switch:KSC222JLFS
- added SJ2: JUMPER-SMT_2_NC_TRACE_NO-SILK, SparkFun-Jumpers:JUMPER-SMT_2_NC_TRACE_NO-SILK
- added TB3: 3.5MM_TB_X6, 3.5mm terminal block rs pro:3.5MM_TB_X6
- C10, C15, C24, C25, C27: value 2.2uF -> 22uF
- C11: value 22uf -> 22uF
- C23: value 22uf -> 2.2uf
- C26, C28: value 100nF -> 2.2uF
- C35: value 22uF -> 100nF; device rcl:C-EUC0805 -> resistor:C-EUC0603
- C52, C7, C9: value 1uF -> 2.2uF
- C54, C55: value 47uF -> 22uF
- D1, D4: value ESD5Z3.3T1G -> (none); device microbuilder:DIODESOD-523 -> adafruit:DIODESOD-523; MPN (none) -> PESD3V3S1UB
- D14, D17, D18, D21, D26, D33, D34, D35: device microbuilder:DIODESOD-523 -> adafruit:DIODESOD-523
- D2, D3: value SCHOTTKY_MBR0520LT1GDO-219-AB(SOD123F) -> ESD5Z3.3T1G; device Diode:SCHOTTKY_MBR0520LT1GDO-219-AB(SOD123F) -> adafruit:DIODESOD-523; MPN MBR130LSFT1G -> (none)
- FB3, FB4, FB7: value (none) -> 0R; MPN BLM18BD252SN1D -> (none)
- FB8, FB9: value (none) -> 600R
- HSE: MPN (none) -> X50328MSD4SC; MPN2 (none) -> MCSJK-6G-8.00-16-10-80-B-20
- IC_VBAT: MPN (none) -> AP7313-33SRG-7
- KSS331GLFS: MPN (none) -> KSS331GLFS
- LED1, LED_PWR: value Green 1.85V -> Green; MPN (none) -> C2297
- LED2: value Orange 1.85V -> Yellow; MPN (none) -> C2296
- LED3: value Red 1.85V -> Blue; MPN (none) -> C2293
- LSE: MPN (none) -> ABS25-32.768KHZ-T
- R17: value 220K -> 220k
- R18, R19: value 1k -> 1k5
- R53: value 10k -> 9k53
- R6: value 20R -> 0R
- RB10, RB11, RB12, RB13, RB14, RB15, RB16, RB17, RB18, RB19, RB20, RB21, RB22, RB23, RB24, RB44, RB55, RB66: device rcl:R-EU_R0805 -> rcl:R-EU_R0603
- U$2: value BOOST_MODULE -> BOOST_MODULEBOTHCONN; device BOOST MODULE CN6009:BOOST_MODULE -> BOOST MODULE CN6009:BOOST_MODULEBOTHCONN
- renumbered LED4 to LED_PWR, S2 to KSS331GLFS, STM32F303VE to STM32F303VCT6, U$7 to MICROSD
Connections:
- removed net BIAS: D2.A, D3.C, LMV1.4IN+, LMV2.4IN+, LMV3.4IN+, LMV824.4IN+, R34.2, R53.2, R6.2, TP5.1, VT1.RING, VT1.RING_SW
- removed net BIAS_SOT23: IC1.-V, IC1.OUT, JP5.2
- removed net N$39: C20.1, IC1.+V, JP3.3, TP6.1
- removed net N$42: JP5.3, R6.1, TP3.1
- new net BIAS_INPUT: C20.1, C35.1, C36.1, C50.1, C56.1, LMV1.4IN+, LMV2.4IN+, LMV3.4IN+, LMV824.4IN+, R55.1, R56.2
- new net N$44: IC_VBAT.OUT, SJ2.2
- net +3V3: now also BOOT.1, C53.1, D11.C, D2.C, D3.C, S3.3, S3.4; no longer BOOT_STM.2
- net +3V3ANA: now also D10.C, D6.C, D8.C; no longer D2.C, IC1.VDD
- net +5V: no longer TP4.1
- net 3PH_BIAS: now also D1.C, D4.A, R34.2, R53.2, TB3.P$1, TB3.P$3, TB3.P$5, VT1.RING, VT1.RING_SW; no longer TERM3.P$1, TERM3.P$3, TERM3.P$5
- net AC1: no longer D1.C, D4.A
- net AGND: now also C36.2, C50.2, C56.2, D5.A, D7.A, D9.A; no longer D3.A, IC1.VCC
- net ANT: now also R6.2; no longer SMA.1
- net BIAS123: now also D5.C, D6.A
- net BIAS456: now also D7.C, D8.A
- net BIAS789: now also D10.A, D9.C
- net BOOT_STM: now also BOOT.2, S3.1, S3.2; no longer BOOT_STM.1
- net DGND: now also C53.2, RST_STM.2
- net EXT_TERM1: now also D11.A
- net EXT_TERM2: now also D3.A
- net EXT_TERM3: now also D2.A
- net L1-: now also TB3.P$2; no longer TERM3.P$2
- net L2-: now also TB3.P$4; no longer TERM3.P$4
- net L3-: now also TB3.P$6; no longer TERM3.P$6
- net N$16: now also SJ2.1; no longer IC_VBAT.OUT
- net N$37: now also R6.1, SMA.1; no longer JP3.2, R55.1, R56.2
- net NRST_STM: now also RST_STM.1
- net STM32_OPAMP_NON-INVERT+: no longer C35.1, JP3.1
- net STM32_OPAMP_OUT: no longer JP5.1
Other:
- note added: "3ph bias ESD diodes"
- note added: "I2C etc."
- note added: "STM32F3 OpenEnergyMonitor Concept"
- note removed: "STM32F303 OpenEnergyMonitor Concept"
- note removed: "Schematic Version v0.9"
- moved on the sheet: C1, C19, C20, C22, C35, C40, C41, C42, C45, C46, C47, C52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

Commit message: sync
Parts:
- added C57, C59, C60: 22uF, rcl:C-EUC0805
- added C58, C61: 100nF, resistor:C-EUC0603
- FB1: value 1600R -> 600R
- FB10, FB11, FB5: value (none) -> 0R
- FB6: value (none) -> 600R
- R22: value 0R -> (none)
- renumbered RB10 to R60, RB11 to R63, RB12 to R64, RB13 to R65, RB14 to R61, RB15 to R62, RB16 to R66, RB17 to R67, RB18 to R68
Connections:
- net +5V: no longer TB2.P$6, U$2.+5V
- net +5V_USB: now also C58.1, C59.1, C60.1, TB2.P$6, U$2.+5V
- net AGND: now also C57.2, C61.2
- net DGND: now also C58.2, C59.2, C60.2
- net N$29: now also C57.1, C61.1
Other:
- moved on the sheet: C20, R55, R56
