File: Hardware/stm32-pi_full/stm32 v1.2.brd (EAGLE design)
At the start: 131.4 x 105.8 mm, 277 parts, among them J1 JUMPER-SMT_2_NC_TRACE_NO-SILK, Q1 PNP, Q2 NPN, Q3 NPN, U1 ESP32-WROOM-32D, U2 RFM69HCW/RFM95W

Commit message: sync
Parts:
- R43: value 220k -> 140k
- R53: value 9k53 -> 10k
- VT1: value ADC-028-2-T -> ADC-028-1-T
- moved D12 122.2 mm to (81.8, 41.3), turned to 90 degrees
- moved RST_STM 2.16 mm to (129.3, 34.8), turned to 270 degrees
- moved BOOT 2.08 mm to (128.5, 14.7), turned to 270 degrees
- moved C7 1.66 mm to (81.2, 43.8)
- moved C31 1.26 mm to (89.3, 48.5), turned to 0 degrees
- moved C32 0.86 mm to (89.5, 50.8), turned to 0 degrees
- moved R8 0.46 mm to (78.7, 42.1)
- renumbered KSS331GLFS to RST, LED_PWR to PWR, S3 to BOOT_
Routing:
- net N$16: track 1.48 -> 3.44 mm
- net +3V3: track 94.8 -> 96.0 mm
- net BOOT_STM: track 167.5 -> 168.5 mm
- net +5V: track 269.4 -> 270.0 mm
Other:
- board text added: "v1.2"
- board text removed: "v1.1"

Commit message: sync
Connections:
- net 3PH_BIAS: now also VT1.PWR2; no longer VT1.GND, VT1.GNDBREAK
- net _AC1: now also VT1.GND, VT1.GNDBREAK; no longer VT1.PWR2
Routing:
- net 3PH_BIAS: track 80.2 -> 68.9 mm
- net _AC1: track 24.7 -> 18.4 mm
Changed lines of the file:
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@@
 <wire x1="127.18029375" y1="72.644084375" x2="128.711421875" y2="71.11295625" width="0.3048" layer="16"/>
 <wire x1="128.711421875" y1="71.11295625" x2="129.282953125" y2="69.733159375" width="0.3048" layer="16" curve="-45"/>
-<contactref element="VT1" pad="GND"/>
-<contactref element="VT1" pad="GNDBREAK"/>
 <contactref element="R53" pad="2"/>
 <contactref element="R34" pad="2"/>
@@
 <wire x1="120.345403125" y1="55.833340625" x2="120.345403125" y2="55.12409375" width="0.4064" layer="1"/>
 <wire x1="120.345403125" y1="55.12409375" x2="122.552953125" y2="52.91654375" width="0.4064" layer="1"/>
-<wire x1="122.552953125" y1="52.91654375" x2="123.8" y2="52.4" width="0.4064" layer="1" curve="45"/>
-<wire x1="123.8" y1="52.4" x2="130" y2="52.4" width="0.3556" layer="1"/>
 <contactref element="D1" pad="K"/>
 <contactref element="D4" pad="A"/>
@@
 <wire x1="127.18029375" y1="58.644084375" x2="127.18029375" y2="56.832396875" width="0.4064" layer="1"/>
 <wire x1="127.18029375" y1="56.832396875" x2="126.43634375" y2="55.03634375" width="0.4064" layer="1" curve="-45"/>
-<wire x1="126.43634375" y1="55.03634375" x2="123.8" y2="52.4" width="0.4064" layer="1"/>
+<contactref element="VT1" pad="PWR2"/>
+<wire x1="122.552953125" y1="52.91654375" x2="126.43634375" y2="55.03634375" width="0" layer="19" extent="1-1"/>
+<wire x1="123.8" y1="41.4" x2="122.552953125" y2="52.91654375" width="0" layer="19" extent="1-1"/>
 </signal>
 <signal name="L1-">
@@
 </signal>
 <signal name="_AC1">
-<contactref element="VT1" pad="PWR2"/>
 <contactref element="R43" pad="2"/>
 <contactref element="R34" pad="1"/>
-<wire x1="123.8" y1="43.1171125" x2="123.8" y2="41.4" width="0.3048" layer="1"/>
 <wire x1="113.824821875" y1="51.934403125" x2="115.5788125" y2="52.66093125" width="0.4064" layer="1" curve="45"/>
 <wire x1="115.5788125" y1="52.66093125" x2="116.8614875" y2="53.94360625" width="0.4064" layer="1"/>
 <wire x1="117.044096875" y1="54.6227875" x2="117.545403125" y2="55.12409375" width="0.4064" layer="1"/>
-<wire x1="123.8" y1="41.4" x2="123.8" y2="45.952990625" width="0.4064" layer="1"/>
 <wire x1="123.8" y1="45.952990625" x2="123.05605" y2="47.74904375" width="0.4064" layer="1" curve="45"/>
 <wire x1="123.05605" y1="47.74904375" x2="116.8614875" y2="53.94360625" width="0.4064" layer="1"/>
@@
 <wire x1="117.545403125" y1="55.12409375" x2="117.194275" y2="54.27639375" width="0.4064" layer="1" curve="-45"/>
 <wire x1="117.194275" y1="54.27639375" x2="116.8614875" y2="53.94360625" width="0.4064" layer="1"/>
+<contactref element="VT1" pad="GND"/>
+<contactref element="VT1" pad="GNDBREAK"/>
+<wire x1="123.8" y1="52.4" x2="130" y2="52.4" width="0" layer="19" extent="1-1"/>
+<wire x1="123.8" y1="45.952990625" x2="123.8" y2="52.4" width="0" layer="19" extent="1-1"/>
 </signal>
 <signal name="AC1">

Commit message: sync
Parts:
- removed RB20: 680R | 681R 0.1%, rcl:R0603
- added RB77: 680R | 681R 0.1%, rcl:R0603
- moved RB22 64.1 mm to (109.1, 90.9)
- moved LOGO1 38.0 mm to (118.0, 54.9)
- renumbered RB19 to RB11, RB21 to RB33, RB23 to RB88, RB24 to RB99
Connections:
- net BIAS123: now also RB22.2; no longer RB20.2
- net BIAS789: now also RB77.2; no longer RB22.2
- net N$27: now also RB22.1; no longer RB20.1
- net N$46: now also RB77.1; no longer RB22.1
