File: Hardware/stm32-pi_full/stm32 v1.2.sch (EAGLE design)
At the start: 276 parts, among them J1 JUMPER-SMT_2_NC_TRACE_NO-SILK, Q1 PNP, Q2 NPN, Q3 NPN, U1 ESP32-WROOM-32D, U2 RFM69HCW/RFM95W

Commit message: sync
Parts:
- R43: value 220k -> 140k
- R53: value 9k53 -> 10k
- VT1: value ADC-028-2-T -> ADC-028-1-T; MPN FC68148S -> PJ-002AH-SMT-TR; MPN2 (none) -> ADC-028-1-T; NOTE (none) -> 2.0-2.35mm PIN DIA.
- renumbered KSS331GLFS to RST, LED_PWR to PWR, S3 to BOOT_
Other:
- note added: "2.0-2.35mm PIN DIA."
- note added: "9.333kOhm equiv. output impedance"
Changed lines of the file:
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@@
 <attribute name="MPN" value="SJ-3523-SMT"/>
 </part>
-<part name="VT1" library="adafruit" library_urn="urn:adsk.eagle:library:420" deviceset="2.1MMJACK" device="SMT" package3d_urn="urn:adsk.eagle:package:6240730/1" value="ADC-028-2-T">
-<attribute name="MPN" value="FC68148S"/>
+<part name="VT1" library="adafruit" library_urn="urn:adsk.eagle:library:420" deviceset="2.1MMJACK" device="SMT" package3d_urn="urn:adsk.eagle:package:6240730/1" value="ADC-028-1-T">
+<attribute name="MPN" value="PJ-002AH-SMT-TR"/>
+<attribute name="MPN2" value="ADC-028-1-T"/>
+<attribute name="NOTE" value="2.0-2.35mm PIN DIA."/>
 </part>
 <part name="RJ1" library="95501-6889 rj45 smt" deviceset="95501-6889" device="" value="95501-6889"/>
 <part name="STM32F303VET6" library="stm32f303" deviceset="STM32F303XB" device="" value="STM32F303VE"/>
-<part name="R43" library="resistor" deviceset="R-EU_" device="R0603" value="220k"/>
+<part name="R43" library="resistor" deviceset="R-EU_" device="R0603" value="140k"/>
 <part name="CV2" library="rcl" library_urn="urn:adsk.eagle:library:334" deviceset="C-EU" device="C0805" package3d_urn="urn:adsk.eagle:package:23617/2" value="10nF 5%"/>
 <part name="CV1" library="rcl" library_urn="urn:adsk.eagle:library:334" deviceset="C-EU" device="C0805" package3d_urn="urn:adsk.eagle:package:23617/2" value="10nF 5%"/>
-<part name="R53" library="resistor" deviceset="R-EU_" device="R0603" value="9k53"/>
+<part name="R53" library="resistor" deviceset="R-EU_" device="R0603" value="10k"/>
 <part name="RF6" library="resistor" deviceset="R-EU_" device="R0603" value="9k1 0.1%"/>
 <part name="CF6" library="rcl" library_urn="urn:adsk.eagle:library:334" deviceset="C-EU" device="C0805" package3d_urn="urn:adsk.eagle:package:23617/2" value="10nF 5%"/>
@@
 <part name="C42" library="resistor" deviceset="C-EU" device="C0603" value="100nF"/>
 <part name="SUPPLY42" library="supply2" library_urn="urn:adsk.eagle:library:372" deviceset="DGND" device=""/>
-<part name="KSS331GLFS" library="KSS221GLFS" deviceset="KSS221GLFS" device="">
+<part name="RST" library="KSS221GLFS" deviceset="KSS221GLFS" device="">
 <attribute name="MPN" value="KSS331GLFS"/>
 </part>
@@
 <part name="AGND22" library="supply1" library_urn="urn:adsk.eagle:library:371" deviceset="AGND" device=""/>
 <part name="R6" library="rcl" library_urn="urn:adsk.eagle:library:334" deviceset="R-EU_" device="R0603" package3d_urn="urn:adsk.eagle:package:23555/3" value="0R"/>
-<part name="LED_PWR" library="adafruit" library_urn="urn:adsk.eagle:library:420" deviceset="LED" device="CHIP-LED0805" package3d_urn="urn:adsk.eagle:package:6240557/1" value="Green">
+<part name="PWR" library="adafruit" library_urn="urn:adsk.eagle:library:420" deviceset="LED" device="CHIP-LED0805" package3d_urn="urn:adsk.eagle:package:6240557/1" value="Green">
 <attribute name="MPN" value="C2297"/>
 </part>
 <part name="C53" library="resistor" deviceset="C-EU" device="C0603" value="100nF"/>
-<part name="S3" library="Switch" library_urn="urn:adsk.eagle:library:11396471" deviceset="KSC222JLFS" device="" package3d_urn="urn:adsk.eagle:package:19992274/4">
+<part name="BOOT_" library="Switch" library_urn="urn:adsk.eagle:library:11396471" deviceset="KSC222JLFS" device="" package3d_urn="urn:adsk.eagle:package:19992274/4">
 <attribute name="MPN2" value="C318887"/>
 </part>
@@
 <text x="289.56" y="304.8" size="1.778" layer="91">3ph bias ESD diodes</text>
 <text x="282.448" y="-58.42" size="2.54" layer="91" ratio="15">I2C etc.</text>
+<text x="404.368" y="356.616" size="1.778" layer="95">2.0-2.35mm PIN DIA.</text>
+<text x="393.954" y="326.898" size="1.778" layer="95">9.333kOhm equiv. output impedance</text>
 </plain>
 <instances>
@@
 <attribute name="NAME" x="416.052" y="350.774" size="2.54" layer="95" rot="R270"/>
 <attribute name="MPN" x="414.02" y="345.44" size="1.778" layer="96" rot="R180" display="off"/>
+<attribute name="MPN2" x="414.02" y="345.44" size="1.778" layer="96" rot="R180" display="off"/>
+<attribute name="NOTE" x="414.02" y="345.44" size="1.778" layer="96" rot="R180" display="off"/>
 </instance>
 <instance part="RJ1" gate="G$1" x="411.48" y="-66.04" smashed="yes">
@@
 <attribute name="VALUE" x="371.475" y="-89.535" size="1.778" layer="96"/>
 </instance>
-<instance part="KSS331GLFS" gate="G$1" x="-37.084" y="96.774" smashed="yes" rot="R90">
+<instance part="RST" gate="G$1" x="-37.084" y="96.774" smashed="yes" rot="R90">
 <attribute name="NAME" x="-41.148" y="102.108" size="1.778" layer="95" rot="R90" align="center-left"/>
 <attribute name="MPN" x="-37.084" y="96.774" size="1.27" layer="96" rot="R90" display="off"/>
@@
 <attribute name="VALUE" x="165.862" y="-201.93" size="1.778" layer="96" rot="R90"/>
 </instance>
-<instance part="LED_PWR" gate="G$1" x="-3.556" y="166.624" smashed="yes">
+<instance part="PWR" gate="G$1" x="-3.556" y="166.624" smashed="yes">
 <attribute name="NAME" x="0" y="162.052" size="1.778" layer="95" rot="R90"/>
 <attribute name="VALUE" x="2.921" y="162.052" size="1.778" layer="96" rot="R90"/>
@@
 <attribute name="VALUE" x="-206.756" y="-190.119" size="1.778" layer="96"/>
 </instance>
-<instance part="S3" gate="G$1" x="-66.04" y="109.22" smashed="yes" rot="R90">
+<instance part="BOOT_" gate="G$1" x="-66.04" y="109.22" smashed="yes" rot="R90">
 <attribute name="NAME" x="-70.866" y="106.172" size="1.778" layer="95" rot="R90"/>
 <attribute name="VALUE" x="-68.834" y="111.252" size="1.778" layer="96" rot="R90"/>
@@
 <pinref part="SUPPLY36" gate="G$1" pin="DGND"/>
 <wire x1="-3.556" y1="161.544" x2="-3.556" y2="159.004" width="0.1524" layer="91"/>
-<pinref part="LED_PWR" gate="G$1" pin="C"/>
+<pinref part="PWR" gate="G$1" pin="C"/>
 </segment>
 <segment>
@@
 <pinref part="SUPPLY3" gate="G$1" pin="DGND"/>
 <wire x1="-37.084" y1="96.774" x2="-37.084" y2="91.948" width="0.1524" layer="91"/>
-<pinref part="KSS331GLFS" gate="G$1" pin="1"/>
+<pinref part="RST" gate="G$1" pin="1"/>
 <pinref part="RST_STM" gate="G$1" pin="2"/>
 <wire x1="-32.004" y1="106.68" x2="-32.004" y2="96.774" width="0.1524" layer="91"/>
@@
 <segment>
 <pinref part="+3V2" gate="G$1" pin="+3V3"/>
-<pinref part="S3" gate="G$1" pin="3"/>
-<pinref part="S3" gate="G$1" pin="4"/>
+<pinref part="BOOT_" gate="G$1" pin="3"/>
+<pinref part="BOOT_" gate="G$1" pin="4"/>
 <wire x1="-55.88" y1="116.84" x2="-55.88" y2="123.19" width="0.1524" layer="91"/>
 <wire x1="-66.04" y1="116.84" x2="-63.5" y2="116.84" width="0.1524" layer="91"/>
@@
 <wire x1="-55.88" y1="104.14" x2="-55.88" y2="101.6" width="0.1524" layer="91"/>
 <pinref part="R2" gate="G$1" pin="1"/>
-<pinref part="S3" gate="G$1" pin="1"/>
-<pinref part="S3" gate="G$1" pin="2"/>
+<pinref part="BOOT_" gate="G$1" pin="1"/>
+<pinref part="BOOT_" gate="G$1" pin="2"/>
 <wire x1="-66.04" y1="104.14" x2="-63.5" y2="104.14" width="0.1524" layer="91"/>
 <junction x="-63.5" y="104.14"/>
@@
 <pinref part="R10" gate="G$1" pin="1"/>
 <wire x1="-3.556" y1="175.26" x2="-3.556" y2="169.164" width="0.1524" layer="91"/>
-<pinref part="LED_PWR" gate="G$1" pin="A"/>
+<pinref part="PWR" gate="G$1" pin="A"/>
 </segment>
 </net>
@@
 <label x="-36.576" y="122.936" size="1.778" layer="95"/>
 <wire x1="-37.084" y1="117.094" x2="-37.084" y2="122.936" width="0.1524" layer="91"/>
-<pinref part="KSS331GLFS" gate="G$1" pin="2"/>
+<pinref part="RST" gate="G$1" pin="2"/>
 <pinref part="RST_STM" gate="G$1" pin="1"/>
 <wire x1="-32.004" y1="109.22" x2="-32.004" y2="117.094" width="0.1524" layer="91"/>
@@
 </segment>
 <segment>
-<wire x1="33.02" y1="114.3" x2="34.544" y2="114.3" width="0.1524" layer="91"/>
-<label x="33.02" y="114.3" size="1.27" layer="95" rot="R180" xref="yes"/>
+<wire x1="27.94" y1="114.3" x2="34.544" y2="114.3" width="0.1524" layer="91"/>
+<label x="27.94" y="114.3" size="1.27" layer="95" rot="R180" xref="yes"/>
 <pinref part="R33" gate="G$1" pin="2"/>
 <wire x1="34.544" y1="119.38" x2="34.544" y2="114.3" width="0.1524" layer="91"/>

Commit message: sync
Connections:
- net 3PH_BIAS: now also VT1.TIP; no longer VT1.RING, VT1.RING_SW
- net _AC1: now also VT1.RING, VT1.RING_SW; no longer VT1.TIP
Other:
- moved on the sheet: VT1
Changed lines of the file:
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@@
 <attribute name="MPN" x="246.38" y="182.88" size="1.778" layer="96" rot="R180" display="off"/>
 </instance>
-<instance part="VT1" gate="G$1" x="414.02" y="345.44" smashed="yes" rot="R180">
-<attribute name="NAME" x="416.052" y="350.774" size="2.54" layer="95" rot="R270"/>
-<attribute name="MPN" x="414.02" y="345.44" size="1.778" layer="96" rot="R180" display="off"/>
-<attribute name="MPN2" x="414.02" y="345.44" size="1.778" layer="96" rot="R180" display="off"/>
-<attribute name="NOTE" x="414.02" y="345.44" size="1.778" layer="96" rot="R180" display="off"/>
+<instance part="VT1" gate="G$1" x="421.64" y="345.44" smashed="yes" rot="R180">
+<attribute name="NAME" x="423.672" y="350.774" size="2.54" layer="95" rot="R270"/>
+<attribute name="MPN" x="421.64" y="345.44" size="1.778" layer="96" rot="R180" display="off"/>
+<attribute name="MPN2" x="421.64" y="345.44" size="1.778" layer="96" rot="R180" display="off"/>
+<attribute name="NOTE" x="421.64" y="345.44" size="1.778" layer="96" rot="R180" display="off"/>
 </instance>
 <instance part="RJ1" gate="G$1" x="411.48" y="-66.04" smashed="yes">
@@
 </segment>
 <segment>
-<pinref part="VT1" gate="G$1" pin="RING_SW"/>
-<pinref part="VT1" gate="G$1" pin="RING"/>
-<wire x1="408.94" y1="347.98" x2="408.94" y2="345.44" width="0.1524" layer="91"/>
-<junction x="408.94" y="347.98"/>
 <wire x1="408.94" y1="355.6" x2="408.94" y2="350.52" width="0.1524" layer="91"/>
-<wire x1="408.94" y1="350.52" x2="408.94" y2="347.98" width="0.1524" layer="91"/>
 <wire x1="393.7" y1="355.6" x2="408.94" y2="355.6" width="0.1524" layer="91"/>
 <pinref part="R53" gate="G$1" pin="2"/>
@@
 <pinref part="R34" gate="G$1" pin="2"/>
 <wire x1="406.908" y1="350.52" x2="408.94" y2="350.52" width="0.1524" layer="91"/>
-<junction x="408.94" y="350.52"/>
 <wire x1="388.62" y1="355.6" x2="393.7" y2="355.6" width="0.1524" layer="91"/>
+<pinref part="VT1" gate="G$1" pin="TIP"/>
+<wire x1="416.56" y1="342.9" x2="408.94" y2="350.52" width="0.1524" layer="91"/>
+<junction x="408.94" y="350.52"/>
 </segment>
 <segment>
@@
 <segment>
 <pinref part="R43" gate="G$1" pin="2"/>
-<pinref part="VT1" gate="G$1" pin="TIP"/>
-<wire x1="408.94" y1="342.9" x2="408.94" y2="340.36" width="0.1524" layer="91"/>
-<junction x="408.94" y="340.36"/>
 <pinref part="R34" gate="G$1" pin="1"/>
 <wire x1="406.908" y1="340.36" x2="408.94" y2="340.36" width="0.1524" layer="91"/>
 <label x="415.036" y="340.36" size="1.778" layer="95"/>
+<pinref part="VT1" gate="G$1" pin="RING"/>
+<pinref part="VT1" gate="G$1" pin="RING_SW"/>
+<wire x1="416.56" y1="347.98" x2="416.56" y2="345.44" width="0.1524" layer="91"/>
+<wire x1="416.56" y1="345.44" x2="408.94" y2="340.36" width="0.1524" layer="91"/>
+<junction x="416.56" y="345.44"/>
+<junction x="408.94" y="340.36"/>
 </segment>
 </net>

Commit message: sync
Parts:
- removed RB20: 680R | 681R 0.1%, rcl:R-EU_R0603
- added RB77: 680R | 681R 0.1%, rcl:R-EU_R0603
- renumbered RB19 to RB11, RB21 to RB33, RB23 to RB88, RB24 to RB99
Connections:
- net BIAS123: now also RB22.2; no longer RB20.2
- net BIAS789: now also RB77.2; no longer RB22.2
- net N$27: now also RB22.1; no longer RB20.1
- net N$46: now also RB77.1; no longer RB22.1
Other:
- moved on the sheet: RB22
Changed lines of the file:
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@@
 <part name="R67" library="rcl" library_urn="urn:adsk.eagle:library:334" deviceset="R-EU_" device="R0603" package3d_urn="urn:adsk.eagle:package:23555/3" value="510R 0.1%"/>
 <part name="R68" library="rcl" library_urn="urn:adsk.eagle:library:334" deviceset="R-EU_" device="R0603" package3d_urn="urn:adsk.eagle:package:23555/3" value="510R 0.1%"/>
-<part name="RB19" library="rcl" library_urn="urn:adsk.eagle:library:334" deviceset="R-EU_" device="R0603" package3d_urn="urn:adsk.eagle:package:23555/3" value="680R | 681R 0.1%"/>
-<part name="RB20" library="rcl" library_urn="urn:adsk.eagle:library:334" deviceset="R-EU_" device="R0603" package3d_urn="urn:adsk.eagle:package:23555/3" value="680R | 681R 0.1%"/>
-<part name="RB21" library="rcl" library_urn="urn:adsk.eagle:library:334" deviceset="R-EU_" device="R0603" package3d_urn="urn:adsk.eagle:package:23555/3" value="680R | 681R 0.1%"/>
+<part name="RB11" library="rcl" library_urn="urn:adsk.eagle:library:334" deviceset="R-EU_" device="R0603" package3d_urn="urn:adsk.eagle:package:23555/3" value="680R | 681R 0.1%"/>
 <part name="RB22" library="rcl" library_urn="urn:adsk.eagle:library:334" deviceset="R-EU_" device="R0603" package3d_urn="urn:adsk.eagle:package:23555/3" value="680R | 681R 0.1%"/>
-<part name="RB23" library="rcl" library_urn="urn:adsk.eagle:library:334" deviceset="R-EU_" device="R0603" package3d_urn="urn:adsk.eagle:package:23555/3" value="680R | 681R 0.1%"/>
-<part name="RB24" library="rcl" library_urn="urn:adsk.eagle:library:334" deviceset="R-EU_" device="R0603" package3d_urn="urn:adsk.eagle:package:23555/3" value="680R | 681R 0.1%"/>
+<part name="RB33" library="rcl" library_urn="urn:adsk.eagle:library:334" deviceset="R-EU_" device="R0603" package3d_urn="urn:adsk.eagle:package:23555/3" value="680R | 681R 0.1%"/>
+<part name="RB77" library="rcl" library_urn="urn:adsk.eagle:library:334" deviceset="R-EU_" device="R0603" package3d_urn="urn:adsk.eagle:package:23555/3" value="680R | 681R 0.1%"/>
+<part name="RB88" library="rcl" library_urn="urn:adsk.eagle:library:334" deviceset="R-EU_" device="R0603" package3d_urn="urn:adsk.eagle:package:23555/3" value="680R | 681R 0.1%"/>
+<part name="RB99" library="rcl" library_urn="urn:adsk.eagle:library:334" deviceset="R-EU_" device="R0603" package3d_urn="urn:adsk.eagle:package:23555/3" value="680R | 681R 0.1%"/>
 <part name="FB6" library="microbuilder" deviceset="FERRITE" device="_0603" value="600R">
 <attribute name="MPN" value="BLM18BD252SN1D"/>
@@
 <instance part="RB1" gate="G$1" x="231.14" y="185.42" smashed="yes" rot="R90">
 <attribute name="NAME" x="229.6414" y="181.61" size="1.778" layer="95" rot="R90"/>
+<attribute name="VALUE" x="234.442" y="181.61" size="1.778" layer="96" rot="R90"/>
 </instance>
 <instance part="RB4" gate="G$1" x="304.8" y="185.42" smashed="yes" rot="R90">
@@
 <instance part="R60" gate="G$1" x="220.98" y="274.32" smashed="yes">
 <attribute name="NAME" x="217.17" y="275.8186" size="1.778" layer="95"/>
+<attribute name="VALUE" x="217.17" y="271.018" size="1.778" layer="96"/>
 </instance>
 <instance part="LMV1" gate="G$1" x="228.6" y="276.86" smashed="yes">
@@
 <attribute name="NAME" x="405.13" y="265.6586" size="1.778" layer="95"/>
 </instance>
-<instance part="RB19" gate="G$1" x="251.46" y="193.04" smashed="yes">
+<instance part="RB11" gate="G$1" x="251.46" y="193.04" smashed="yes">
 <attribute name="NAME" x="247.65" y="194.5386" size="1.778" layer="95"/>
+<attribute name="VALUE" x="247.65" y="189.738" size="1.778" layer="96"/>
 </instance>
-<instance part="RB20" gate="G$1" x="248.92" y="137.16" smashed="yes">
+<instance part="RB22" gate="G$1" x="248.92" y="137.16" smashed="yes">
 <attribute name="NAME" x="245.11" y="138.6586" size="1.778" layer="95"/>
 </instance>
-<instance part="RB21" gate="G$1" x="248.92" y="81.28" smashed="yes">
+<instance part="RB33" gate="G$1" x="248.92" y="81.28" smashed="yes">
 <attribute name="NAME" x="245.11" y="82.7786" size="1.778" layer="95"/>
 </instance>
-<instance part="RB22" gate="G$1" x="401.32" y="193.04" smashed="yes">
+<instance part="RB77" gate="G$1" x="401.32" y="193.04" smashed="yes">
 <attribute name="NAME" x="397.51" y="194.5386" size="1.778" layer="95"/>
 </instance>
-<instance part="RB23" gate="G$1" x="401.32" y="137.16" smashed="yes">
+<instance part="RB88" gate="G$1" x="401.32" y="137.16" smashed="yes">
 <attribute name="NAME" x="397.51" y="138.6586" size="1.778" layer="95"/>
 </instance>
-<instance part="RB24" gate="G$1" x="401.32" y="81.28" smashed="yes">
+<instance part="RB99" gate="G$1" x="401.32" y="81.28" smashed="yes">
 <attribute name="NAME" x="397.51" y="82.7786" size="1.778" layer="95"/>
 </instance>
@@
 </segment>
 <segment>
-<pinref part="RB19" gate="G$1" pin="2"/>
-<pinref part="RB20" gate="G$1" pin="2"/>
+<pinref part="RB11" gate="G$1" pin="2"/>
+<pinref part="RB22" gate="G$1" pin="2"/>
 <wire x1="254" y1="137.16" x2="259.08" y2="137.16" width="0.1524" layer="91"/>
-<pinref part="RB21" gate="G$1" pin="2"/>
+<pinref part="RB33" gate="G$1" pin="2"/>
 <wire x1="259.08" y1="193.04" x2="259.08" y2="137.16" width="0.1524" layer="91"/>
 <wire x1="259.08" y1="137.16" x2="259.08" y2="81.28" width="0.1524" layer="91"/>
@@
 </segment>
 <segment>
-<pinref part="RB22" gate="G$1" pin="2"/>
+<pinref part="RB77" gate="G$1" pin="2"/>
 <wire x1="406.4" y1="193.04" x2="408.94" y2="193.04" width="0.1524" layer="91"/>
 <wire x1="408.94" y1="193.04" x2="408.94" y2="137.16" width="0.1524" layer="91"/>
-<pinref part="RB23" gate="G$1" pin="2"/>
+<pinref part="RB88" gate="G$1" pin="2"/>
 <wire x1="408.94" y1="137.16" x2="406.4" y2="137.16" width="0.1524" layer="91"/>
-<pinref part="RB24" gate="G$1" pin="2"/>
+<pinref part="RB99" gate="G$1" pin="2"/>
 <wire x1="406.4" y1="81.28" x2="408.94" y2="81.28" width="0.1524" layer="91"/>
 <wire x1="408.94" y1="137.16" x2="408.94" y2="81.28" width="0.1524" layer="91"/>
@@
 <pinref part="RB1_" gate="G$1" pin="2"/>
 <wire x1="231.14" y1="190.5" x2="236.22" y2="190.5" width="0.1524" layer="91"/>
-<pinref part="RB19" gate="G$1" pin="1"/>
+<pinref part="RB11" gate="G$1" pin="1"/>
 <wire x1="231.14" y1="190.5" x2="231.14" y2="193.04" width="0.1524" layer="91"/>
 <wire x1="231.14" y1="193.04" x2="241.3" y2="193.04" width="0.1524" layer="91"/>
@@
 <pinref part="RB2" gate="G$1" pin="2"/>
 <wire x1="236.22" y1="134.62" x2="231.14" y2="134.62" width="0.1524" layer="91"/>
-<pinref part="RB20" gate="G$1" pin="1"/>
+<pinref part="RB22" gate="G$1" pin="1"/>
 <wire x1="231.14" y1="134.62" x2="231.14" y2="137.16" width="0.1524" layer="91"/>
 <wire x1="231.14" y1="137.16" x2="241.3" y2="137.16" width="0.1524" layer="91"/>
@@
 <pinref part="RB3" gate="G$1" pin="2"/>
 <wire x1="236.22" y1="78.74" x2="231.14" y2="78.74" width="0.1524" layer="91"/>
-<pinref part="RB21" gate="G$1" pin="1"/>
+<pinref part="RB33" gate="G$1" pin="1"/>
 <wire x1="231.14" y1="78.74" x2="231.14" y2="81.28" width="0.1524" layer="91"/>
 <wire x1="231.14" y1="81.28" x2="241.3" y2="81.28" width="0.1524" layer="91"/>
@@
 <pinref part="RB9" gate="G$1" pin="2"/>
 <wire x1="388.62" y1="78.74" x2="383.54" y2="78.74" width="0.1524" layer="91"/>
-<pinref part="RB24" gate="G$1" pin="1"/>
+<pinref part="RB99" gate="G$1" pin="1"/>
 <wire x1="383.54" y1="78.74" x2="383.54" y2="81.28" width="0.1524" layer="91"/>
 <wire x1="383.54" y1="81.28" x2="393.7" y2="81.28" width="0.1524" layer="91"/>
@@
 <pinref part="RB8" gate="G$1" pin="2"/>
 <wire x1="388.62" y1="134.62" x2="383.54" y2="134.62" width="0.1524" layer="91"/>
-<pinref part="RB23" gate="G$1" pin="1"/>
+<pinref part="RB88" gate="G$1" pin="1"/>
 <wire x1="383.54" y1="134.62" x2="383.54" y2="137.16" width="0.1524" layer="91"/>
 <wire x1="383.54" y1="137.16" x2="393.7" y2="137.16" width="0.1524" layer="91"/>
@@
 <pinref part="RB7" gate="G$1" pin="2"/>
 <wire x1="388.62" y1="190.5" x2="383.54" y2="190.5" width="0.1524" layer="91"/>
-<pinref part="RB22" gate="G$1" pin="1"/>
+<pinref part="RB77" gate="G$1" pin="1"/>
 <wire x1="383.54" y1="190.5" x2="383.54" y2="193.04" width="0.1524" layer="91"/>
 <wire x1="383.54" y1="193.04" x2="393.7" y2="193.04" width="0.1524" layer="91"/>
