File: Hardware/stm32-pi_full/images/v0.6 Sept 2019/v0.6 stm32-pi.brd (EAGLE design)
At the start: 128.9 x 105.8 mm, 198 parts, among them Q1 MMBT3906, Q2 MMBT3904, Q3 MMBT3904, U1 ESP32-WROOM-32D

Commit message: commit
Parts:
- removed D20: (no value), diode:SMBJ
- removed TP4, TP5, TP6: TPB1,27, testpad:B1,27
- USB-C: value CSP-USC16-TR -> 105450-0101; device CSP-USC16-TR:USB-C -> 105450-0101:MOLEX_105450-0101
- moved USB-C 2.15 mm to (125.1, 23.7)
- moved CF1 0.47 mm to (11.7, 83.8)
- moved C29 0.35 mm to (6.21, 14.9)
- moved SJ22 0.17 mm to (73.3, 34.2), turned to 0 degrees
Connections:
- removed net NRST_STM: JP3.6, PCB2.P$71, S2.2, STM32F303VB.14, U1.30
- removed net RST_RFM: PCB2.P$69, RFM69HCW.6, U1.28
- new net NRST: JP3.6, PCB2.P$69, RFM69HCW.6, S2.2, STM32F303VB.14
- net +5V: now also USB-C.A4, USB-C.A9, USB-C.B4, USB-C.B9; no longer D20.C, TP4.TP, USB-C.A4/B9, USB-C.B4/A9
- net D+: now also USB-C.B6; no longer TP5.TP
- net D-: now also USB-C.B7; no longer TP6.TP
- net GND: now also USB-C.A1, USB-C.A12, USB-C.B1, USB-C.B12, USB-C.S1, USB-C.S2, USB-C.S3, USB-C.S4; no longer D20.A, U1.31, USB-C.A1/B12, USB-C.B1/A12, USB-C.GND1, USB-C.GND2, USB-C.GND3, USB-C.GND4
Routing:
- net +3V3: track 494.8 -> 0.00 mm, vias 31 -> 0
- net GND: track 469.6 -> 0.00 mm, vias 175 -> 0
- net BIAS: track 390.1 -> 0.00 mm, vias 2 -> 0
- net +5V: track 304.3 -> 0.00 mm, vias 12 -> 0
- net NRST_STM: track 304.2 -> 0.00 mm, vias 18 -> 0
- net DIO0: track 145.6 -> 0.00 mm, vias 6 -> 0
- net CS_RFM69: track 132.1 -> 0.00 mm, vias 7 -> 0
- net ADC_RJ45IN: track 124.4 -> 0.00 mm, vias 6 -> 0
- net DS18B20_RJ45: track 124.0 -> 0.00 mm, vias 2 -> 0
- net PULSE1_RJ45: track 115.8 -> 0.00 mm, vias 2 -> 0
- net LED1_GREEN: track 114.7 -> 0.00 mm, vias 4 -> 0
- net PULSE2: track 114.5 -> 0.00 mm, vias 6 -> 0
- net SCL: track 111.7 -> 0.00 mm, vias 7 -> 0
- net BUTTON1: track 100.4 -> 0.00 mm, vias 2 -> 0
- net SPI_CLK: track 100.3 -> 0.00 mm, vias 8 -> 0
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Other:
- board text added: "v0.5"
- board text removed: "v0.6"
