File: Hardware/stm32-pi_full/images/v0.6 Sept 2019/v0.6 stm32-pi.sch (EAGLE design)
At the start: 197 parts, among them Q1 MMBT3906, Q2 MMBT3904, Q3 MMBT3904, U1 ESP32-WROOM-32D

Commit message: commit
Parts:
- removed D20: (no value), diode:SUPPRESSOR-SMBJ
- removed TP4, TP5, TP6: TPB1,27, testpad:TPB1,27
- USB-C: value CSP-USC16-TR -> 105450-0101; device CSP-USC16-TR:CSP-USC16-TR -> 105450-0101:105450-0101
Connections:
- removed net NRST_STM: JP3.6, PCB2.GPIO6, S2.2, STM32F303VB.NRST, U1.IO18
- removed net RST_RFM: PCB2.GPIO5, RFM69HCW.!RES, U1.IO17
- new net NRST: JP3.6, PCB2.GPIO5, RFM69HCW.!RES, S2.2, STM32F303VB.NRST
- net +5V: now also USB-C.VBUS3, USB-C.VBUS4; no longer D20.C, TP4.TP
- net D+: now also USB-C.D2+; no longer TP5.TP
- net D-: now also USB-C.D2-; no longer TP6.TP
- net GND: now also USB-C.GND3, USB-C.GND4; no longer D20.A, U1.IO19
