File: Hardware/stm32-pi_basic/6/stm32hw06.brd (EAGLE design)
At the start: 54 x 55 mm, 52 parts

Commit message: modified:   Hardware/stm32-pi_basic/6/stm32hw06.brd 	modified:   Hardware/stm32-pi_full/stm32 v1.1.brd 	deleted:    Protecting Inputs in Digital Electronics ESD Protection | DigiKey.pdf
Parts:
- moved CT3 3.55 mm to (20.7, 54.9)
- moved CT2 2.43 mm to (32.8, 54.5)
- moved U$1 1.82 mm to (7.56, 51.1)
Routing:
- net GND: track 185.0 -> 0.00 mm, vias 28 -> 0
- net BIAS: track 142.6 -> 0.00 mm, vias 2 -> 0
- net +3V3: track 131.2 -> 0.00 mm, vias 5 -> 0
- net +5V: track 90.9 -> 0.00 mm, vias 1 -> 0
- net NRST: track 46.2 -> 0.00 mm, vias 1 -> 0
- net BOOT0: track 31.8 -> 0.00 mm, vias 1 -> 0
- net UART_RX: track 27.9 -> 0.00 mm
- net UART_TX: track 25.8 -> 0.00 mm
- net DS18B20: track 23.7 -> 0.00 mm, vias 2 -> 0
- net N$2: track 23.3 -> 0.00 mm
- net GND_USB: track 23.3 -> 0.00 mm, vias 1 -> 0
- net CT3: track 22.5 -> 0.00 mm
- net VSIG: track 21.1 -> 0.00 mm
- net CT2: track 19.4 -> 0.00 mm
- net HSE_IN: track 18.8 -> 0.00 mm
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
Commit message: deleted:    Hardware/stm32-pi_basic/6/dxfimp.scr 	modified:   Hardware/stm32-pi_basic/6/stm32hw06.brd 	modified:   Hardware/stm32-pi_basic/6/stm32hw06.sch
Parts:
- added PCB1: RPI3RPI3, e14_Rpi3_RevA+mirror-pcb:RPI3
Other:
- board size 54 x 55 mm -> 149.4 x 77.7 mm
Changed lines of the file:
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@@
 <text x="43.5" y="10.25" size="0.8128" layer="27" font="vector" ratio="20">RX</text>
 <text x="41" y="10.25" size="0.8128" layer="27" font="vector" ratio="20">TX</text>
+<wire x1="142.48261875" y1="7.1612" x2="142.48261875" y2="4.641459375" width="0.000253125" layer="20"/>
+<wire x1="149.432409375" y1="11.5909" x2="149.432409375" y2="69.73085" width="0.000253125" layer="20"/>
+<wire x1="145.912559375" y1="70.73061875" x2="148.4323" y2="70.73061875" width="0.000253125" layer="20"/>
+<wire x1="142.48261875" y1="76.680640625" x2="142.48261875" y2="74.1609" width="0.000253125" layer="20"/>
+<wire x1="145.912559375" y1="10.591140625" x2="148.4323" y2="10.591140625" width="0.000253125" layer="20"/>
+<wire x1="83.342909375" y1="77.68075" x2="141.482509375" y2="77.68075" width="0.000253125" layer="20"/>
+<wire x1="82.3428" y1="76.680640625" x2="82.3428" y2="74.1609" width="0.000253125" layer="20"/>
+<wire x1="78.912690625" y1="70.73061875" x2="76.392940625" y2="70.73061875" width="0.000253125" layer="20"/>
+<wire x1="75.393" y1="69.73085" x2="75.393" y2="11.5909" width="0.000253125" layer="20"/>
+<wire x1="78.912690625" y1="10.591140625" x2="76.392940625" y2="10.591140625" width="0.000253125" layer="20"/>
+<wire x1="82.3428" y1="4.641459375" x2="82.3428" y2="7.1612" width="0.000253125" layer="20"/>
+<wire x1="141.482509375" y1="3.641" x2="83.342909375" y2="3.641" width="0.000253125" layer="20"/>
+<wire x1="75.393" y1="69.73085" x2="76.392940625" y2="70.73061875" width="0.000253125" layer="20" curve="-90"/>
+<wire x1="78.912690625" y1="70.73061875" x2="82.3428" y2="74.1609" width="0.000253125" layer="20" curve="90"/>
+<wire x1="82.3428" y1="76.680640625" x2="83.342909375" y2="77.68075" width="0.000253125" layer="20" curve="-90"/>
+<wire x1="142.48261875" y1="74.1609" x2="145.912559375" y2="70.73061875" width="0.000253125" layer="20" curve="90"/>
+<wire x1="141.482509375" y1="77.68075" x2="142.48261875" y2="76.680640625" width="0.000253125" layer="20" curve="-90"/>
+<wire x1="148.4323" y1="70.73061875" x2="149.432409375" y2="69.73085" width="0.000253125" layer="20" curve="-90"/>
+<wire x1="145.912559375" y1="10.591140625" x2="142.48261875" y2="7.1612" width="0.000253125" layer="20" curve="90"/>
+<wire x1="149.432409375" y1="11.5909" x2="148.4323" y2="10.591140625" width="0.000253125" layer="20" curve="-90"/>
+<wire x1="142.48261875" y1="4.641459375" x2="141.482509375" y2="3.641" width="0.000253125" layer="20" curve="-90"/>
+<wire x1="82.3428" y1="7.1612" x2="78.912690625" y2="10.591140625" width="0.000253125" layer="20" curve="90"/>
+<wire x1="83.342909375" y1="3.641" x2="82.3428" y2="4.641459375" width="0.000253125" layer="20" curve="-90"/>
+<wire x1="76.392940625" y1="10.591140625" x2="75.393" y2="11.5909" width="0.000253125" layer="20" curve="-90"/>
+<circle x="82.413" y="15.661" radius="1.60525625" width="0.000253125" layer="20"/>
+<circle x="82.413" y="65.661" radius="1.60525625" width="0.000253125" layer="20"/>
+<circle x="142.413" y="65.661" radius="1.60525625" width="0.000253125" layer="20"/>
+<circle x="142.413" y="15.661" radius="1.60525625" width="0.000253125" layer="20"/>
 </plain>
 <attributes>
@@
 <attribute name="VALUE" x="-28.887928125" y="-34.492690625" size="1.27" layer="27"/>
 </element>
+<element name="PCB1" library="e14_Rpi3_RevA+mirror-pcb" package="RPI3" value="RPI3RPI3" x="143.948" y="69.156" smashed="yes" rot="R180"/>
 </elements>
 <signals>

Commit message: sync
Parts:
- added U1: ESP32-WROOM-32D, ESP32-WROOM-32D:MODULE_ESP32-WROOM-32D
- moved U$10 136.8 mm to (134.4, 2.95), turned to 90 degrees
- moved MCP1825 109.0 mm to (117.0, 9.86), turned to 180 degrees
- moved STM32 90.5 mm to (120.4, 44.9)
- moved CT2 89.9 mm to (119.6, 78.2)
- moved U$1 89.6 mm to (93.7, 75.7)
- moved CT1 89.2 mm to (132.3, 78.2)
- moved CT3 89.2 mm to (106.8, 78.2)
- moved RASPBERRYPI 84.8 mm to (129.4, 16.5)
- moved LOGO1 79.8 mm to (83.6, 21.9)
- moved DS18B20 74.3 mm to (95.3, 10.4)
- moved PULSE 74.3 mm to (105.8, 10.4)
- moved PCB1 0.23 mm to (144.1, 69.0)
Connections:
- new net 3V3: U1.2
- net GND: now also U1.1, U1.15, U1.38, U1.39
Other:
- outline, holes or cut-outs redrawn
- board text added: "emonSTM32mini"
- board text added: "v0.2"
- board text removed: "emonSTM32"
- board text removed: "v0.1"

Commit message: sync
Parts:
- removed GND: UART, con-lsta:FE05-1
- removed PCB1: RPI3RPI3, e14_Rpi3_RevA+mirror-pcb:RPI3
- removed RASPBERRYPI: (no value), con-lsta:FE06-2
- removed SJ1: SOLDERJUMPERNO, SparkFun:SJ_2S-NO
- added C10, C11, C7: 100nF, rcl:C0603
- added C12: 2.2uF, rcl:C0603
- added FB4: FBCHIP-0603(1608-METRIC), Filter:BEADC1608X95N
- added IC1: CP2102, silabs:MLP28
- added J1: CONN_12X2, SparkFun-Connectors:2X12
- added JP1: PINHD-1X2, Connector:1X02
- added JP2: UART_STM, Connector:1X06
- added R5, R6, R7: (no value), rcl:0207/10
- added SMA: 5-1814400-1, 5-1814400-1 sma connector:518144001
- added U$2: RFM12_SMDSMD, rfm12b _ rfm69cw:RFM12
- CF1, CF2, CF3, CFV: value 100nF -> 10nF; device resistor:C0603 -> rcl:C0805
- RB2, RB3: value 22r -> 6R8
- RF1, RF2, RF3, RFV: value 330R -> 9k1
- moved R4 106.3 mm to (56.9, 37.9)
- moved STM32 97.4 mm to (23.0, 42.0), turned to 135 degrees
- moved FB3 88.7 mm to (52.9, 34.3)
- moved CT3 85.8 mm to (21.0, 80.9)
- moved CT1 85.8 mm to (46.6, 80.9)
- moved CT2 85.8 mm to (33.8, 80.9)
- moved FB2 79.6 mm to (57.0, 33.0)
- moved C2 79.2 mm to (25.8, 25.7)
- moved DS18B20 75.3 mm to (20.1, 12.9)
- moved PULSE 75.3 mm to (30.6, 12.9)
- moved U$10 71.1 mm to (63.3, 5.59)
- moved LOGO1 71.1 mm to (12.5, 23.8)
- moved MCP1825 69.7 mm to (47.3, 11.5)
- moved FB1 68.5 mm to (51.8, 39.6)
- moved R19 56.7 mm to (58.9, 65.2)
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Connections:
- removed net 3V3: U1.2
- new net +3V3RPI: J1.1, J1.17
- new net AGND: C1.2, C22.2, FB4.1, STM32.8
- new net CLK_RPI: J1.23
- new net CS_RPI: J1.24
- new net D+: IC1.4, U$10.D+
- new net D-: IC1.5, U$10.D-
- new net ESP_BOOT0: U1.25
- new net ESP_RST: U1.3
- new net ESP_RX: U1.34
- new net ESP_TX: U1.35
- new net MISO_RPI: J1.21
- new net MOSI_RPI: J1.19
- new net N$11: U$2.14
- new net N$13: U$2.2
- new net N$14: U$2.12
- new net N$15: U$2.1
- new net N$16: U$2.13
- new net N$17: U$2.6
- new net N$18: SMA.1, U$2.8
- new net N$19: JP2.5
- new net N$5: J1.9
- new net SCL: J1.5, STM32.45, U1.36
- new net SDA: J1.3, STM32.46, U1.33
- new net SPI3_CLK: STM32.39
- new net SPI3_MISO: STM32.40
- new net SPI3_MOSI: STM32.41
- new net SPI3_NSS: STM32.38
- new net STM_RX: J1.8, JP2.2, STM32.31
- new net STM_TX: J1.10, JP2.3, STM32.30
- net +3V3: now also C11.1, IC1.6, U$2.9, U1.2; no longer C5.1, SJ1.2, STM32.9
- net +3V3ANA: now also STM32.9
- net +5V: now also C10.1, C12.1, IC1.7, IC1.8, J1.2, J1.4, JP2.4; no longer GND.3, RASPBERRYPI.1, RASPBERRYPI.3
- net BIAS: now also R5.2, R6.2, R7.2
- net BIAS_IN: now also C5.1
- net BOOT0: now also IC1.28, J1.7; no longer RASPBERRYPI.8
- net CT1: now also STM32.25; no longer STM32.10
- net CT2: now also CF2.1, STM32.27; no longer CF2.2, STM32.11
- net CT3: now also CF3.1, STM32.28; no longer CF3.2, STM32.12
- net GND: now also C10.2, C11.2, C12.2, C7.2, CF2.2, CF3.2, FB4.2, IC1.3, IC1.EXP, IC1.M, J1.14, J1.20, J1.6, JP2.6, SMA.2, SMA.3, SMA.4, SMA.5, U$2.10, U$2.7; no longer C1.2, C22.2, CF2.1, CF3.1, GND.1, RASPBERRYPI.10, RASPBERRYPI.5, STM32.8
- net LED: now also STM32.42; no longer STM32.27
- net N$1: now also IC1.9; no longer GND.2, SJ1.1
- net N$10: now also R7.1
- net N$2: now also R5.1
- net N$8: now also R6.1
- net PULSE: now also C7.1, STM32.43; no longer STM32.28
- net RST_STM: now also IC1.24, J1.11, JP2.1; no longer RASPBERRYPI.12
- net UART_RX: now also IC1.26, JP1.1; no longer GND.4, RASPBERRYPI.7, STM32.31
- net UART_TX: now also IC1.25, JP1.2; no longer GND.5, RASPBERRYPI.9, STM32.30
- net VSIG: now also STM32.20; no longer STM32.25
Routing:
- net BIAS: track 0.00 -> 197.3 mm, vias 0 -> 3
- net ADC0: track 0.00 -> 29.7 mm
- net N$2: track 0.00 -> 26.1 mm
- net N$8: track 0.00 -> 18.8 mm
- net VSIG: track 0.00 -> 18.3 mm
- net N$10: track 0.00 -> 18.0 mm
- net CT1: track 0.00 -> 16.4 mm
- net STM_TX: track 0.00 -> 15.1 mm
- net CT2: track 0.00 -> 14.1 mm
- net CT3: track 0.00 -> 13.1 mm
- net STM_RX: track 0.00 -> 12.8 mm
- net BIAS_IN: track 0.00 -> 11.9 mm
- net HSE_IN: track 0.00 -> 10.5 mm
- net HSE_OUT: track 0.00 -> 7.82 mm
- net AC: track 0.00 -> 7.44 mm
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Other:
- board size 149.4 x 77.7 mm -> 73.1 x 74 mm
- board text added: "Rx"
- board text added: "Tx"
- board text removed: "3.3"
- board text removed: "RX"
- board text removed: "TX"

Commit message: sync
Parts:
- removed C7: 100nF, rcl:C0603
- added C13: 100nF, rcl:C0603
- added C17: 2.2uF, rcl:C0603
- added JP10, JP3, JP4, JP5, JP6, JP7, JP8, JP9: JUMPER-SMT_2_NC_TRACE_NO-SILK, SparkFun-Jumpers:SMT-JUMPER_2_NC_TRACE_NO-SILK
- added R8: 10k, rcl:R0603
- moved FB1 25.4 mm to (59.6, 15.5), turned to 180 degrees
- moved FB4 21.8 mm to (53.4, 14.7)
- moved C12 13.4 mm to (55.1, 11.3), turned to 270 degrees
- moved IC1 11.6 mm to (59.6, 24.9), turned to 90 degrees
- moved JP1 11.2 mm to (53.1, 25.0)
- moved C10 10.6 mm to (64.2, 23.5)
- moved R22 3.82 mm to (33.3, 45.7), turned to 270 degrees
- moved C5 3.30 mm to (35.5, 48.4), turned to 90 degrees
- moved U$2 3.17 mm to (57.6, 35.4)
- moved C18 2.47 mm to (31.1, 48.5), turned to 90 degrees
- moved C11 2.40 mm to (43.9, 32.5)
- moved U1 1.62 mm to (66.2, 41.7)
- moved R23 1.01 mm to (33.4, 49.1), turned to 270 degrees
- moved C9 0.75 mm to (21.2, 35.3)
- moved HSE 0.60 mm to (30.0, 34.1)
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Connections:
- removed net CLK_RPI: J1.23
- removed net CS_RPI: J1.24
- removed net N$11: U$2.14
- removed net N$13: U$2.2
- removed net N$14: U$2.12
- removed net N$15: U$2.1
- removed net N$16: U$2.13
- removed net N$17: U$2.6
- new net ESP_CLK: JP7.1, U1.30
- new net ESP_CS: JP10.1, U1.29
- new net ESP_MISO: JP8.1, U1.31
- new net ESP_MOSI: JP9.1, U1.37
- new net RFM_IRQ: STM32.11, U$2.2
- new net RFM_RST: STM32.12, U$2.6
- new net RPI_CLK: J1.23, JP5.2, JP7.2
- new net RPI_CONNECTED: R8.2, STM32.2, U1.23
- new net RPI_CONNECTED_PR: J1.17, R8.1
- new net RPI_CS: J1.24, JP10.2, JP6.1
- new net RPI_MISO: JP8.2
- new net RPI_MOSI: JP9.2
- net +3V3: now also C13.1, C17.1; no longer R22.2
- net +3V3ANA: now also R22.2
- net +3V3RPI: no longer J1.17
- net GND: now also C13.2, C17.2; no longer C7.2
- net MISO_RPI: now also JP4.2
- net MOSI_RPI: now also JP3.2
- net PULSE: no longer C7.1
- net SPI3_CLK: now also JP5.1, U$2.13
- net SPI3_MISO: now also JP4.1, U$2.1
- net SPI3_MOSI: now also JP3.1, U$2.12
- net SPI3_NSS: now also JP6.2, U$2.14
Routing:
- net +3V3: track 6.24 -> 97.3 mm, vias 0 -> 4
- net PULSE: track 0.00 -> 44.6 mm
- net +5V: track 0.00 -> 29.8 mm
- net GND: track 5.84 -> 21.4 mm, vias 0 -> 19
- net +3V3ANA: track 4.33 -> 13.3 mm
- net BOOT0: track 0.00 -> 7.94 mm
- net LED: track 0.00 -> 7.43 mm
- net AGND: track 1.83 -> 5.68 mm, vias 0 -> 2
- net BIAS_IN: track 11.9 -> 15.2 mm
- net N$41: track 0.00 -> 2.51 mm
- net +5V_EXT: track 0.00 -> 2.50 mm
- net RPI_CONNECTED_PR: track 0.00 -> 2.26 mm
- net RPI_CS: track 0.00 -> 2.05 mm
- net RPI_CLK: track 0.00 -> 1.91 mm
- net MOSI_RPI: track 0.00 -> 1.91 mm
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
Commit message: sync mini v0.2
Parts:
- removed FB3: FBCHIP-0603(1608-METRIC), Filter:BEADC1608X95N
- removed JP5: JUMPER-SMT_2_NC_TRACE_NO-SILK, SparkFun-Jumpers:SMT-JUMPER_2_NC_TRACE_NO-SILK
- added JP11, JP12: JUMPER-SMT_2_NC_TRACE_NO-SILK, SparkFun-Jumpers:SMT-JUMPER_2_NC_TRACE_NO-SILK
- added R9: 10k, rcl:R0603
- C2: value 100nF -> 2.2uF
- R8: value 10k -> 120k
- moved R4 33.4 mm to (25.5, 26.4), turned to 270 degrees
- moved FB2 24.2 mm to (35.9, 44.8), turned to 180 degrees
- moved C13 24.0 mm to (63.0, 54.7), turned to 90 degrees
- moved C17 23.8 mm to (60.8, 54.7), turned to 90 degrees
- moved C11 18.9 mm to (60.3, 23.2)
- moved FB4 15.7 mm to (39.0, 8.68)
- moved U$2 10.3 mm to (60.4, 45.3)
- moved C10 4.78 mm to (60.4, 26.5), turned to 90 degrees
- moved JP1 4.47 mm to (48.7, 25.8), turned to 270 degrees
- moved C2 3.96 mm to (23.7, 29.0), turned to 90 degrees
- moved IC1 3.52 mm to (56.4, 26.4)
- moved C12 0.94 mm to (55.1, 10.4)
- moved C3 0.94 mm to (52.6, 10.5)
- moved HSE 0.42 mm to (29.6, 34.2)
- moved C9 0.18 mm to (21.3, 35.2)
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Connections:
- removed net GND_USB: FB3.2, U$10.GND, U$10.MTN1, U$10.MTN2, U$10.MTN3, U$10.MTN4
- removed net MISO_RPI: J1.21, JP4.2
- removed net MOSI_RPI: J1.19, JP3.2
- removed net RPI_CLK: J1.23, JP5.2, JP7.2
- removed net SPI3_CLK: JP5.1, STM32.39, U$2.13
- removed net UART_RX: IC1.26, JP1.1
- removed net UART_TX: IC1.25, JP1.2
- new net CP2102_RX: IC1.25, JP1.1, JP11.1
- new net CP2102_TX: IC1.26, JP1.2, JP12.1
- new net SPI_CLK: J1.23, JP7.2, STM32.39, U$2.13
- net ESP_RX: now also JP12.2
- net ESP_TX: now also JP11.2
- net GND: now also R9.1, U$10.GND, U$10.MTN1, U$10.MTN2, U$10.MTN3, U$10.MTN4; no longer FB3.1
- net NRST: no longer STLINK.3
- net RPI_CONNECTED: now also R9.2
- net RPI_MISO: now also J1.21, JP4.2
- net RPI_MOSI: now also J1.19, JP3.2
- net RST_STM: now also STLINK.3
Routing:
- net +3V3: track 97.3 -> 220.7 mm, vias 4 -> 10
- net +5V: track 29.8 -> 135.1 mm, vias 0 -> 2
- net STM_RX: track 13.1 -> 116.2 mm, vias 0 -> 3
- net STM_TX: track 15.3 -> 117.8 mm, vias 0 -> 4
- net SCL: track 0.00 -> 93.9 mm, vias 0 -> 10
- net SPI_CLK: track 0.00 -> 89.2 mm, vias 0 -> 5
- net RST_STM: track 0.00 -> 88.6 mm, vias 0 -> 8
- net SDA: track 0.00 -> 84.4 mm, vias 0 -> 10
- net SPI3_NSS: track 0.00 -> 82.2 mm, vias 0 -> 5
- net RPI_CONNECTED: track 0.00 -> 72.5 mm, vias 0 -> 5
- net SPI3_MOSI: track 0.00 -> 72.0 mm, vias 0 -> 5
- net BOOT0: track 7.94 -> 75.2 mm, vias 0 -> 8
- net DS18B20: track 0.00 -> 55.5 mm, vias 0 -> 4
- net SPI3_MISO: track 0.00 -> 50.9 mm, vias 0 -> 5
- net AGND: track 5.68 -> 56.0 mm, vias 2 -> 3
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Other:
- board size 73.1 x 74 mm -> 71.5 x 74 mm
