File: Hardware/stm32-pi_basic/6/stm32hw06.sch (EAGLE design)
At the start: 51 parts

Commit message: deleted:    Hardware/stm32-pi_basic/6/dxfimp.scr 	modified:   Hardware/stm32-pi_basic/6/stm32hw06.brd 	modified:   Hardware/stm32-pi_basic/6/stm32hw06.sch
Parts:
- added PCB1: RPI3RPI3, e14_Rpi3_RevA+mirror-pcb:RPI3RPI3
Changed lines of the file:
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@@
 <drawing>
 <settings>
-<setting alwaysvectorfont="yes"/>
+<setting alwaysvectorfont="no"/>
 <setting keepoldvectorfont="yes"/>
 <setting verticaltext="up"/>
@@
 <part name="C2" library="resistor" deviceset="C-EU" device="C0603" value="100nF"/>
 <part name="+3V5" library="supply1" deviceset="+3V3" device=""/>
+<part name="PCB1" library="e14_Rpi3_RevA+mirror-pcb" deviceset="RPI3" device="RPI3"/>
 </parts>
 <sheets>
@@
 <attribute name="VALUE" x="-7.62" y="68.326" size="1.778" layer="96" rot="R90"/>
 </instance>
+<instance part="PCB1" gate="G$1" x="355.6" y="-203.2" smashed="yes"/>
 </instances>
 <busses>

Commit message: sync
Parts:
- added U1: ESP32-WROOM-32D, ESP32-WROOM-32D:ESP32-WROOM-32D
Changed lines of the file:
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@@
 <part name="+3V5" library="supply1" deviceset="+3V3" device=""/>
 <part name="PCB1" library="e14_Rpi3_RevA+mirror-pcb" deviceset="RPI3" device="RPI3"/>
+<part name="U1" library="ESP32-WROOM-32D" deviceset="ESP32-WROOM-32D" device=""/>
 </parts>
 <sheets>
@@
 </instance>
 <instance part="PCB1" gate="G$1" x="355.6" y="-203.2" smashed="yes"/>
+<instance part="U1" gate="G$1" x="254" y="-149.86" smashed="yes">
+<attribute name="NAME" x="238.9641" y="-113.1855" size="1.783840625" layer="95"/>
+<attribute name="VALUE" x="238.7133" y="-188.0681" size="1.78345" layer="96"/>
+</instance>
 </instances>
 <busses>

Commit message: sync
Parts:
- removed GND: UART, con-lsta:FE05-1
- removed PCB1: RPI3RPI3, e14_Rpi3_RevA+mirror-pcb:RPI3RPI3
- removed RASPBERRYPI: (no value), con-lsta:FE06-2
- removed SJ1: SOLDERJUMPERNO, SparkFun:SOLDERJUMPERNO
- added C10, C11, C7: 100nF, rcl:C-EUC0603
- added C12: 2.2uF, rcl:C-EUC0603
- added FB4: FBCHIP-0603(1608-METRIC), Filter:FBCHIP-0603(1608-METRIC)
- added IC1: CP2102, silabs:CP2102
- added J1: CONN_12X2, SparkFun-Connectors:CONN_12X2
- added JP1: PINHD-1X2, Connector:PINHD-1X2
- added JP2: UART_STM, Connector:PINHD-1X6
- added R5, R6, R7: (no value), rcl:R-EU_0207/10
- added SMA: 5-1814400-1, 5-1814400-1 sma connector:5-1814400-1
- added U$2: RFM12_SMDSMD, rfm12b _ rfm69cw:RFM12_SMDSMD
- CF1, CF2, CF3, CFV: value 100nF -> 10nF; device resistor:C-EUC0603 -> rcl:C-EUC0805
- RB2, RB3: value 22r -> 6R8
- RF1, RF2, RF3, RFV: value 330R -> 9k1
Connections:
- new net +3V3RPI: J1.1, J1.17
- new net AGND: C1.2, C22.2, FB4.1, STM32.VSSA/VREF-
- new net CLK_RPI: J1.23
- new net CS_RPI: J1.24
- new net D+: IC1.D+, U$10.D+
- new net D-: IC1.D-, U$10.D-
- new net ESP_BOOT0: U1.IO0
- new net ESP_RST: U1.EN
- new net ESP_RX: U1.RXD0
- new net ESP_TX: U1.TXD0
- new net MISO_RPI: J1.21
- new net MOSI_RPI: J1.19
- new net N$11: U$2.!SEL
- new net N$13: U$2.!IRQ
- new net N$14: U$2.SDI
- new net N$15: U$2.SDO
- new net N$16: U$2.SCK
- new net N$17: U$2.!RES
- new net N$18: SMA.1, U$2.ANT
- new net N$19: JP2.5
- new net N$5: J1.9
- new net SCL: J1.5, STM32.PB8, U1.IO22
- new net SDA: J1.3, STM32.PB9, U1.IO21
- new net SPI3_CLK: STM32.PB3
- new net SPI3_MISO: STM32.PB4
- new net SPI3_MOSI: STM32.PB5
- new net SPI3_NSS: STM32.PA15
- new net STM_RX: J1.8, JP2.2, STM32.PA10
- new net STM_TX: J1.10, JP2.3, STM32.PA9
- net +3V3: now also C11.1, IC1.VDD, U$2.VDD, U1.3V3; no longer C5.1, SJ1.2, STM32.VDDA/VREF+
- net +3V3ANA: now also STM32.VDDA/VREF+
- net +5V: now also C10.1, C12.1, IC1.REGIN, IC1.VBUS, J1.2, J1.4, JP2.4; no longer GND.3, RASPBERRYPI.1, RASPBERRYPI.3
- net BIAS: now also R5.2, R6.2, R7.2
- net BIAS_IN: now also C5.1
- net BOOT0: now also IC1.DTR, J1.7; no longer RASPBERRYPI.8
- net CT1: now also STM32.PB12; no longer STM32.PA0
- net CT2: now also CF2.1, STM32.PB14; no longer CF2.2, STM32.PA1
- net CT3: now also CF3.1, STM32.PB15; no longer CF3.2, STM32.PA2
- net GND: now also C10.2, C11.2, C12.2, C7.2, CF2.2, CF3.2, FB4.2, IC1.GND, IC1.GND@EXP, IC1.GND@M, J1.14, J1.20, J1.6, JP2.6, SMA.2, SMA.3, SMA.4, SMA.5, U$2.GND, U$2.GND@1, U1.GND; no longer C1.2, C22.2, CF2.1, CF3.1, GND.1, RASPBERRYPI.10, RASPBERRYPI.5, STM32.VSSA/VREF-
- net LED: now also STM32.PB6; no longer STM32.PB14
- net N$1: now also IC1.!RST; no longer GND.2, SJ1.1
- net N$10: now also R7.1
- net N$2: now also R5.1
- net N$8: now also R6.1
- net PULSE: now also C7.1, STM32.PB7; no longer STM32.PB15
- net RST_STM: now also IC1.RTS, J1.11, JP2.1; no longer RASPBERRYPI.12
- net UART_RX: now also IC1.TXD, JP1.1; no longer GND.4, RASPBERRYPI.7, STM32.PA10
- net UART_TX: now also IC1.RXD, JP1.2; no longer GND.5, RASPBERRYPI.9, STM32.PA9
- net VSIG: now also STM32.PB2; no longer STM32.PB12
Other:
- note added: "STM32 VDD/VSS Decoupling Capacitors"
- note removed: "5V"
- note removed: "VDD/VSS Decoupling Capacitors"
- moved on the sheet: C1, C18, C2, C22, C5, CF1, CF2, CF3, CFV, CT1, CT2, CT3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

Commit message: sync
Parts:
- removed C7: 100nF, rcl:C-EUC0603
- added C13: 100nF, rcl:C-EUC0603
- added C17: 2.2uF, rcl:C-EUC0603
- added JP10, JP3, JP4, JP5, JP6, JP7, JP8, JP9: JUMPER-SMT_2_NC_TRACE_NO-SILK, SparkFun-Jumpers:JUMPER-SMT_2_NC_TRACE_NO-SILK
- added R8: 10k, rcl:R-EU_R0603
Connections:
- removed net CLK_RPI: J1.23
- removed net CS_RPI: J1.24
- removed net N$11: U$2.!SEL
- removed net N$13: U$2.!IRQ
- removed net N$14: U$2.SDI
- removed net N$15: U$2.SDO
- removed net N$16: U$2.SCK
- removed net N$17: U$2.!RES
- new net ESP_CLK: JP7.1, U1.IO18
- new net ESP_CS: JP10.1, U1.IO5
- new net ESP_MISO: JP8.1, U1.IO19
- new net ESP_MOSI: JP9.1, U1.IO23
- new net RFM_IRQ: STM32.PA1, U$2.!IRQ
- new net RFM_RST: STM32.PA2, U$2.!RES
- new net RPI_CLK: J1.23, JP5.2, JP7.2
- new net RPI_CONNECTED: R8.2, STM32.PC13, U1.IO15
- new net RPI_CONNECTED_PR: J1.17, R8.1
- new net RPI_CS: J1.24, JP10.2, JP6.1
- new net RPI_MISO: JP8.2
- new net RPI_MOSI: JP9.2
- net +3V3: now also C13.1, C17.1; no longer R22.2
- net +3V3ANA: now also R22.2
- net +3V3RPI: no longer J1.17
- net GND: now also C13.2, C17.2; no longer C7.2
- net MISO_RPI: now also JP4.2
- net MOSI_RPI: now also JP3.2
- net PULSE: no longer C7.1
- net SPI3_CLK: now also JP5.1, U$2.SCK
- net SPI3_MISO: now also JP4.1, U$2.SDO
- net SPI3_MOSI: now also JP3.1, U$2.SDI
- net SPI3_NSS: now also JP6.2, U$2.!SEL
Other:
- moved on the sheet: J1

Commit message: sync mini v0.2
Parts:
- removed FB3: FBCHIP-0603(1608-METRIC), Filter:FBCHIP-0603(1608-METRIC)
- removed JP5: JUMPER-SMT_2_NC_TRACE_NO-SILK, SparkFun-Jumpers:JUMPER-SMT_2_NC_TRACE_NO-SILK
- added JP11, JP12: JUMPER-SMT_2_NC_TRACE_NO-SILK, SparkFun-Jumpers:JUMPER-SMT_2_NC_TRACE_NO-SILK
- added R9: 10k, rcl:R-EU_R0603
- C2: value 100nF -> 2.2uF
- R8: value 10k -> 120k
Connections:
- removed net GND_USB: FB3.2, U$10.GND, U$10.MTN1, U$10.MTN2, U$10.MTN3, U$10.MTN4
- removed net MISO_RPI: J1.21, JP4.2
- removed net MOSI_RPI: J1.19, JP3.2
- removed net RPI_CLK: J1.23, JP5.2, JP7.2
- removed net SPI3_CLK: JP5.1, STM32.PB3, U$2.SCK
- removed net UART_RX: IC1.TXD, JP1.1
- removed net UART_TX: IC1.RXD, JP1.2
- new net CP2102_RX: IC1.RXD, JP1.1, JP11.1
- new net CP2102_TX: IC1.TXD, JP1.2, JP12.1
- new net SPI_CLK: J1.23, JP7.2, STM32.PB3, U$2.SCK
- net ESP_RX: now also JP12.2
- net ESP_TX: now also JP11.2
- net GND: now also R9.1, U$10.GND, U$10.MTN1, U$10.MTN2, U$10.MTN3, U$10.MTN4; no longer FB3.1
- net NRST: no longer STLINK.3
- net RPI_CONNECTED: now also R9.2
- net RPI_MISO: now also J1.21, JP4.2
- net RPI_MOSI: now also J1.19, JP3.2
- net RST_STM: now also STLINK.3
Other:
- moved on the sheet: STLINK
