File: Hardware/stm32-pi_basic/7/stm32hw07.brd (EAGLE design)
At the start: 71.5 x 74 mm, 75 parts, among them IC1 CP2102, J1 CONN_12X2, U1 ESP32-WROOM-32D

Commit message: sync
Parts:
- added BOOT1: (no value), SparkFun:1X02
- added R10: 10k, resistor:R0603
Connections:
- removed net LSE_IN: STM32.3
- removed net LSE_OUT: STM32.4
- new net HSE_IN_: C14.1, HSE.1, R10.1
- net GND: now also BOOT1.2
- net HSE_IN: now also R10.2; no longer C14.1, HSE.1
- net NRST: now also BOOT1.1
Routing:
- net HSE_IN: track 10.9 -> 2.40 mm
- net HSE_IN_: track 0.00 -> 7.11 mm

Commit message: sync, raido tested
Other:
- board text added: "PULSE"
Changed lines of the file:
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@@
 <layer number="14" name="Route14" color="1" fill="6" visible="no" active="no"/>
 <layer number="15" name="Route15" color="4" fill="6" visible="no" active="no"/>
-<layer number="16" name="Bottom" color="1" fill="1" visible="yes" active="yes"/>
+<layer number="16" name="Bottom" color="1" fill="1" visible="no" active="yes"/>
 <layer number="17" name="Pads" color="2" fill="1" visible="yes" active="yes"/>
 <layer number="18" name="Vias" color="2" fill="1" visible="yes" active="yes"/>
@@
 <layer number="110" name="fp0" color="7" fill="1" visible="no" active="yes"/>
 <layer number="111" name="LPC17xx" color="7" fill="1" visible="no" active="yes"/>
-<layer number="112" name="tSilk" color="7" fill="1" visible="yes" active="yes"/>
+<layer number="112" name="tSilk" color="7" fill="1" visible="no" active="yes"/>
 <layer number="113" name="IDFDebug" color="4" fill="1" visible="no" active="yes"/>
 <layer number="114" name="Route14" color="7" fill="1" visible="no" active="no"/>
@@
 <wire x1="43.482753125" y1="53.1352625" x2="42.738803125" y2="51.339209375" width="0.508" layer="42" curve="45.00007"/>
 <wire x1="42.738803125" y1="51.339209375" x2="42.738803125" y2="48.560228125" width="0.508" layer="42"/>
+<text x="36.953365625" y="8.771184375" size="0.8128" layer="21" font="vector" ratio="20" rot="R90">PULSE</text>
+<text x="13.727" y="15.73270625" size="0.8128" layer="21" font="vector" ratio="20" rot="R270">DS18B20</text>
 </plain>
 <attributes>
@@
 <attribute name="NAME" x="42.095746875" y="76.3895" size="1.27" layer="25" rot="R270"/>
 </element>
-<element name="RB1" library="resistor" package="R0603" value="22r" x="47.33749375" y="61.487934375" smashed="yes">
-<attribute name="NAME" x="45.58749375" y="60.487934375" size="0.8128" layer="25" font="vector" ratio="20" rot="R90"/>
-</element>
+<element name="RB1" library="resistor" package="R0603" value="22r" x="47.33749375" y="61.487934375" smashed="yes"/>
 <element name="RF1" library="resistor" package="R0603" value="9k1" x="30.245315625" y="57.08205625" smashed="yes" rot="R180">
 <attribute name="NAME" x="28.745315625" y="58.08205625" size="0.8128" layer="25" font="vector" ratio="20"/>
@@
 <attribute name="NAME" x="29.322746875" y="76.3895" size="1.27" layer="25" rot="R270"/>
 </element>
-<element name="RB2" library="resistor" package="R0603" value="6R8" x="34.622996875" y="61.487934375" smashed="yes">
-<attribute name="NAME" x="32.0911875" y="58.923040625" size="0.8128" layer="25" font="vector" ratio="20" rot="R90"/>
-</element>
+<element name="RB2" library="resistor" package="R0603" value="6R8" x="34.622996875" y="61.487934375" smashed="yes"/>
 <element name="RF2" library="resistor" package="R0603" value="9k1" x="25.67895" y="57.08205625" smashed="yes" rot="R180">
 <attribute name="NAME" x="24.17895" y="58.08205625" size="0.8128" layer="25" font="vector" ratio="20"/>
@@
 <attribute name="NAME" x="16.549746875" y="76.3895" size="1.27" layer="25" rot="R270"/>
 </element>
-<element name="RB3" library="resistor" package="R0603" value="6R8" x="21.933640625" y="61.487934375" smashed="yes">
-<attribute name="NAME" x="20.183640625" y="60.487934375" size="0.8128" layer="25" font="vector" ratio="20" rot="R90"/>
-</element>
+<element name="RB3" library="resistor" package="R0603" value="6R8" x="21.933640625" y="61.487934375" smashed="yes"/>
 <element name="RF3" library="resistor" package="R0603" value="9k1" x="21.112584375" y="57.08205625" smashed="yes" rot="R180">
 <attribute name="NAME" x="19.612584375" y="58.08205625" size="0.8128" layer="25" font="vector" ratio="20"/>
@@
 </element>
 <element name="R5" library="rcl" library_urn="urn:adsk.eagle:library:334" package="0207/10" package3d_urn="urn:adsk.eagle:package:23491/2" value="" x="47.23638125" y="61.487934375" smashed="yes">
-<attribute name="NAME" x="44.06138125" y="62.884934375" size="1.27" layer="25" ratio="10"/>
+<attribute name="NAME" x="49.064675" y="63.070353125" size="1.27" layer="25" ratio="10"/>
 <attribute name="POPULARITY" value="81" x="47.23638125" y="61.487934375" size="1.778" layer="27" display="off"/>
 <attribute name="SPICEPREFIX" value="R" x="47.23638125" y="61.487934375" size="1.778" layer="27" display="off"/>
@@
 </element>
 <element name="R6" library="rcl" library_urn="urn:adsk.eagle:library:334" package="0207/10" package3d_urn="urn:adsk.eagle:package:23491/2" value="" x="34.610553125" y="61.487934375" smashed="yes">
-<attribute name="NAME" x="31.435553125" y="62.884934375" size="1.27" layer="25" ratio="10"/>
+<attribute name="NAME" x="36.207196875" y="62.9311625" size="1.27" layer="25" ratio="10"/>
 <attribute name="POPULARITY" value="81" x="34.610553125" y="61.487934375" size="1.778" layer="27" display="off"/>
 <attribute name="SPICEPREFIX" value="R" x="34.610553125" y="61.487934375" size="1.778" layer="27" display="off"/>
@@
 </element>
 <element name="R7" library="rcl" library_urn="urn:adsk.eagle:library:334" package="0207/10" package3d_urn="urn:adsk.eagle:package:23491/2" value="" x="21.814540625" y="61.487934375" smashed="yes">
-<attribute name="NAME" x="18.639540625" y="62.884934375" size="1.27" layer="25" ratio="10"/>
+<attribute name="NAME" x="23.411184375" y="62.9311625" size="1.27" layer="25" ratio="10"/>
 <attribute name="POPULARITY" value="81" x="21.814540625" y="61.487934375" size="1.778" layer="27" display="off"/>
 <attribute name="SPICEPREFIX" value="R" x="21.814540625" y="61.487934375" size="1.778" layer="27" display="off"/>

Commit message: sync
Parts:
- added C7: 22uF, rcl:C0805
- added U$3: 47219-2001_MICROSD, MOLEX 47219-2001:47219-2001_MICROSD
- moved SMA 0.87 mm to (73.5, 59.7)
Connections:
- new net MICROSD_CS: U$3.PIN2, U1.16
- net +3V3: now also C7.1, U$3.PIN4
- net BOOT0: no longer IC1.28
- net ESP_BOOT0: now also IC1.23
- net ESP_CLK: now also U$3.PIN5
- net ESP_MISO: now also U$3.PIN7
- net ESP_MOSI: now also U$3.PIN3
- net ESP_RST: now also IC1.24
- net GND: now also C7.2, U$3.P$1, U$3.P$2, U$3.P$3, U$3.P$4, U$3.PIN6
- net RPI_CONNECTED: now also U1.13; no longer U1.23
- net RPI_MISO: now also JP3.2; no longer JP4.2
- net RPI_MOSI: now also JP4.2; no longer JP3.2
- net RST_STM: no longer IC1.24
- net STM_RX: now also U1.28
- net STM_TX: now also U1.27
Routing:
- net +3V3: track 219.4 -> 233.9 mm
- net RPI_MOSI: track 42.5 -> 38.7 mm
- net RPI_CONNECTED: track 72.5 -> 71.0 mm
- net ESP_RST: track 0.00 -> 1.18 mm
- net RST_STM: track 88.6 -> 87.6 mm
- net BOOT0: track 75.2 -> 74.2 mm
- net N$18: track 12.0 -> 12.9 mm

Commit message: sync
Parts:
- removed FB4: FBCHIP-0603(1608-METRIC), Filter:BEADC1608X95N
- removed HSE: 8MHZ, crystal:CTS406
- removed JP1: PINHD-1X2, Connector:1X02
- removed JP10, JP11, JP12, JP3, JP4, JP7, JP8, JP9: JUMPER-SMT_2_NC_TRACE_NO-SILK, SparkFun-Jumpers:SMT-JUMPER_2_NC_TRACE_NO-SILK
- removed U$10: USB-MINIB-5PIN, Ciseco USB miniB_Updated:USB-MINIB-CISECO
- added 5VUSB: (no value), adafruit:USB-MINIB-THM-MOLEX
- added LED2: (no value), led:CHIP-LED0805
- added PAD1, PAD2, PAD3, PAD4: (no value), wirepad:1,6/0,8
- added Q1, Q2: (no value), microbuilder:SOT23-R
- added Q3: (no value), adafruit:NX3225
- added R11: 10k, resistor:R0603
- added R12: 510R, resistor:R0603
- added R13: 0R, resistor:R0603
- added U2: (no value), microbuilder:SOT23-WIDE
- FB1, FB2: value FBCHIP-0603(1608-METRIC) -> 0R
- R9: device rcl:R0603 -> resistor:R0603
- moved LOGO1 54.0 mm to (53.7, 58.7)
- moved R9 5.72 mm to (51.8, 25.0), turned to 0 degrees
- moved C14 1.40 mm to (27.4, 32.1)
- moved FB2 1.27 mm to (35.3, 44.7)
- moved C15 0.88 mm to (32.7, 37.0)
- moved R23 0.66 mm to (32.8, 49.4)
- moved C5 0.64 mm to (34.9, 48.2)
- moved C18 0.48 mm to (30.7, 48.5)
- moved C2 0.45 mm to (23.8, 28.6), turned to 180 degrees
- moved R22 0.21 mm to (33.2, 45.9)
- moved R8 0.18 mm to (44.0, 23.5)
Connections:
- removed net CP2102_RX: IC1.25, JP1.1, JP11.1
- removed net CP2102_TX: IC1.26, JP1.2, JP12.1
- removed net ESP_CLK: JP7.1, U$3.PIN5, U1.30
- removed net ESP_CS: JP10.1, U1.29
- removed net ESP_MISO: JP8.1, U$3.PIN7, U1.31
- removed net ESP_MOSI: JP9.1, U$3.PIN3, U1.37
- removed net ESP_RST: IC1.24, U1.3
- removed net RPI_CS: J1.24, JP10.2, JP6.1
- removed net RPI_MISO: J1.21, JP3.2, JP8.2
- removed net RPI_MOSI: J1.19, JP4.2, JP9.2
- removed net SPI3_MISO: JP4.1, STM32.40, U$2.1
- removed net SPI3_MOSI: JP3.1, STM32.41, U$2.12
- new net CP2102_DTR: IC1.28, Q1.2, R9.2
- new net CP2102_RTS: IC1.24, Q2.2, R11.2
- new net ESP_EN: PAD1.1, Q2.3, U1.3
- new net G1: Q3.4
- new net G2: Q3.2
- new net MISO: J1.21, STM32.40, U$2.1, U$3.PIN7, U1.31
- new net MOSI: J1.19, STM32.41, U$2.12, U$3.PIN3, U1.37
- new net N$11: J1.13
- new net N$13: LED2.A, R12.1
- new net N$6: Q2.1, R9.1
- new net N$7: Q1.1, R11.1
- new net N$9: J1.15
- new net RPI|ESP_CS: J1.24, JP6.1, U1.29
- net +3V3: now also U2.2
- net +5V: now also R12.2; no longer J1.2, J1.4
- net +5V_EXT: now also 5VUSB.VBUS, J1.2, J1.4; no longer U$10.VBUS
- net AGND: now also C18.2, C5.2, CF1.2, CF2.2, CF3.2, CFV.2, R13.1, R23.1, U2.1; no longer FB4.1
- net BIAS: now also U2.3
- net D+: now also 5VUSB.D+; no longer U$10.D+
- net D-: now also 5VUSB.D-; no longer U$10.D-
- net ESP_BOOT0: now also PAD2.1, Q1.3; no longer IC1.23
- net ESP_RX: now also IC1.26, PAD3.1; no longer JP12.2
- net ESP_TX: now also IC1.25, PAD4.1; no longer JP11.2
- net GND: now also 5VUSB.GND, LED2.C, MCP1825.4, R13.2; no longer C18.2, C5.2, CF1.2, CF2.2, CF3.2, CFV.2, FB4.2, R23.1, R9.1, U$10.GND, U$10.MTN1, U$10.MTN2, U$10.MTN3, U$10.MTN4
- net HSE_IN_: now also Q3.3; no longer HSE.1
- net HSE_OUT: now also Q3.1; no longer HSE.3
- net RFM_IRQ: now also J1.16
- net RFM_RST: now also J1.18
- net RPI_CONNECTED: now also U1.26; no longer R9.2, U1.13
- net SPI_CLK: now also U$3.PIN5, U1.30; no longer JP7.2
Routing:
- net MOSI: track 0.00 -> 115.4 mm, vias 0 -> 8
- net MISO: track 0.00 -> 86.6 mm, vias 0 -> 9
- net SPI3_MOSI: track 72.0 -> 0.00 mm, vias 5 -> 0
- net STM_TX: track 115.8 -> 167.2 mm, vias 4 -> 8
- net STM_RX: track 125.2 -> 176.3 mm, vias 3 -> 7
- net SPI3_MISO: track 50.9 -> 0.00 mm, vias 5 -> 0
- net ESP_EN: track 0.00 -> 46.4 mm, vias 0 -> 2
- net RFM_RST: track 26.7 -> 67.9 mm, vias 3 -> 6
- net RPI|ESP_CS: track 0.00 -> 40.2 mm, vias 0 -> 1
- net RPI_MOSI: track 38.7 -> 0.00 mm, vias 3 -> 0
- net RPI_CS: track 37.2 -> 0.00 mm, vias 1 -> 0
- net RPI_MISO: track 37.1 -> 0.00 mm, vias 3 -> 0
- net RFM_IRQ: track 26.5 -> 62.4 mm, vias 5 -> 9
- net SPI_CLK: track 89.2 -> 124.7 mm, vias 5 -> 8
- net CP2102_TX: track 28.1 -> 0.00 mm, vias 1 -> 0
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- added copper zone on layer 1, net AGND
- added copper zone on layer 16, net AGND
Other:
- board text added: "by DB"
- board text added: "v0.3"
- board text removed: "v0.2"

Commit message: sync
Parts:
- removed Q3: (no value), adafruit:NX3225
- added Y1: (no value), adafruit:NX3225
- moved 5VUSB 9.37 mm to (56.3, -2.37)
- moved C1 9.37 mm to (21.8, 32.8)
- moved C10 9.37 mm to (53.5, 20.2)
- moved C11 9.37 mm to (53.4, 16.9)
- moved C14 9.37 mm to (20.4, 25.8)
- moved C3 9.37 mm to (45.6, 4.26)
- moved C5 9.37 mm to (27.9, 42.0)
- moved C6 9.37 mm to (9.84, 38.1)
- moved C8 9.37 mm to (18.5, 41.8)
- moved CF1 9.37 mm to (23.3, 47.8)
- moved CF2 9.37 mm to (18.7, 47.8)
- moved CF3 9.37 mm to (14.2, 47.8)
- moved CFV 9.37 mm to (27.9, 47.8)
- moved CT1 9.37 mm to (39.6, 74.6)
- moved CT2 9.37 mm to (26.9, 74.6)
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Connections:
- net G1: now also Y1.4; no longer Q3.4
- net G2: now also Y1.2; no longer Q3.2
- net HSE_IN_: now also Y1.3; no longer Q3.3
- net HSE_OUT: now also Y1.1; no longer Q3.1
Routing:
- net +5V: track 148.1 -> 150.8 mm
- net HSE_IN_: track 8.86 -> 6.68 mm
- net +3V3ANA: track 15.7 -> 16.4 mm
- net RFM_RST: track 67.9 -> 68.5 mm
- net +5V_EXT: track 7.42 -> 7.98 mm
- net AGND: track 56.0 -> 55.7 mm, vias 23 -> 24
Other:
- board size 71.5 x 74 mm -> 71.4 x 74 mm
- board text added: "74.04 y axis 71.39 x axis"
