File: Hardware/stm32-pi_basic/7/stm32hw07.sch (EAGLE design)
At the start: 74 parts, among them IC1 CP2102, J1 CONN_12X2, U1 ESP32-WROOM-32D

Commit message: sync
Parts:
- added BOOT1: (no value), SparkFun:M02PTH
- added R10: 10k, resistor:R-EU_R0603
Connections:
- removed net LSE_IN: STM32.PC14-OSC32_IN
- removed net LSE_OUT: STM32.PC15-OSC_OUT
- new net HSE_IN_: C14.1, HSE.1, R10.1
- net GND: now also BOOT1.2
- net HSE_IN: now also R10.2; no longer C14.1, HSE.1
- net NRST: now also BOOT1.1
Changed lines of the file:
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@@
 <part name="R9" library="rcl" deviceset="R-EU_" device="R0603" value="10k"/>
 <part name="GND2" library="supply1" deviceset="GND" device=""/>
+<part name="BOOT1" library="SparkFun" deviceset="M02" device="PTH"/>
+<part name="SUPPLY2" library="supply2" deviceset="GND" device=""/>
+<part name="R10" library="resistor" deviceset="R-EU_" device="R0603" value="10k"/>
 </parts>
 <sheets>
@@
 <text x="-53.34" y="129.54" size="3.81" layer="91">STM32</text>
 <text x="-53.34" y="215.9" size="2.54" layer="91">Open Source Hardware: GNU General Public Licence v3</text>
-<text x="24.13" y="104.14" size="1.778" layer="91" rot="R90">Frequency 8MHZ to 32MHZ</text>
+<text x="21.59" y="106.68" size="1.778" layer="91" rot="R90">Frequency 8MHZ to 32MHZ</text>
 </plain>
 <instances>
@@
 <instance part="GND2" gate="1" x="75.692" y="-49.022" smashed="yes">
 <attribute name="VALUE" x="73.152" y="-51.562" size="1.778" layer="96"/>
+</instance>
+<instance part="BOOT1" gate="G$1" x="21.59" y="87.63" smashed="yes" rot="R270">
+<attribute name="VALUE" x="16.51" y="90.17" size="1.778" layer="96" rot="R270"/>
+<attribute name="NAME" x="27.432" y="90.17" size="1.778" layer="95" rot="R270"/>
+</instance>
+<instance part="SUPPLY2" gate="GND" x="33.02" y="73.66" smashed="yes">
+<attribute name="VALUE" x="31.115" y="70.485" size="1.778" layer="96"/>
+</instance>
+<instance part="R10" gate="G$1" x="27.94" y="127" smashed="yes" rot="R90">
+<attribute name="NAME" x="26.4414" y="123.19" size="1.778" layer="95" rot="R90"/>
+<attribute name="VALUE" x="31.242" y="123.19" size="1.778" layer="96" rot="R90"/>
 </instance>
 </instances>
@@
 <pinref part="GND2" gate="1" pin="GND"/>
 </segment>
+<segment>
+<pinref part="BOOT1" gate="G$1" pin="2"/>
+<wire x1="24.13" y1="80.01" x2="33.02" y2="80.01" width="0.1524" layer="91"/>
+<wire x1="33.02" y1="80.01" x2="33.02" y2="76.2" width="0.1524" layer="91"/>
+<pinref part="SUPPLY2" gate="GND" pin="GND"/>
+</segment>
 </net>
 <net name="+5V" class="0">
@@
 <wire x1="10.16" y1="76.2" x2="12.7" y2="76.2" width="0.1524" layer="91"/>
 <label x="12.7" y="76.2" size="1.778" layer="95" xref="yes"/>
+<pinref part="BOOT1" gate="G$1" pin="1"/>
+<wire x1="12.7" y1="76.2" x2="12.7" y2="80.01" width="0.1524" layer="91"/>
+<wire x1="12.7" y1="80.01" x2="21.59" y2="80.01" width="0.1524" layer="91"/>
 </segment>
 </net>
@@
 <net name="HSE_IN" class="0">
 <segment>
-<pinref part="C14" gate="G$1" pin="1"/>
-<wire x1="27.94" y1="114.3" x2="27.94" y2="119.38" width="0.1524" layer="91"/>
-<pinref part="HSE" gate="G$1" pin="1"/>
-<wire x1="27.94" y1="119.38" x2="30.48" y2="119.38" width="0.1524" layer="91"/>
-<wire x1="27.94" y1="119.38" x2="27.94" y2="129.54" width="0.1524" layer="91"/>
-<label x="27.94" y="129.54" size="1.778" layer="95" rot="R90"/>
-<junction x="27.94" y="119.38"/>
-</segment>
-<segment>
 <pinref part="STM32" gate="A" pin="PF0-OSC_IN"/>
 <wire x1="68.58" y1="91.44" x2="63.5" y2="91.44" width="0.1524" layer="91"/>
 <label x="63.5" y="91.44" size="1.27" layer="95" rot="R180" xref="yes"/>
+</segment>
+<segment>
+<wire x1="27.94" y1="132.08" x2="27.94" y2="134.62" width="0.1524" layer="91"/>
+<label x="27.94" y="134.62" size="1.778" layer="95" rot="R90"/>
+<pinref part="R10" gate="G$1" pin="2"/>
 </segment>
 </net>
@@
 <wire x1="124.46" y1="88.9" x2="132.08" y2="88.9" width="0.1524" layer="91"/>
 <label x="132.08" y="88.9" size="1.27" layer="95" xref="yes"/>
-</segment>
-</net>
-<net name="LSE_IN" class="0">
-<segment>
-<pinref part="STM32" gate="A" pin="PC14-OSC32_IN"/>
-<wire x1="68.58" y1="96.52" x2="63.5" y2="96.52" width="0.1524" layer="91"/>
-<label x="63.5" y="96.52" size="1.27" layer="95" rot="R180" xref="yes"/>
-</segment>
-</net>
-<net name="LSE_OUT" class="0">
-<segment>
-<pinref part="STM32" gate="A" pin="PC15-OSC_OUT"/>
-<wire x1="68.58" y1="93.98" x2="63.5" y2="93.98" width="0.1524" layer="91"/>
-<label x="63.5" y="93.98" size="1.27" layer="95" rot="R180" xref="yes"/>
 </segment>
 </net>
@@
 </segment>
 </net>
+<net name="HSE_IN_" class="0">
+<segment>
+<pinref part="C14" gate="G$1" pin="1"/>
+<wire x1="27.94" y1="114.3" x2="27.94" y2="119.38" width="0.1524" layer="91"/>
+<pinref part="HSE" gate="G$1" pin="1"/>
+<wire x1="27.94" y1="119.38" x2="30.48" y2="119.38" width="0.1524" layer="91"/>
+<junction x="27.94" y="119.38"/>
+<wire x1="27.94" y1="119.38" x2="27.94" y2="121.92" width="0.1524" layer="91"/>
+<pinref part="R10" gate="G$1" pin="1"/>
+</segment>
+</net>

Commit message: sync, raido tested
Other:
- note added: "todo: . Protection Diode"
Changed lines of the file:
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@@
 <text x="-53.34" y="215.9" size="2.54" layer="91">Open Source Hardware: GNU General Public Licence v3</text>
 <text x="21.59" y="106.68" size="1.778" layer="91" rot="R90">Frequency 8MHZ to 32MHZ</text>
+<text x="210.82" y="-22.86" size="6.4516" layer="91">todo:
+. Protection Diode</text>
 </plain>
 <instances>

Commit message: sync
Parts:
- added C7: 22uF, rcl:C-EUC0805
- added U$3: 47219-2001_MICROSD, MOLEX 47219-2001:47219-2001_MICROSD
Connections:
- new net MICROSD_CS: U$3.CD/DAT3, U1.IO13
- net +3V3: now also C7.1, U$3.VDD
- net BOOT0: no longer IC1.DTR
- net ESP_BOOT0: now also IC1.CTS
- net ESP_CLK: now also U$3.CLK
- net ESP_MISO: now also U$3.DAT0
- net ESP_MOSI: now also U$3.CMD
- net ESP_RST: now also IC1.RTS
- net GND: now also C7.2, U$3.GND, U$3.VSS
- net RPI_CONNECTED: now also U1.IO14; no longer U1.IO15
- net RPI_MISO: now also JP3.2; no longer JP4.2
- net RPI_MOSI: now also JP4.2; no longer JP3.2
- net RST_STM: no longer IC1.RTS
- net STM_RX: now also U1.IO17
- net STM_TX: now also U1.IO16
Changed lines of the file:
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@@
 <part name="SUPPLY2" library="supply2" deviceset="GND" device=""/>
 <part name="R10" library="resistor" deviceset="R-EU_" device="R0603" value="10k"/>
+<part name="C7" library="rcl" library_urn="urn:adsk.eagle:library:334" deviceset="C-EU" device="C0805" package3d_urn="urn:adsk.eagle:package:23617/2" value="22uF"/>
+<part name="SUPPLY17" library="supply2" deviceset="GND" device=""/>
+<part name="U$3" library="MOLEX 47219-2001" deviceset="47219-2001_MICROSD" device=""/>
+<part name="SUPPLY18" library="supply2" deviceset="GND" device=""/>
 </parts>
 <sheets>
@@
 <attribute name="VALUE" x="31.242" y="123.19" size="1.778" layer="96" rot="R90"/>
 </instance>
+<instance part="C7" gate="G$1" x="292.1" y="-109.22" smashed="yes">
+<attribute name="NAME" x="293.624" y="-108.839" size="1.778" layer="95"/>
+<attribute name="VALUE" x="293.624" y="-113.919" size="1.778" layer="96"/>
+</instance>
+<instance part="SUPPLY17" gate="GND" x="299.72" y="-121.92" smashed="yes">
+<attribute name="VALUE" x="297.815" y="-125.095" size="1.778" layer="96"/>
+</instance>
+<instance part="U$3" gate="G$1" x="-17.78" y="-121.92" smashed="yes"/>
+<instance part="SUPPLY18" gate="GND" x="-25.4" y="-129.54" smashed="yes">
+<attribute name="VALUE" x="-27.305" y="-132.715" size="1.778" layer="96"/>
+</instance>
 </instances>
 <busses>
@@
 <pinref part="SUPPLY2" gate="GND" pin="GND"/>
 </segment>
+<segment>
+<pinref part="C7" gate="G$1" pin="2"/>
+<wire x1="292.1" y1="-114.3" x2="292.1" y2="-116.84" width="0.1524" layer="91"/>
+<wire x1="292.1" y1="-116.84" x2="299.72" y2="-116.84" width="0.1524" layer="91"/>
+<wire x1="299.72" y1="-116.84" x2="299.72" y2="-119.38" width="0.1524" layer="91"/>
+<pinref part="SUPPLY17" gate="GND" pin="GND"/>
+</segment>
+<segment>
+<pinref part="U$3" gate="G$1" pin="GND"/>
+<wire x1="-20.32" y1="-119.38" x2="-25.4" y2="-119.38" width="0.1524" layer="91"/>
+<wire x1="-25.4" y1="-119.38" x2="-25.4" y2="-127" width="0.1524" layer="91"/>
+<pinref part="SUPPLY18" gate="GND" pin="GND"/>
+<pinref part="U$3" gate="G$1" pin="VSS"/>
+<wire x1="5.08" y1="-114.3" x2="-25.4" y2="-114.3" width="0.1524" layer="91"/>
+<wire x1="-25.4" y1="-114.3" x2="-25.4" y2="-119.38" width="0.1524" layer="91"/>
+<junction x="-25.4" y="-119.38"/>
+</segment>
 </net>
 <net name="+5V" class="0">
@@
 <pinref part="U1" gate="G$1" pin="3V3"/>
 <wire x1="271.78" y1="-116.84" x2="279.4" y2="-116.84" width="0.1524" layer="91"/>
-<wire x1="279.4" y1="-116.84" x2="279.4" y2="-111.76" width="0.1524" layer="91"/>
-<label x="279.4" y="-111.76" size="1.27" layer="95" xref="yes"/>
+<label x="279.4" y="-101.6" size="1.27" layer="95" xref="yes"/>
+<pinref part="C7" gate="G$1" pin="1"/>
+<wire x1="279.4" y1="-116.84" x2="279.4" y2="-106.68" width="0.1524" layer="91"/>
+<wire x1="279.4" y1="-106.68" x2="292.1" y2="-106.68" width="0.1524" layer="91"/>
+<junction x="279.4" y="-106.68"/>
+<wire x1="279.4" y1="-106.68" x2="279.4" y2="-101.6" width="0.1524" layer="91"/>
 </segment>
 <segment>
@@
 <label x="213.36" y="33.02" size="1.778" layer="95"/>
 </segment>
+<segment>
+<pinref part="U$3" gate="G$1" pin="VDD"/>
+<wire x1="5.08" y1="-109.22" x2="15.24" y2="-109.22" width="0.1524" layer="91"/>
+<label x="15.24" y="-109.22" size="1.27" layer="95" xref="yes"/>
+</segment>
 </net>
 <net name="BOOT0" class="0">
@@
 <label x="121.92" y="-20.32" size="1.27" layer="95" rot="R180" xref="yes"/>
 <pinref part="J1" gate="G$1" pin="7"/>
-</segment>
-<segment>
-<pinref part="IC1" gate="G$1" pin="DTR"/>
-<wire x1="160.02" y1="-116.84" x2="167.64" y2="-116.84" width="0.1524" layer="91"/>
-<label x="167.64" y="-116.84" size="1.778" layer="95"/>
 </segment>
 </net>
@@
 </segment>
 <segment>
-<pinref part="IC1" gate="G$1" pin="RTS"/>
-<wire x1="160.02" y1="-127" x2="167.64" y2="-127" width="0.1524" layer="91"/>
-<label x="167.64" y="-127" size="1.778" layer="95"/>
-</segment>
-<segment>
 <pinref part="JP2" gate="A" pin="1"/>
 <wire x1="-40.64" y1="93.98" x2="-30.48" y2="93.98" width="0.1524" layer="91"/>
@@
 <label x="279.4" y="-121.92" size="1.27" layer="95" xref="yes"/>
 </segment>
+<segment>
+<pinref part="IC1" gate="G$1" pin="CTS"/>
+<wire x1="160.02" y1="-129.54" x2="167.64" y2="-129.54" width="0.1524" layer="91"/>
+<label x="167.64" y="-129.54" size="1.778" layer="95"/>
+</segment>
 </net>
 <net name="ESP_RST" class="0">
@@
 <wire x1="236.22" y1="-121.92" x2="228.6" y2="-121.92" width="0.1524" layer="91"/>
 <label x="228.6" y="-121.92" size="1.27" layer="95" rot="R180" xref="yes"/>
+</segment>
+<segment>
+<pinref part="IC1" gate="G$1" pin="RTS"/>
+<wire x1="160.02" y1="-127" x2="167.64" y2="-127" width="0.1524" layer="91"/>
+<label x="167.64" y="-127" size="1.778" layer="95"/>
 </segment>
 </net>
@@
 <label x="-30.48" y="99.06" size="1.27" layer="95" xref="yes"/>
 </segment>
+<segment>
+<pinref part="U1" gate="G$1" pin="IO17"/>
+<wire x1="271.78" y1="-144.78" x2="281.94" y2="-144.78" width="0.1524" layer="91"/>
+<label x="281.94" y="-144.78" size="1.27" layer="95" xref="yes"/>
+</segment>
 </net>
 <net name="STM_TX" class="0">
@@
 <label x="-30.48" y="96.52" size="1.27" layer="95" xref="yes"/>
 </segment>
+<segment>
+<pinref part="U1" gate="G$1" pin="IO16"/>
+<wire x1="271.78" y1="-142.24" x2="281.94" y2="-142.24" width="0.1524" layer="91"/>
+<label x="281.94" y="-142.24" size="1.27" layer="95" xref="yes"/>
+</segment>
 </net>
 <net name="SPI3_NSS" class="0">
@@
 <pinref part="J1" gate="G$1" pin="23"/>
 <label x="127" y="-40.64" size="1.27" layer="95" rot="R180" xref="yes"/>
-<wire x1="114.3" y1="-40.64" x2="129.54" y2="-40.64" width="0.1524" layer="91"/>
+<wire x1="127" y1="-40.64" x2="129.54" y2="-40.64" width="0.1524" layer="91"/>
 </segment>
 <segment>
@@
 </segment>
 <segment>
-<pinref part="U1" gate="G$1" pin="IO15"/>
-<wire x1="271.78" y1="-139.7" x2="276.86" y2="-139.7" width="0.1524" layer="91"/>
-<label x="276.86" y="-139.7" size="1.27" layer="95" xref="yes"/>
+<label x="279.4" y="-137.16" size="1.27" layer="95" xref="yes"/>
+<pinref part="U1" gate="G$1" pin="IO14"/>
+<wire x1="271.78" y1="-137.16" x2="279.4" y2="-137.16" width="0.1524" layer="91"/>
 </segment>
 <segment>
@@
 <pinref part="JP9" gate="G$1" pin="1"/>
 </segment>
+<segment>
+<pinref part="U$3" gate="G$1" pin="CMD"/>
+<wire x1="5.08" y1="-106.68" x2="15.24" y2="-106.68" width="0.1524" layer="91"/>
+<label x="15.24" y="-106.68" size="1.27" layer="95" xref="yes"/>
+</segment>
 </net>
 <net name="ESP_MISO" class="0">
@@
 <pinref part="JP8" gate="G$1" pin="1"/>
 </segment>
+<segment>
+<pinref part="U$3" gate="G$1" pin="DAT0"/>
+<wire x1="5.08" y1="-116.84" x2="15.24" y2="-116.84" width="0.1524" layer="91"/>
+<label x="15.24" y="-116.84" size="1.27" layer="95" xref="yes"/>
+</segment>
 </net>
 <net name="ESP_CLK" class="0">
@@
 <pinref part="JP7" gate="G$1" pin="1"/>
 </segment>
+<segment>
+<pinref part="U$3" gate="G$1" pin="CLK"/>
+<wire x1="5.08" y1="-111.76" x2="15.24" y2="-111.76" width="0.1524" layer="91"/>
+<label x="15.24" y="-111.76" size="1.27" layer="95" xref="yes"/>
+</segment>
 </net>
 <net name="ESP_CS" class="0">
@@
 <segment>
 <pinref part="J1" gate="G$1" pin="21"/>
-<label x="127" y="-38.1" size="1.27" layer="95" rot="R180" xref="yes"/>
-<pinref part="JP4" gate="G$1" pin="2"/>
-<wire x1="129.54" y1="-38.1" x2="114.3" y2="-38.1" width="0.1524" layer="91"/>
+<label x="129.54" y="-38.1" size="1.27" layer="95" rot="R180" xref="yes"/>
+<pinref part="JP3" gate="G$1" pin="2"/>
+<wire x1="129.54" y1="-38.1" x2="114.3" y2="-35.56" width="0.1524" layer="91"/>
 </segment>
 </net>
@@
 <segment>
 <pinref part="J1" gate="G$1" pin="19"/>
-<label x="127" y="-35.56" size="1.27" layer="95" rot="R180" xref="yes"/>
-<pinref part="JP3" gate="G$1" pin="2"/>
-<wire x1="114.3" y1="-35.56" x2="129.54" y2="-35.56" width="0.1524" layer="91"/>
+<pinref part="JP4" gate="G$1" pin="2"/>
+<wire x1="114.3" y1="-38.1" x2="129.54" y2="-35.56" width="0.1524" layer="91"/>
+<label x="129.54" y="-35.56" size="1.27" layer="95" rot="R180" xref="yes"/>
 </segment>
 </net>
@@
 </segment>
 </net>
+<net name="MICROSD_CS" class="0">
+<segment>
+<pinref part="U$3" gate="G$1" pin="CD/DAT3"/>
+<wire x1="5.08" y1="-104.14" x2="15.24" y2="-104.14" width="0.1524" layer="91"/>
+<label x="15.24" y="-104.14" size="1.27" layer="95" xref="yes"/>
+</segment>
+<segment>
+<pinref part="U1" gate="G$1" pin="IO13"/>
+<wire x1="271.78" y1="-134.62" x2="279.4" y2="-134.62" width="0.1524" layer="91"/>
+<label x="279.4" y="-134.62" size="1.27" layer="95" xref="yes"/>
+</segment>
+</net>

Commit message: sync
Parts:
- removed FB4: FBCHIP-0603(1608-METRIC), Filter:FBCHIP-0603(1608-METRIC)
- removed HSE: 8MHZ, crystal:CRYSTALCTS406
- removed JP1: PINHD-1X2, Connector:PINHD-1X2
- removed JP10, JP11, JP12, JP3, JP4, JP7, JP8, JP9: JUMPER-SMT_2_NC_TRACE_NO-SILK, SparkFun-Jumpers:JUMPER-SMT_2_NC_TRACE_NO-SILK
- removed U$10: USB-MINIB-5PIN, Ciseco USB miniB_Updated:USB-MINIB-5PIN
- added 5VUSB: (no value), adafruit:USBMOLEX
- added LED2: (no value), led:LEDCHIP-LED0805
- added PAD1, PAD2, PAD3, PAD4: (no value), wirepad:1,6/0,8
- added Q1, Q2: (no value), microbuilder:TRANSISTOR_NPN
- added Q3: (no value), adafruit:XTAL-4-3225
- added R11: 10k, resistor:R-EU_R0603
- added R12: 510R, resistor:R-EU_R0603
- added R13: 0R, resistor:R-EU_R0603
- added U2: (no value), microbuilder:ESDDIODEARRAY_SINGLE_UNIDIR
- FB1, FB2: value FBCHIP-0603(1608-METRIC) -> 0R
- R9: device rcl:R-EU_R0603 -> resistor:R-EU_R0603
Connections:
- removed net CP2102_RX: IC1.RXD, JP1.1, JP11.1
- removed net CP2102_TX: IC1.TXD, JP1.2, JP12.1
- removed net ESP_CLK: JP7.1, U$3.CLK, U1.IO18
- removed net ESP_CS: JP10.1, U1.IO5
- removed net ESP_MISO: JP8.1, U$3.DAT0, U1.IO19
- removed net ESP_MOSI: JP9.1, U$3.CMD, U1.IO23
- removed net ESP_RST: IC1.RTS, U1.EN
- removed net RPI_CS: J1.24, JP10.2, JP6.1
- removed net RPI_MISO: J1.21, JP3.2, JP8.2
- removed net RPI_MOSI: J1.19, JP4.2, JP9.2
- removed net SPI3_MISO: JP4.1, STM32.PB4, U$2.SDO
- removed net SPI3_MOSI: JP3.1, STM32.PB5, U$2.SDI
- new net CP2102_DTR: IC1.DTR, Q1.E, R9.2
- new net CP2102_RTS: IC1.RTS, Q2.E, R11.2
- new net ESP_EN: PAD1.P, Q2.C, U1.EN
- new net MISO: J1.21, STM32.PB4, U$2.SDO, U$3.DAT0, U1.IO19
- new net MOSI: J1.19, STM32.PB5, U$2.SDI, U$3.CMD, U1.IO23
- new net N$11: J1.13
- new net N$13: LED2.A, R12.1
- new net N$6: Q2.B, R9.1
- new net N$7: Q1.B, R11.1
- new net N$9: J1.15
- new net RPI|ESP_CS: J1.24, JP6.1, U1.IO5
- net +3V3: now also U2.SUPPLYPIN
- net +5V: now also R12.2; no longer J1.2, J1.4
- net +5V_EXT: now also 5VUSB.VBUS, J1.2, J1.4; no longer U$10.VBUS
- net AGND: now also C18.2, C5.2, CF1.2, CF2.2, CF3.2, CFV.2, R13.1, R23.1, U2.GNDPIN; no longer FB4.1
- net BIAS: now also U2.IO
- net D+: now also 5VUSB.D+; no longer U$10.D+
- net D-: now also 5VUSB.D-; no longer U$10.D-
- net ESP_BOOT0: now also PAD2.P, Q1.C; no longer IC1.CTS
- net ESP_RX: now also IC1.TXD, PAD3.P; no longer JP12.2
- net ESP_TX: now also IC1.RXD, PAD4.P; no longer JP11.2
- net GND: now also 5VUSB.GND, LED2.C, MCP1825.GND@1, R13.2; no longer C18.2, C5.2, CF1.2, CF2.2, CF3.2, CFV.2, FB4.2, R23.1, R9.1, U$10.GND, U$10.MTN1, U$10.MTN2, U$10.MTN3, U$10.MTN4
- net HSE_IN_: now also Q3.X2; no longer HSE.1
- net HSE_OUT: now also Q3.X1; no longer HSE.2
- net RFM_IRQ: now also J1.16
- net RFM_RST: now also J1.18
- net RPI_CONNECTED: now also U1.IO4; no longer R9.2, U1.IO14
- net SPI_CLK: now also U$3.CLK, U1.IO18; no longer JP7.2
Other:
- note added: "BIAS input"
- note added: "CP2102 USB-TTL converter"
- note added: "DS18B20 pullup"
- note added: "ESP32 WROOM"
- note added: "LED"
- note added: "auto boot/reset for esp32"
- note added: "boot mode"
- note added: "input protection"
- note added: "microSD card adaptor"
- note added: "pulse input filter"
- note added: "raspberryPi header"
- note added: "reset"
- note added: "rfm69 radio"
- note added: "todo: . Protection Diode (done on BIAS)"
- note removed: "todo: . Protection Diode"
- moved on the sheet: C13, C17, J1, JP6, R8, R9, SMA

Commit message: sync
Other:
- note added: "2.0-2.35mm center pin dia."
Changed lines of the file:
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@@
 <layer number="91" name="Nets" color="2" fill="1" visible="yes" active="yes"/>
 <layer number="92" name="Busses" color="1" fill="1" visible="yes" active="yes"/>
-<layer number="93" name="Pins" color="2" fill="1" visible="no" active="yes"/>
+<layer number="93" name="Pins" color="2" fill="1" visible="yes" active="yes"/>
 <layer number="94" name="Symbols" color="4" fill="1" visible="yes" active="yes"/>
 <layer number="95" name="Names" color="7" fill="1" visible="yes" active="yes"/>
@@
 <text x="-30.48" y="-88.9" size="3.81" layer="91">microSD card
 adaptor</text>
+<text x="270.764" y="200.152" size="1.778" layer="97">2.0-2.35mm center pin dia.</text>
 </plain>
 <instances>

Commit message: sync
Parts:
- U2: MPN (none) -> NUP1301ML3T1G
- renumbered Q3 to Y1
Other:
- note removed: "2.0-2.35mm center pin dia."
Changed lines of the file:
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@@
 <layer number="91" name="Nets" color="2" fill="1" visible="yes" active="yes"/>
 <layer number="92" name="Busses" color="1" fill="1" visible="yes" active="yes"/>
-<layer number="93" name="Pins" color="2" fill="1" visible="yes" active="yes"/>
+<layer number="93" name="Pins" color="2" fill="1" visible="no" active="yes"/>
 <layer number="94" name="Symbols" color="4" fill="1" visible="yes" active="yes"/>
 <layer number="95" name="Names" color="7" fill="1" visible="yes" active="yes"/>
@@
 <part name="PAD3" library="wirepad" library_urn="urn:adsk.eagle:library:412" deviceset="1,6/0,8" device="" package3d_urn="urn:adsk.eagle:package:30830/1"/>
 <part name="PAD4" library="wirepad" library_urn="urn:adsk.eagle:library:412" deviceset="1,6/0,8" device="" package3d_urn="urn:adsk.eagle:package:30830/1"/>
-<part name="U2" library="microbuilder" deviceset="ESDDIODEARRAY_SINGLE_UNIDIR" device=""/>
+<part name="U2" library="microbuilder" deviceset="ESDDIODEARRAY_SINGLE_UNIDIR" device="">
+<attribute name="MPN" value="NUP1301ML3T1G"/>
+</part>
 <part name="R12" library="resistor" deviceset="R-EU_" device="R0603" value="510R"/>
 <part name="LED2" library="led" library_urn="urn:adsk.eagle:library:259" deviceset="LED" device="CHIP-LED0805" package3d_urn="urn:adsk.eagle:package:15818/2"/>
@@
 <part name="R13" library="resistor" deviceset="R-EU_" device="R0603" value="0R"/>
 <part name="5VUSB" library="adafruit" deviceset="USB" device="MOLEX"/>
-<part name="Q3" library="adafruit" deviceset="XTAL-4" device="-3225"/>
+<part name="Y1" library="adafruit" deviceset="XTAL-4" device="-3225"/>
 </parts>
 <sheets>
@@
 <text x="-30.48" y="-88.9" size="3.81" layer="91">microSD card
 adaptor</text>
-<text x="270.764" y="200.152" size="1.778" layer="97">2.0-2.35mm center pin dia.</text>
 </plain>
 <instances>
@@
 </instance>
 <instance part="U2" gate="G$1" x="129.54" y="129.54" smashed="yes" rot="R180">
-<attribute name="NAME" x="120.65" y="128.27" size="1.27" layer="95" rot="R180"/>
+<attribute name="NAME" x="121.412" y="131.826" size="1.27" layer="95" rot="R180"/>
 <attribute name="VALUE" x="120.65" y="130.81" size="1.27" layer="96" rot="R180"/>
+<attribute name="MPN" x="130.048" y="124.46" size="1.778" layer="96"/>
 </instance>
 <instance part="R12" gate="G$1" x="-55.88" y="165.1" smashed="yes" rot="R90">
@@
 <attribute name="VALUE" x="83.82" y="167.64" size="1.27" layer="96"/>
 </instance>
-<instance part="Q3" gate="G$1" x="48.26" y="124.46" smashed="yes" rot="R90">
+<instance part="Y1" gate="G$1" x="48.26" y="124.46" smashed="yes" rot="R90">
 <attribute name="NAME" x="44.45" y="121.92" size="1.27" layer="95" font="vector" rot="R90"/>
 <attribute name="VALUE" x="53.34" y="120.65" size="1.27" layer="96" font="vector" rot="R90"/>
@@
 <wire x1="38.1" y1="114.3" x2="38.1" y2="119.38" width="0.1524" layer="91"/>
 <label x="38.1" y="129.54" size="1.778" layer="95" rot="R90"/>
-<pinref part="Q3" gate="G$1" pin="X1"/>
+<pinref part="Y1" gate="G$1" pin="X1"/>
 <wire x1="38.1" y1="119.38" x2="38.1" y2="129.54" width="0.1524" layer="91"/>
 <wire x1="38.1" y1="119.38" x2="48.26" y2="119.38" width="0.1524" layer="91"/>
@@
 <wire x1="27.94" y1="114.3" x2="27.94" y2="121.92" width="0.1524" layer="91"/>
 <pinref part="R10" gate="G$1" pin="1"/>
-<pinref part="Q3" gate="G$1" pin="X2"/>
+<pinref part="Y1" gate="G$1" pin="X2"/>
 <wire x1="27.94" y1="121.92" x2="48.26" y2="129.54" width="0.1524" layer="91"/>
 <junction x="27.94" y="121.92"/>
